Commit message: robot + parser ok

File: robots/robot_marcheur_4/robot.urdf (robot description, URDF)
Before this commit: robot onshape, 62 links, 61 joints
Links:
- removed link centre_pied
- removed link fermeture10_A
- removed link fermeture10_B
- removed link hanche_2
- added link bout_pied, mass 1e-9
- added link fermeture0_A, mass 1e-9
- added link fermeture0_B, mass 1e-9
- added link hanche_batis, mass 1.1356034209800021095; collision mesh filename=package:///hanche_batis.stl; visual mesh filename=package:///hanche_batis.stl
- link foot: mass 0.4130405170811343174 -> 0.41304051708113420638
- link hanche: mass 1.1356034209800021095 -> 0.14955339898895028683
- link renvois_hanche: mass 0.052048361392958063243 -> 0.052048361392958070182
- link rode_foot: mass 0.04066693929476376812 -> 0.040666939294763761181
- link rode_foot_2: mass 0.04066693929476376812 -> 0.040666939294763761181
- link rode_foot_3: mass 0.04066693929476376812 -> 0.040666939294763761181
- link rode_foot_4: mass 0.04066693929476376812 -> 0.040666939294763761181
- link tarsus: mass 2.1073238681812558326 -> 2.1073238681812553885
Joints:
- removed joint centre_pied_frame
- removed joint fermeture10_A_frame
- removed joint fermeture10_B_frame
- added joint bout_pied_frame: type fixed, parent foot, child bout_pied, origin xyz=0.014111017407571480042 0.044041666666666756669 1.5991513668822676664e-09 rpy=-1.570796326794896558 1.3017041712644265466e-17 3.141592653589793116, axis 0 0 0
- added joint fermeture0_A_frame: type fixed, parent rode_tarsus, child fermeture0_A, origin xyz=0 2.7755575615628913511e-16 -0.19189583333333326554 rpy=3.141592653589793116 -1.6721638379069471494e-17 3.075854684320635955e-18, axis 0 0 0
- added joint fermeture0_B_frame: type fixed, parent rode_tarsus_4, child fermeture0_B, origin xyz=5.5511151231257827021e-17 -1.1102230246251565404e-16 -0.19189583333333348758 rpy=2.5464045949721037905e-16 -3.8499906812161220182e-16 -3.141592653589793116, axis 0 0 0
- joint centre_hanche_frame: origin xyz=0.0072868371002145423954 -0.12388192121052921113 5.290906601729261638e-17 rpy=0 -1.5429430116984873749e-15 0 -> xyz=0.0072868371002148442372 -0.28888192121052924666 -0.19749999999999995337 rpy=0 -1.5429430116984873749e-15 0; parent hanche -> hanche_batis
- joint fermeture1_A_frame: origin xyz=0 0 -0.025000000000000133227 rpy=8.8831754777918187002e-30 -2.3157694083552497375e-29 2.8144901665607526915e-30 -> xyz=1.3877787807814456755e-17 -5.5511151231257827021e-17 -0.025000000000000160982 rpy=-1.8744017465649457593e-18 -9.818041624348521577e-17 -2.79836129840733741e-20
- joint fermeture1_B_frame: origin xyz=-2.7755575615628913511e-17 -5.5511151231257827021e-17 -0.025000000000000244249 rpy=-3.141592653589793116 -6.2877883210336418487e-17 3.1275980329687938195e-17 -> xyz=-8.3266726846886740532e-17 -5.5511151231257827021e-17 -0.025000000000000244249 rpy=-3.141592653589793116 -8.7685925630935976107e-17 2.9906032515748721767e-17
- joint fermeture2_A_frame: origin xyz=0 0 -0.024999999999999994449 rpy=4.5710791672064410631e-29 -6.6855961717480750509e-29 7.600290954118671857e-29 -> xyz=-6.9388939039072283776e-18 -5.5511151231257827021e-17 -0.025000000000000105471 rpy=1.7473559706539229754e-22 -5.5001239547193146538e-21 1.6842726119609899759e-24
- joint fermeture2_B_frame: origin xyz=4.1633363423443370266e-17 0 -0.025000000000000188738 rpy=3.141592653589793116 1.3779502303722609972e-17 -1.6028373921264690291e-17 -> xyz=1.1102230246251565404e-16 2.7755575615628913511e-17 -0.025000000000000133227 rpy=-3.141592653589793116 3.1456406373773374106e-16 -5.3319186701923333256e-17
- joint fermeture3_A_frame: origin xyz=1.3877787807814456755e-17 0 -0.025000000000000188738 rpy=3.141592653589793116 1.1832913578315177081e-30 2.6715483397867810683e-30 -> xyz=0 -5.5511151231257827021e-17 -0.025000000000000216493 rpy=-3.141592653589793116 -1.4924298254456226231e-19 -4.5162089082963286946e-24
- joint fermeture3_B_frame: origin xyz=0 0 -0.025000000000000077716 rpy=-1.5777218104420376238e-30 -2.8398992587956424995e-29 4.5495763117987201118e-30 -> xyz=-1.3877787807814456755e-17 2.7755575615628913511e-17 -0.025000000000000133227 rpy=7.7095856618526664724e-20 -2.8590462254934253294e-20 1.8588697243342543712e-18
- joint fermeture4_A_frame: origin xyz=1.3877787807814456755e-17 0 -0.025000000000000188738 rpy=3.141592653589793116 1.1832913578315177081e-30 2.6715483397867810683e-30 -> xyz=0 8.3266726846886740532e-17 -0.025000000000000077716 rpy=-3.141592653589793116 -1.4924298254456226231e-19 -4.5162089082963286946e-24
- joint fermeture4_B_frame: origin xyz=0 0 -0.025000000000000077716 rpy=-1.5777218104420376238e-30 -2.8398992587956424995e-29 4.5495763117987201118e-30 -> xyz=0 -2.7755575615628913511e-17 -0.025000000000000022204 rpy=1.1160994889302602654e-18 6.2394804750431383568e-20 1.1774112289867942571e-17
- joint fermeture5_B_frame: origin xyz=0 -1.3877787807814456755e-17 -0.025000000000000074246 rpy=-3.141592653589793116 3.0278985551981991197e-28 -1.570796326794896558 -> xyz=-8.3266726846886740532e-17 -2.7755575615628913511e-17 -0.025000000000000105471 rpy=3.141592653589793116 3.025978467155636249e-28 -1.570796326794896558
- joint fermeture6_A_frame: origin xyz=-5.5511151231257827021e-17 -6.9388939039072283776e-18 -0.2225000000000000866 rpy=9.211775309298636418e-27 -7.0307228177822677157e-28 -1.570796326794896558 -> xyz=-6.9388939039072283776e-18 -1.6653345369377348106e-16 -0.28249999999999997335 rpy=-4.2029392900949747559e-17 -7.4606014470714686977e-18 -1.570796326794896558
- joint fermeture6_B_frame: origin xyz=0 0 -0.025000000000000022204 rpy=3.141592653589793116 -2.622962509859864253e-29 -3.141592653589793116 -> xyz=-3.6082248300317587564e-16 1.6653345369377348106e-16 -0.025000000000000133227 rpy=-3.141592653589793116 1.1119874650498309646e-21 3.141592653589793116
- joint fermeture7_A_frame: origin xyz=-1.1102230246251565404e-16 -2.6367796834847467835e-16 -0.207625000000000004 rpy=-3.1415926535897913396 -2.9426902788492800649e-16 -1.5707963267948954478 -> xyz=-2.7755575615628913511e-17 -3.0531133177191804862e-16 -0.20762500000000022604 rpy=3.1415926535897846783 2.3079233611404340129e-17 -1.570796326794896558
- joint fermeture7_B_frame: origin xyz=-1.3877787807814456755e-17 -2.2204460492503130808e-16 -0.20762500000000011502 rpy=1.794624726976586498e-17 1.2103825396487620425e-17 -3.141592653589793116 -> xyz=4.1633363423443370266e-17 -3.0531133177191804862e-16 -0.20762499999999989297 rpy=4.7657994470008846293e-18 1.6442732956008238335e-17 -3.141592653589793116
- joint fermeture8_A_frame: origin xyz=-2.7755575615628913511e-17 5.5511151231257827021e-17 -0.207625000000000004 rpy=-2.6307610252349813393e-16 -4.4967931276871329446e-17 3.1415926535897926719 -> xyz=-1.3877787807814456755e-17 -4.4408920985006261617e-16 -0.20762499999999994849 rpy=-2.9697957125138915857e-16 -4.8836916697961571375e-16 3.1415926535897926719
- joint fermeture8_B_frame: origin xyz=-1.1102230246251565404e-16 -1.6653345369377348106e-16 -0.20762500000000005951 rpy=-3.141592653589793116 2.9827937381168234235e-17 1.2988615198508003668e-17 -> xyz=-2.7755575615628913511e-17 1.1102230246251565404e-16 -0.20762500000000005951 rpy=3.141592653589793116 4.8299363385392145085e-17 3.5495078826400279975e-19
- joint fermeture9_A_frame: origin xyz=0 2.7755575615628913511e-17 -0.19189583333333337656 rpy=-4.1946134630726214399e-30 -2.8134745357242634154e-17 -3.141592653589793116 -> xyz=0 -3.3306690738754696213e-16 -0.19189583333333326554 rpy=6.9071019648092707407e-18 2.6624167757425087404e-17 -3.141592653589793116
- joint fermeture9_B_frame: origin xyz=-6.9388939039072283776e-18 2.7755575615628913511e-17 -0.19189583333333304349 rpy=-3.141592653589793116 -3.3743525220828779976e-28 3.0361798708208753015e-29 -> xyz=0 1.1102230246251565404e-16 -0.19189583333333337656 rpy=3.141592653589793116 -1.6721638379069471494e-17 3.075854684320635955e-18
- joint free_attache_moeur_hanche_1: origin xyz=0.012500000000000000694 -0.0424687499999999718 -0.08808333333333337456 rpy=1.570796326794896558 1.5777218104420306173e-30 -1.570796326794896558 -> xyz=0.012499999999999990286 -0.0424687499999999718 -0.088083333333333277415 rpy=1.570796326794896558 0.0047435069561565304519 -1.570796326794896336; parent hanche_2 -> hanche
- joint free_attache_moeur_hanche_2: parent hanche -> hanche_batis
- joint free_attache_moeur_hanche_3: origin xyz=0.012500000000000000694 0.042468750000000027311 -0.08808333333333337456 rpy=1.570796326794896558 1.5777218104420306173e-30 -1.570796326794896558 -> xyz=0.012500000000000011102 0.042468750000000055067 -0.088083333333333485582 rpy=1.570796326794896558 0.0047908213534053481833 -1.57079632679489678; parent hanche_2 -> hanche
- joint free_attache_moeur_hanchexy: origin xyz=0 2.0816681711721685133e-16 -0.062916666666666690166 rpy=-0 -1.5707963267948950037 0 -> xyz=-5.5511151231257827021e-17 3.1918911957973250537e-16 -0.062916666666666662411 rpy=-1.570796326794672737 -1.5705013744383484742 1.5707963267936437823
- joint free_attache_moeur_hanchexy2: origin xyz=0 -1.3877787807814456755e-17 -0.062916666666666662411 rpy=-0 -1.5707963267948950037 0 -> xyz=-8.3266726846886740532e-17 -1.3877787807814456755e-16 -0.062916666666666676289 rpy=-1.5707963267950315611 -1.5704936563091338453 1.5707963267928437556
- joint free_cardan_xhips: origin xyz=7.5000000000019495516e-05 0 -7.5000000000000413558e-05 rpy=-3.141592653589793116 1.570796326794896558 0 -> xyz=7.4999999999936228789e-05 7.2164496600635175128e-16 -7.5000000000697772395e-05 rpy=1.5707963267932967266 1.5702141424144824278 -1.570796326796419784
- joint free_cardans_yhips: origin xyz=1.7347234759768070944e-18 0 -0.18875000000000008438 rpy=-1.570796326794896558 -8.6002330739638796169e-18 1.570796326794896558 -> xyz=9.5409791178724390193e-18 -2.7755575615628913511e-17 -0.18875000000000002887 rpy=-1.57079632679489678 -0.00013745695438837276787 1.570796326794896558; parent hanche_2 -> hanche
- joint free_cheville_cardanx: origin xyz=7.5000000000047251092e-05 0 -7.5000000000068067774e-05 rpy=-4.1267286104374180071e-29 -1.570796326794896558 0 -> xyz=7.4999999999825206487e-05 -2.2204460492503130808e-16 -7.5000000000002365122e-05 rpy=-1.570796326794896558 -1.0283708790559382695 1.570796326794896558
- joint free_cheville_cardany: origin xyz=-0.1698000000000028098 0.34604166666666669183 5.5511151231257827021e-17 rpy=-0 1.570796326794896558 0 -> xyz=-0.16980000000000278204 0.34604166666666646979 -1.1102230246251565404e-16 rpy=-1.5707963267942939289 1.5706585553043288517 -1.5707963267950366681
- joint free_genoux: origin xyz=0.17616666666662494922 -0.49075000000001511857 -0.081791666666666706931 rpy=3.141592653589793116 -3.8921152931043281558e-31 4.1415197524103119784e-30 -> xyz=0.17616666666662503249 -0.49075000000001500755 -0.081791666666666845709 rpy=3.141592653589793116 -1.2407226412650767997e-16 -0.00058875972722544967809
- joint free_renvois_hanche1: origin xyz=0.072354166666666955288 -0.053479166666666633212 -0.13527083333333345117 rpy=1.308414229027936131e-29 7.507728643138478293e-30 0.37563002773728437766 -> xyz=0.072354166666666039354 -0.053479166666666105856 -0.13527083333333353443 rpy=-8.54568753867082763e-17 -1.8407509512760167408e-16 0.43838119428272348532
- joint free_renvois_hanche2: origin xyz=0.072354166666666844265 -0.053479166666666633212 -0.028312500000000018208 rpy=3.141592653589793116 -1.5804407405094530311e-30 0.26045626790084336344 -> xyz=0.072354166666667982244 -0.05347916666666752139 -0.028312500000000073719 rpy=3.141592653589793116 1.1335268030418274217e-15 0.40020166506191917621
- joint free_triangle1_tibias: origin xyz=0.13841666666666663232 -0.47187500000000004441 -0.044041666666666701158 rpy=3.141592653589793116 1.9899601408349094571e-30 -0.32415406750443093165 -> xyz=0.13841666666666663232 -0.47187499999999993339 -0.044041666666666784424 rpy=-3.141592653589793116 -1.3748255421293126449e-16 -0.066056290258646024882
- joint free_triangle2_tibias: origin xyz=0.13841666666666660457 -0.47187500000000015543 -0.1195416666666667127 rpy=-5.8177101283745972593e-29 9.3322004381232959028e-30 -0.23874661370881070099 -> xyz=0.13841666666666668783 -0.47187499999999993339 -0.11954166666666668495 rpy=-1.8461492555022878416e-18 -1.0252669703201268269e-16 -0.10263776941217567229
- joint free_zhips: child hanche_2 -> hanche; origin xyz=-0.012499999999999976408 -0.20499999999999998779 -0.0049999999999998934186 rpy=-7.8886090522101180541e-31 1.5429430116984919109e-15 3.141592653589793116 -> xyz=-0.012499999999999986816 -0.20499999999999996003 -0.0049999999999998934186 rpy=-1.4726037963295123608e-16 1.5370811015985778338e-15 3.0459941681722826345; parent hanche -> hanche_batis
- joint mot_cheville1: origin xyz=0 0 2.498001805406602216e-16 rpy=-3.141592653589793116 6.705317694378600346e-29 3.141592653589793116 -> xyz=1.3877787807814456755e-17 -1.3877787807814456755e-16 -4.1245097658793028472e-05 rpy=3.141592653589793116 5.6902940387883940848e-17 -3.141592653589793116
- joint mot_cheville2: origin xyz=-9.7144514654701197287e-17 2.2204460492503130808e-16 -4.7184478546569152968e-16 rpy=-3.141592653589793116 2.3759403100678058489e-29 3.141592653589793116 -> xyz=6.2450045135165055399e-17 -2.2204460492503130808e-16 -2.9548398438994372128e-05 rpy=-3.141592653589793116 -1.2075888392074055418e-16 3.141592653589793116
- joint mot_genoux: origin xyz=-6.9388939039072283776e-18 5.5511151231257827021e-17 -0.062916666666666620777 rpy=-1.3213420162451947741e-29 -1.4845376160127915913e-28 1.570796326794896558 -> xyz=-5.5511151231257827021e-17 7.6327832942979512154e-17 -0.063110639745103724874 rpy=-6.0511400049598649395e-18 4.1907451314458865479e-18 1.570796326794896558
- joint mot_hanchexy1: origin xyz=-1.3877787807814456755e-17 -0.031458333333333254878 0 rpy=-1.570796326794896558 3.0366328384956959949e-47 0 -> xyz=5.5511151231257827021e-17 -0.03147530555841833444 8.3266726846886740532e-17 rpy=-1.570796326794896558 -4.8539988437297803109e-17 3.2508222489336867815e-16
- joint mot_hanchexy2: origin xyz=-1.3877787807814456755e-17 -0.031458333333333476922 -5.5511151231257827021e-17 rpy=-1.570796326794896558 3.0366328384956959949e-47 0 -> xyz=4.1633363423443370266e-17 -0.031475761426423623512 0 rpy=-1.570796326794896558 -4.0842560888460044134e-16 3.7225087496077564125e-16
- joint to_rotule_free_attache2_moeur_hanchez: origin xyz=1.616762279610384212e-15 0.044041666666666673402 -0.053479166666666744234 rpy=1.570796326794896558 7.4941785995994790281e-30 1.570796326794896558 -> xyz=1.7078352620991665844e-15 0.044041666666666673402 -0.053479166666666723418 rpy=1.570796326794896558 -1.9832067293240475674e-17 1.570796326794896558; parent hanche_2 -> hanche
- joint to_rotule_free_attache_genoux: origin xyz=-0.044041666666666673402 0.050333333333333230009 -5.5511151231257827021e-17 rpy=-1.57079632679489678 1.9438969795233453561e-29 -9.6635460889573946163e-30 -> xyz=-0.044041666666667284025 0.050333333333332563875 5.5511151231257827021e-17 rpy=-1.57079632679489678 0.026729912583035628226 -8.6038674056888522762e-19
- joint to_rotule_free_attache_hanche1: origin xyz=-0.13212500000000010347 -0.037750000000000172307 -2.7755575615628913511e-16 rpy=-1.57079632679489678 2.9120385417269680563e-17 -3.141592653589793116 -> xyz=-0.13212499999999993694 -0.037750000000000172307 5.5511151231257827021e-17 rpy=-1.57079632679489678 -0.094042986969348249526 -3.1415926535897926719
- joint to_rotule_free_attache_hanche2: origin xyz=-0.13212499999999988143 0.037750000000000116795 -2.7755575615628913511e-17 rpy=1.570796326794896558 8.014186960619273474e-18 3.141592653589793116 -> xyz=-0.13212499999999971489 0.037749999999999950262 -2.7755575615628913511e-17 rpy=1.570796326794896558 0.092185476461817641991 3.141592653589793116
- joint to_rotule_free_attache_moeur_4: origin xyz=-0.075500000000000150324 -0.044041666666666701158 -0.13527083333333378423 rpy=1.570796326794896558 -1.4677322981672841489e-30 1.242455925723093033e-29 -> xyz=-0.075500000000000150324 -0.044041666666666673402 -0.13527083333333314585 rpy=1.570796326794896558 0.095598525430158579064 -7.5072756837122450885e-16
- joint to_rotule_free_attache_moeur_5: origin xyz=-0.075500000000000150324 -0.044041666666666756669 -0.028312500000000073719 rpy=1.570796326794896558 -3.8063482729435784759e-29 3.4118234150808760584e-29 -> xyz=-0.075500000000000136446 -0.044041666666666645646 -0.028312499999999851674 rpy=1.570796326794896558 0.095598525430158620697 -6.4409731452178782971e-16
- joint to_rotule_free_attache_mour_6: origin xyz=0.037750000000000172307 -0.1887499999999999456 -0.081791666666666706931 rpy=1.570796326794896558 -2.30400890492067767e-30 -3.141592653589793116 -> xyz=0.037749999999999464539 -0.188749999999999446 -0.081791666666666845709 rpy=1.5707963267948961139 1.4741965910877770085 3.1415926535897922278
- joint to_rotule_free_foot1: origin xyz=-0.0629166666666667318 -0.012583333333333612813 0.04404166666666681218 rpy=1.570796326794896558 -6.7617285292989753398e-30 3.141592653589793116 -> xyz=-0.0629166666666667318 -0.012583333333333390769 0.044041666666666368091 rpy=1.570796326794896558 0.081892649261537886485 -3.141592653589793116
- joint to_rotule_free_goot2: origin xyz=-0.062916666666666745678 -0.012583333333333612813 -0.044041666666666590135 rpy=1.570796326794896558 -6.7617285292989753398e-30 3.141592653589793116 -> xyz=-0.062916666666666620777 -0.012583333333333168724 -0.044041666666666950958 rpy=1.570796326794896558 0.081892649261537886485 -3.141592653589793116
- joint to_rotule_free_hanche_attache1: origin xyz=0.069208333333333371673 -2.7755575615628913511e-17 -0.044041666666666645646 rpy=-1.57079632679489678 1.4184284915909716117e-30 -3.141592653589793116 -> xyz=0.069208333333333316162 -1.6653345369377348106e-16 -0.04404166666666681218 rpy=-1.57079632679489678 -0.095598525430158579064 3.1415926535897926719
- joint to_rotule_free_hanche_attache2: origin xyz=0.069208333333333357795 -2.7755575615628913511e-17 0.044041666666666645646 rpy=-1.57079632679489678 1.4184284915909716117e-30 -3.141592653589793116 -> xyz=0.069208333333333357795 0 0.044041666666666673402 rpy=-1.57079632679489678 -0.095598525430158579064 3.1415926535897926719
- joint to_rotule_free_renvois_hanche3: origin xyz=-0.10695833333333418236 -0.062916666666666842822 -3.7747582837255322374e-15 rpy=-1.57079632679489678 -3.8105612564473861213e-16 -3.5207910199695531523e-17 -> xyz=-0.10695833333333404358 -0.062916666666667009356 -1.6653345369377348106e-16 rpy=-1.57079632679489678 0.09404298696934784707 -4.8159767687053810446e-16
- joint to_rotule_free_renvois_hanche4: origin xyz=-0.10695833333333407134 0.062916666666667064867 5.5511151231257827021e-17 rpy=1.570796326794896558 -2.1694817664039273641e-17 -1.2103825396487620425e-17 -> xyz=-0.1069583333333340297 0.062916666666667064867 1.1102230246251565404e-16 rpy=1.570796326794896558 -0.092185476461817753013 2.6802825518558815111e-17
- joint to_rotule_free_triangle1: origin xyz=-0.068058330216350798603 0.012564119186792122029 -0.012583333333333335258 rpy=-1.57079632679489678 1.2422533291766141538e-17 -3.6260592545799792035e-17 -> xyz=-0.068058330216350965136 0.012564119186792344074 -0.012583333333333557302 rpy=-1.57079632679489678 0.16864244180508916604 3.6078898931567104179e-17
- joint to_rotule_free_triangle2: origin xyz=-0.068058330216350937381 -0.012564119186792344074 -0.012583333333333335258 rpy=1.570796326794896558 -9.8721378529962509943e-18 5.2019339086040904528e-17 -> xyz=-0.068058330216350965136 -0.012564119186792344074 -0.012583333333333057702 rpy=1.570796326794896558 -0.095385008856607569894 -2.6902869908268245684e-16
- joint to_rotule_free_triangle4: origin xyz=-0.041015624251386162413 -0.047709805194672050277 -0.047187500000000215383 rpy=-1.57079632679489678 -1.5156783735639931857e-19 -1.570796326794896558 -> xyz=-0.041015624251386273436 -0.047709805194671606188 -0.047187499999999826805 rpy=-1.57079632679489678 -0.095087883447032894857 3.141592653589793116
- joint to_rotule_free_trianle3: origin xyz=-0.041015624251386106902 0.047709805194672050277 -0.047187499999999882316 rpy=1.57079632679489678 -0.40246863389381404286 1.5707963267948956698 -> xyz=-0.041015624251385912613 0.047709805194671939255 -0.047187500000000021094 rpy=1.5707963267948961139 -1.4687456221646373322 3.141592653589658557
