Commit message: maj kangaroo

File: robots/robot_marcheur_4/robot.urdf (robot description, URDF)
Before this commit: robot onshape, 62 links, 61 joints
Links:
- removed link rode_foot
- removed link rode_foot_2
- removed link rode_foot_3
- removed link rode_foot_4
- added link fermeture10_A, mass 1e-9
- added link fermeture10_B, mass 1e-9
- added link part_18, mass 0.079498471341342247243; collision mesh filename=package:///part_18.stl; visual mesh filename=package:///part_18.stl
- added link part_19, mass 0.038809173972269447872; collision mesh filename=package:///part_19.stl; visual mesh filename=package:///part_19.stl
- added link part_19_2, mass 0.038809173972269447872; collision mesh filename=package:///part_19.stl; visual mesh filename=package:///part_19.stl
- added link part_19_3, mass 0.038809173972269447872; collision mesh filename=package:///part_19.stl; visual mesh filename=package:///part_19.stl
- added link part_19_4, mass 0.038809173972269447872; collision mesh filename=package:///part_19.stl; visual mesh filename=package:///part_19.stl
- added link part_19_5, mass 0.038809173972269447872; collision mesh filename=package:///part_19.stl; visual mesh filename=package:///part_19.stl
- added link part_19_6, mass 0.038809173972269447872; collision mesh filename=package:///part_19.stl; visual mesh filename=package:///part_19.stl
- link attache_hanche: mass 0.013302651224255402848 -> 0.012829478999097282399
- link cardan_foot: mass 0.0066552634961090364682 -> 0.0064135211594024193679
- link cardan_foot_2: mass 0.0066552634961090364682 -> 0.0064135211594024193679
- link cardan_hache: mass 0.015650981021718499836 -> 0.015608633111865832799
- link cardan_hache_2: mass 0.015650981021718499836 -> 0.015608633111865832799
- link foot: mass 0.41304051708113420638 -> 0.3109129822293019707
- link hanche: mass 0.14955339898895028683 -> 0.14908820646980575075
- link hanche_batis: mass 1.1356034209800021095 -> 1.5865591647149874799
- link moteur_hanche1: mass 0.046264571606101846657 -> 0.17794962537636818678
- link moteur_hanche1_2: mass 0.046264571606101846657 -> 0.17794962537636818678
- link motteur_rotation: mass 0.050662516966540720176 -> 0.19339251676417071324
- link motteur_rotation_2: mass 0.050662516966540720176 -> 0.19339251676417071324
- link motteur_rotation_3: mass 0.050662516966540720176 -> 0.19339251676417071324
- link motteur_rotation_4: mass 0.050662516966540720176 -> 0.19339251676417071324
- link piston: mass 0.0048966814322412765756 -> 0.0047041422996690132607
- link piston_10: mass 0.0048966814322412765756 -> 0.0047041422996690132607
- link piston_11: mass 0.0048966814322412765756 -> 0.0047041422996690132607
- link piston_12: mass 0.0048966814322412765756 -> 0.0047041422996690132607
- link piston_2: mass 0.0048966814322412765756 -> 0.0047041422996690132607
- link piston_3: mass 0.0048966814322412765756 -> 0.0047041422996690132607
- link piston_4: mass 0.0048966814322412765756 -> 0.0047041422996690132607
- link piston_5: mass 0.0048966814322412765756 -> 0.0047041422996690132607
- link piston_6: mass 0.0048966814322412765756 -> 0.0047041422996690132607
- link piston_7: mass 0.0048966814322412765756 -> 0.0047041422996690132607
- link piston_8: mass 0.0048966814322412765756 -> 0.0047041422996690132607
- link piston_9: mass 0.0048966814322412765756 -> 0.0047041422996690132607
- link renvois_cheville: mass 0.075465954638112592301 -> 0.074310321213956573305
- link renvois_cheville_2: mass 0.075465953879580452424 -> 0.074310320490076631206
- link renvois_hanche: mass 0.052048361392958070182 -> 0.039425066320412559262
- link renvois_hanche_2: mass 0.052048361392958070182 -> 0.039425066320412559262
- link rode_tarsus: mass 0.037586110560311969397 -> 0.035869085034976246062
- link rode_tarsus_2: mass 0.037586110560311969397 -> 0.035869085034976246062
- link rode_tarsus_3: mass 0.037586110560311969397 -> 0.035869085034976246062
- link rode_tarsus_4: mass 0.037586110560311969397 -> 0.035869085034976246062
- link tarsus: mass 2.1073238681812553885 -> 1.7306025451589581721
- link tibias: mass 0.17811841417215046324 -> 0.17161370666967495913
Joints:
- removed joint mot_genoux
- removed joint to_rotule_free_attache_moeur_4
- removed joint to_rotule_free_attache_moeur_5
- removed joint to_rotule_free_attache_mour_6
- added joint ferme_genoux: type revolute, parent tarsus, child part_18, origin xyz=-0.00046813081423362212785 -0.04675000000000356648 -0.071499999999999980238 rpy=-3.1415926535897904515 7.6158859627596601973e-16 0.1045651135355853828, axis 0 0 1, limit effort=1 velocity=20
- added joint fermeture10_A_frame: type fixed, parent part_19, child fermeture10_A, origin xyz=-1.1102230246251565404e-16 2.7755575615628913511e-16 -0.18149999999999993916 rpy=3.1415926535897895633 1.1988806635353361042e-15 1.570796326794896558, axis 0 0 0
- added joint fermeture10_B_frame: type fixed, parent part_19_6, child fermeture10_B, origin xyz=0 0 -0.18149999999999999467 rpy=-1.0968167807709025411e-17 2.3866997684138820983e-16 -1.570796326794896336, axis 0 0 0
- added joint moteur_genoux: type prismatic, parent motteur_rotation_3, child piston_8, origin xyz=-2.0330959138448179147e-15 1.1102230246251565404e-16 0.10897870887710439658 rpy=-3.141592653589793116 -4.6342802523994222001e-15 -3.7006813932455447112e-15, axis 0 0 1, limit effort=1 velocity=20
- added joint to_rotule_genoux: type revolute, parent part_18, child part_19_6, origin xyz=-0.032999999999999932165 0.066000000000000141887 -2.7755575615628913511e-16 rpy=-1.570796326794896558 -0.21052439488817287216 -3.1415926535897917837, axis 0 0 1, limit effort=1 velocity=20
- added joint to_rotule_genoux2: type revolute, parent tibias, child part_19, origin xyz=-0.038500000000000138278 0.043999999999999817035 2.2204460492503130808e-16 rpy=1.570796326794896558 6.0383780035333910048e-17 1.570796326794896558, axis 0 0 1, limit effort=1 velocity=20
- added joint to_rotule_moeur_cheville_1: type revolute, parent part_18, child motteur_rotation, origin xyz=-0.065531869185765770358 -0.0082499999999992856825 0.046750000000000013767 rpy=1.5707963267948970021 1.4895762776760668178 3.1415926535897735761, axis 0 0 1, limit effort=1 velocity=20
- added joint to_rotule_moeur_cheville_2: type revolute, parent part_18, child motteur_rotation_2, origin xyz=-0.065531869185765770358 -0.0082499999999992301714 -0.046749999999999986011 rpy=1.570796326794896558 -0.26428955298985623568 -3.141592653589788231, axis 0 0 1, limit effort=1 velocity=20
- added joint to_rotule_test: type revolute, parent tarsus, child motteur_rotation_3, origin xyz=-0.00046813081423358049449 -0.046750000000003455458 -0.071499999999999869216 rpy=1.5707963267948954478 -0.050362955011682315754 3.1688621187003315387e-15, axis 0 0 1, limit effort=1 velocity=20
- joint bout_pied_frame: origin xyz=0.014111017407571480042 0.044041666666666756669 1.5991513668822676664e-09 rpy=-1.570796326794896558 1.3017041712644265466e-17 3.141592653589793116 -> xyz=0.012016949221079924193 0.038500000000000089706 6.8117394502742456552e-09 rpy=1.570796326794896558 -8.8759669262812707343e-18 -1.5746176066600222494e-17
- joint centre_hanche_frame: origin xyz=0.0072868371002148442372 -0.28888192121052924666 -0.19749999999999995337 rpy=0 -1.5429430116984873749e-15 0 -> xyz=-0.004747469922900492828 0.288611431583448097 -0.17250000000000004219 rpy=0 -2.5097998118986334965e-18 0
- joint fermeture0_A_frame: origin xyz=0 2.7755575615628913511e-16 -0.19189583333333326554 rpy=3.141592653589793116 -1.6721638379069471494e-17 3.075854684320635955e-18 -> xyz=-6.9388939039072283776e-18 0 -0.16775000000000006573 rpy=3.141592653589793116 2.0456812790238454299e-17 -1.6970722323022375395e-17
- joint fermeture0_B_frame: origin xyz=5.5511151231257827021e-17 -1.1102230246251565404e-16 -0.19189583333333348758 rpy=2.5464045949721037905e-16 -3.8499906812161220182e-16 -3.141592653589793116 -> xyz=4.1633363423443370266e-17 -2.2204460492503130808e-16 -0.16775000000000006573 rpy=2.215784695846231927e-16 -1.1515570310408801353e-15 -3.1415926535897926719
- joint fermeture1_A_frame: origin xyz=1.3877787807814456755e-17 -5.5511151231257827021e-17 -0.025000000000000160982 rpy=-1.8744017465649457593e-18 -9.818041624348521577e-17 -2.79836129840733741e-20 -> xyz=0 -5.5511151231257827021e-17 -0.02200000000000001954 rpy=-3.959506825411487895e-17 -7.4680728089459370449e-16 -1.5846631400359783918e-15; parent piston_4 -> piston_6
- joint fermeture1_B_frame: origin xyz=-8.3266726846886740532e-17 -5.5511151231257827021e-17 -0.025000000000000244249 rpy=-3.141592653589793116 -8.7685925630935976107e-17 2.9906032515748721767e-17 -> xyz=5.5511151231257827021e-17 -2.7755575615628913511e-17 -0.021999999999999964029 rpy=3.1415926535897917837 -7.7655014458189670937e-17 -2.0416603488612588362e-15
- joint fermeture2_A_frame: origin xyz=-6.9388939039072283776e-18 -5.5511151231257827021e-17 -0.025000000000000105471 rpy=1.7473559706539229754e-22 -5.5001239547193146538e-21 1.6842726119609899759e-24 -> xyz=5.5511151231257827021e-17 0 -0.021999999999999936273 rpy=4.9690715383031197353e-17 4.2603243868850291555e-16 -5.3263942368229908787e-16; parent piston_5 -> piston_7
- joint fermeture2_B_frame: origin xyz=1.1102230246251565404e-16 2.7755575615628913511e-17 -0.025000000000000133227 rpy=-3.141592653589793116 3.1456406373773374106e-16 -5.3319186701923333256e-17 -> xyz=2.7755575615628913511e-17 8.3266726846886740532e-17 -0.022000000000000186073 rpy=3.1415926535897926719 -5.2479628515099482691e-16 -1.3723223920406849876e-17
- joint fermeture3_A_frame: origin xyz=0 -5.5511151231257827021e-17 -0.025000000000000216493 rpy=-3.141592653589793116 -1.4924298254456226231e-19 -4.5162089082963286946e-24 -> xyz=-6.9388939039072283776e-18 0 -0.021999999999999853006 rpy=3.1415926535897926719 1.293306172054732989e-15 -4.6717186998541594878e-16; parent piston_7 -> piston_4
- joint fermeture3_B_frame: origin xyz=-1.3877787807814456755e-17 2.7755575615628913511e-17 -0.025000000000000133227 rpy=7.7095856618526664724e-20 -2.8590462254934253294e-20 1.8588697243342543712e-18 -> xyz=-1.3877787807814456755e-17 -2.7755575615628913511e-17 -0.021999999999999964029 rpy=-3.2790004170572019291e-17 -4.1488573318750657904e-16 -9.26667881393621338e-17
- joint fermeture4_A_frame: origin xyz=0 8.3266726846886740532e-17 -0.025000000000000077716 rpy=-3.141592653589793116 -1.4924298254456226231e-19 -4.5162089082963286946e-24 -> xyz=6.9388939039072283776e-18 2.7755575615628913511e-17 -0.02200000000000001954 rpy=-3.141592653589793116 1.2349141206114597266e-15 -8.455101107506878145e-16; parent piston_8 -> piston_5
- joint fermeture4_B_frame: origin xyz=0 -2.7755575615628913511e-17 -0.025000000000000022204 rpy=1.1160994889302602654e-18 6.2394804750431383568e-20 1.1774112289867942571e-17 -> xyz=-2.2204460492503130808e-16 2.498001805406602216e-16 -0.022000000000000158318 rpy=3.1902612722872356481e-17 -2.8778139619308739268e-16 -2.5319202630018849146e-17
- joint fermeture5_A_frame: origin xyz=-6.9388939039072283776e-18 0 -0.025000000000000077716 rpy=0 -0 0 -> xyz=-6.2450045135165055399e-17 -1.6653345369377348106e-16 -0.022000000000000508732 rpy=6.1488129178166477185e-17 3.0252467436341876234e-16 -7.7795934687865175359e-17
- joint fermeture5_B_frame: origin xyz=-8.3266726846886740532e-17 -2.7755575615628913511e-17 -0.025000000000000105471 rpy=3.141592653589793116 3.025978467155636249e-28 -1.570796326794896558 -> xyz=0 -6.9388939039072283776e-18 -0.022000000000000196482 rpy=3.141592653589793116 1.0467333922877013405e-16 -1.570796326794896558
- joint fermeture6_A_frame: origin xyz=-6.9388939039072283776e-18 -1.6653345369377348106e-16 -0.28249999999999997335 rpy=-4.2029392900949747559e-17 -7.4606014470714686977e-18 -1.570796326794896558 -> xyz=4.1633363423443370266e-17 0 -0.27950000000000013722 rpy=-1.1991301870057867169e-15 -5.853160761014184723e-16 -1.5707963267948972241; parent piston_6 -> piston_8
- joint fermeture6_B_frame: origin xyz=-3.6082248300317587564e-16 1.6653345369377348106e-16 -0.025000000000000133227 rpy=-3.141592653589793116 1.1119874650498309646e-21 3.141592653589793116 -> xyz=0 1.3877787807814456755e-17 -0.022000000000000130562 rpy=3.1415926535897913396 -1.5085411047121220284e-15 3.1415926535897922278
- joint fermeture7_A_frame: origin xyz=-2.7755575615628913511e-17 -3.0531133177191804862e-16 -0.20762500000000022604 rpy=3.1415926535897846783 2.3079233611404340129e-17 -1.570796326794896558 -> xyz=0 1.1102230246251565404e-16 -0.18149999999999993916 rpy=3.141592653589793116 -4.7296854721327377417e-17 -1.570796326794896336; parent rode_foot -> part_19_2
- joint fermeture7_B_frame: origin xyz=4.1633363423443370266e-17 -3.0531133177191804862e-16 -0.20762499999999989297 rpy=4.7657994470008846293e-18 1.6442732956008238335e-17 -3.141592653589793116 -> xyz=-1.0581813203458523276e-16 4.4408920985006261617e-16 -0.18149999999999999467 rpy=-1.3951262331068545128e-16 1.4509398861626273799e-16 3.141592653589793116; parent rode_foot_4 -> part_19_5
- joint fermeture8_A_frame: origin xyz=-1.3877787807814456755e-17 -4.4408920985006261617e-16 -0.20762499999999994849 rpy=-2.9697957125138915857e-16 -4.8836916697961571375e-16 3.1415926535897926719 -> xyz=-3.4694469519536141888e-17 -1.1102230246251565404e-16 -0.18149999999999988365 rpy=1.5201522409519212166e-16 1.085313861270160621e-16 -3.141592653589793116; parent rode_foot_3 -> part_19_4
- joint fermeture8_B_frame: origin xyz=-2.7755575615628913511e-17 1.1102230246251565404e-16 -0.20762500000000005951 rpy=3.141592653589793116 4.8299363385392145085e-17 3.5495078826400279975e-19 -> xyz=-6.9388939039072283776e-18 1.6653345369377348106e-16 -0.18150000000000005018 rpy=3.1415926535897846783 -1.0140744846491861695e-15 -1.1625422325305371465e-15; parent rode_foot_2 -> part_19_3
- joint fermeture9_A_frame: origin xyz=0 -3.3306690738754696213e-16 -0.19189583333333326554 rpy=6.9071019648092707407e-18 2.6624167757425087404e-17 -3.141592653589793116 -> xyz=0 -2.7755575615628913511e-16 -0.1677499999999999547 rpy=-1.1523283906495666322e-15 -9.4536328633458138758e-17 3.141592653589793116
- joint fermeture9_B_frame: origin xyz=0 1.1102230246251565404e-16 -0.19189583333333337656 rpy=3.141592653589793116 -1.6721638379069471494e-17 3.075854684320635955e-18 -> xyz=-1.3877787807814456755e-17 -1.1102230246251565404e-16 -0.16775000000000006573 rpy=3.1415926535897922278 -3.067931197502387186e-17 1.1955958917632822073e-17
- joint free_attache_moeur_hanche_1: origin xyz=0.012499999999999990286 -0.0424687499999999718 -0.088083333333333277415 rpy=1.570796326794896558 0.0047435069561565304519 -1.570796326794896336 -> xyz=0.012500000000000042327 -0.037125000000000019096 -0.076999999999999638178 rpy=1.57079632679489678 0.14902323053831087463 -1.5707963267948958919
- joint free_attache_moeur_hanche_2: origin xyz=0.11962499999999837152 -0.24904166666666668895 2.2204460492503130808e-16 rpy=0 -1.5429430116984873749e-15 0 -> xyz=-0.10299999999999835676 0.24349999999999996647 1.1102230246251565404e-16 rpy=1.2301416552510086425e-15 1.6805779747991881159e-15 3.1236367382145302507
- joint free_attache_moeur_hanche_3: origin xyz=0.012500000000000011102 0.042468750000000055067 -0.088083333333333485582 rpy=1.570796326794896558 0.0047908213534053481833 -1.57079632679489678 -> xyz=0.012499999999999993755 0.03712499999999999134 -0.07700000000000019329 rpy=1.570796326794896558 0.054244509264703762164 -1.5707963267948950037
- joint free_attache_moeur_hanchexy: origin xyz=-5.5511151231257827021e-17 3.1918911957973250537e-16 -0.062916666666666662411 rpy=-1.570796326794672737 -1.5705013744383484742 1.5707963267936437823 -> xyz=2.7755575615628913511e-17 1.1102230246251565404e-16 -0.055000000000000055789 rpy=1.5707963267948945596 -1.4670604085028031704 -1.570796326794886566
- joint free_attache_moeur_hanchexy2: origin xyz=-8.3266726846886740532e-17 -1.3877787807814456755e-16 -0.062916666666666676289 rpy=-1.5707963267950315611 -1.5704936563091338453 1.5707963267928437556 -> xyz=5.5511151231257827021e-17 0 -0.054999999999999972522 rpy=-1.570796326794896558 -1.2050105151969217054 1.570796326794896336
- joint free_cardan_xhips: origin xyz=7.4999999999936228789e-05 7.2164496600635175128e-16 -7.5000000000697772395e-05 rpy=1.5707963267932967266 1.5702141424144824278 -1.570796326796419784 -> xyz=6.5999999999927227989e-05 -8.3266726846886740532e-17 -6.5999999999986208588e-05 rpy=-1.570796326794896558 1.3226194741257213394 1.5707963267948958919
- joint free_cardans_yhips: origin xyz=9.5409791178724390193e-18 -2.7755575615628913511e-17 -0.18875000000000002887 rpy=-1.57079632679489678 -0.00013745695438837276787 1.570796326794896558 -> xyz=6.9388939039072283776e-18 2.7755575615628913511e-17 -0.16500000000000006328 rpy=-1.570796326794896558 0.050365505582155675746 1.570796326794896336
- joint free_cheville_cardanx: origin xyz=7.4999999999825206487e-05 -2.2204460492503130808e-16 -7.5000000000002365122e-05 rpy=-1.570796326794896558 -1.0283708790559382695 1.570796326794896558 -> xyz=6.6000000000010494716e-05 1.1102230246251565404e-16 -6.6000000000010494716e-05 rpy=-1.570796326794896558 -1.3771163353918778327 1.5707963267949180963
- joint free_cheville_cardany: origin xyz=-0.16980000000000278204 0.34604166666666646979 -1.1102230246251565404e-16 rpy=-1.5707963267942939289 1.5706585553043288517 -1.5707963267950366681 -> xyz=-0.14843400000000434025 0.3024999999999998801 -5.5511151231257827021e-17 rpy=-1.5707963267948972241 1.5098726879342334595 -1.5707963267948736874
- joint free_genoux: origin xyz=0.17616666666662503249 -0.49075000000001500755 -0.081791666666666845709 rpy=3.141592653589793116 -1.2407226412650767997e-16 -0.00058875972722544967809 -> xyz=0.15399999999994401501 -0.42900000000002025402 -0.071500000000000035749 rpy=-3.1415926535897908956 1.1346434103290295556e-15 0.37642875273344827969
- joint free_renvois_hanche1: origin xyz=0.072354166666666039354 -0.053479166666666105856 -0.13527083333333353443 rpy=-8.54568753867082763e-17 -1.8407509512760167408e-16 0.43838119428272348532 -> xyz=-0.00046813081423434377282 -0.046749999999999486411 -0.11825000000000021605 rpy=3.1245916262671814483e-15 1.9517356246487605074e-15 0.31584837188634162786
- joint free_renvois_hanche2: origin xyz=0.072354166666667982244 -0.05347916666666752139 -0.028312500000000073719 rpy=3.141592653589793116 1.1335268030418274217e-15 0.40020166506191917621 -> xyz=-0.00046813081423434377282 -0.046749999999999625189 -0.024750000000000216271 rpy=-3.141592653589788231 6.5214264370522395898e-15 0.24765175442514256177
- joint free_triangle1_tibias: origin xyz=0.13841666666666663232 -0.47187499999999993339 -0.044041666666666784424 rpy=-3.141592653589793116 -1.3748255421293126449e-16 -0.066056290258646024882 -> xyz=0.1209999999999997744 -0.41250000000000008882 -0.038499999999999950928 rpy=-3.1415926535897917837 6.7309008105477207493e-15 -0.044053173370024609201
- joint free_triangle2_tibias: origin xyz=0.13841666666666668783 -0.47187499999999993339 -0.11954166666666668495 rpy=-1.8461492555022878416e-18 -1.0252669703201268269e-16 -0.10263776941217567229 -> xyz=0.12099999999999982991 -0.41250000000000019984 -0.10450000000000000955 rpy=8.8819479798667695408e-16 6.5393392438603125484e-15 -0.0019752092148057637938
- joint free_zhips: origin xyz=-0.012499999999999986816 -0.20499999999999996003 -0.0049999999999998934186 rpy=-1.4726037963295123608e-16 1.5370811015985778338e-15 3.0459941681722826345 -> xyz=0.012499999999999998959 0.20500000000000007105 -0.0050000000000000044409 rpy=3.9196334302860388858e-19 -2.3551738862908776961e-17 0.066174176975497225883
- joint mot_cheville1: child piston_5 -> piston_7; origin xyz=1.3877787807814456755e-17 -1.3877787807814456755e-16 -4.1245097658793028472e-05 rpy=3.141592653589793116 5.6902940387883940848e-17 -3.141592653589793116 -> xyz=1.3877787807814456755e-17 -8.3266726846886740532e-17 -0.0018968975253284559024 rpy=3.141592653589793116 -5.0324302259697873069e-16 3.1415926535897908956
- joint mot_cheville2: child piston_4 -> piston_6; origin xyz=6.2450045135165055399e-17 -2.2204460492503130808e-16 -2.9548398438994372128e-05 rpy=-3.141592653589793116 -1.2075888392074055418e-16 3.141592653589793116 -> xyz=0 0 0.0040954289115288644574 rpy=-3.1415926535897917837 -3.1962866481529558786e-15 -3.1415926535897922278
- joint mot_hanchexy1: origin xyz=5.5511151231257827021e-17 -0.03147530555841833444 8.3266726846886740532e-17 rpy=-1.570796326794896558 -4.8539988437297803109e-17 3.2508222489336867815e-16 -> xyz=-2.7755575615628913511e-17 -0.057345015123782927535 -8.3266726846886740532e-17 rpy=-1.57079632679489678 -1.0429752318537573658e-15 1.4296832532537950495e-15
- joint mot_hanchexy2: origin xyz=4.1633363423443370266e-17 -0.031475761426423623512 0 rpy=-1.570796326794896558 -4.0842560888460044134e-16 3.7225087496077564125e-16 -> xyz=5.5511151231257827021e-17 -0.044774431464078667808 8.3266726846886740532e-17 rpy=-1.570796326794896558 2.0664159541542064226e-17 2.4647545633750977575e-17
- joint mot_hanchez: origin xyz=2.7755575615628913511e-17 -1.4571677198205179593e-16 -0.062916666666666648533 rpy=0 -0 -1.570796326794896558 -> xyz=2.498001805406602216e-16 6.6613381477509392425e-16 -0.072355931990307195689 rpy=1.5538161385153811095e-15 -5.3149376727347829173e-16 -1.5707963267948990005
- joint to_rotule_free_attache2_moeur_hanchez: origin xyz=1.7078352620991665844e-15 0.044041666666666673402 -0.053479166666666723418 rpy=1.570796326794896558 -1.9832067293240475674e-17 1.570796326794896558 -> xyz=1.8075818619678329924e-15 0.038500000000000006439 -0.046749999999999958256 rpy=1.570796326794896558 7.0078510672975474039e-15 1.570796326794896558
- joint to_rotule_free_attache_genoux: origin xyz=-0.044041666666667284025 0.050333333333332563875 5.5511151231257827021e-17 rpy=-1.57079632679489678 0.026729912583035628226 -8.6038674056888522762e-19 -> xyz=-0.0384999999999999995 0.04400000000000003908 -1.1102230246251565404e-16 rpy=-1.5707963267948972241 -1.4520889402669923118 3.1609121641998322792e-15
- joint to_rotule_free_attache_hanche1: origin xyz=-0.13212499999999993694 -0.037750000000000172307 5.5511151231257827021e-17 rpy=-1.57079632679489678 -0.094042986969348249526 -3.1415926535897926719 -> xyz=-0.054999999999999944766 -0.033000000000000084821 0 rpy=1.5707963267948970021 1.4166502888720968745 -1.6844589433685216916e-14
- joint to_rotule_free_attache_hanche2: origin xyz=-0.13212499999999971489 0.037749999999999950262 -2.7755575615628913511e-17 rpy=1.570796326794896558 0.092185476461817641991 3.141592653589793116 -> xyz=-0.054999999999999951705 0.033000000000000306866 5.5511151231257827021e-17 rpy=-1.570796326794896558 0.39151326041874018324 2.434576526324631611e-15
- joint to_rotule_free_attache_moeur_hanche_z: origin xyz=-1.3877787807814456755e-17 0 -0.058479166666666637653 rpy=1.570796326794896558 -0 1.570796326794896558 -> xyz=-1.3877787807814456755e-17 -5.5511151231257827021e-17 -0.051749999999999997391 rpy=1.5707963267948970021 0.017795322282523534652 1.5707963267948972241
- joint to_rotule_free_foot1: origin xyz=-0.0629166666666667318 -0.012583333333333390769 0.044041666666666368091 rpy=1.570796326794896558 0.081892649261537886485 -3.141592653589793116 -> xyz=-0.054999999999999993339 -0.01100000000000000977 0.038499999999999978684 rpy=-1.570796326794896558 0.02245377174158168232 -1.0028453061676132335e-14
- joint to_rotule_free_goot2: origin xyz=-0.062916666666666620777 -0.012583333333333168724 -0.044041666666666950958 rpy=1.570796326794896558 0.081892649261537886485 -3.141592653589793116 -> xyz=-0.055000000000000014155 -0.010999999999999898748 -0.038500000000000200728 rpy=-1.570796326794896558 0.022453771741563686298 -1.8953531735976104769e-14
- joint to_rotule_free_hanche_attache1: child piston_7 -> piston_4; origin xyz=0.069208333333333316162 -1.6653345369377348106e-16 -0.04404166666666681218 rpy=-1.57079632679489678 -0.095598525430158579064 3.1415926535897926719 -> xyz=0.060499999999999859446 -1.1102230246251565404e-16 -0.038500000000000006439 rpy=-1.570796326794896558 0.3088492434818621013 -3.141592653589793116
- joint to_rotule_free_hanche_attache2: child piston_8 -> piston_5; origin xyz=0.069208333333333357795 0 0.044041666666666673402 rpy=-1.57079632679489678 -0.095598525430158579064 3.1415926535897926719 -> xyz=0.060499999999999845568 -1.6653345369377348106e-16 0.038500000000000006439 rpy=-1.570796326794896558 0.5119562997150467476 -3.141592653589793116
- joint to_rotule_free_renvois_hanche3: child rode_foot_3 -> part_19_4; origin xyz=-0.10695833333333404358 -0.062916666666667009356 -1.6653345369377348106e-16 rpy=-1.57079632679489678 0.09404298696934784707 -4.8159767687053810446e-16 -> xyz=-0.033000000000000015432 -0.066000000000000197398 1.1102230246251565404e-16 rpy=1.57079632679489678 -0.14846352767658158034 3.1415926535897922278
- joint to_rotule_free_renvois_hanche4: child rode_foot_4 -> part_19_5; origin xyz=-0.1069583333333340297 0.062916666666667064867 1.1102230246251565404e-16 rpy=1.570796326794896558 -0.092185476461817753013 2.6802825518558815111e-17 -> xyz=-0.032999999999999980738 0.066000000000000030864 -2.7755575615628913511e-17 rpy=-1.570796326794896558 0.14330741373895086732 -3.141592653589793116
- joint to_rotule_free_triangle1: origin xyz=-0.068058330216350965136 0.012564119186792344074 -0.012583333333333557302 rpy=-1.57079632679489678 0.16864244180508916604 3.6078898931567104179e-17 -> xyz=-0.059494699261975619864 0.010983203527526907983 -0.010999999999999787725 rpy=1.570796326794896558 0.21334546122709105442 3.1415926535897895633
- joint to_rotule_free_triangle2: origin xyz=-0.068058330216350965136 -0.012564119186792344074 -0.012583333333333057702 rpy=1.570796326794896558 -0.095385008856607569894 -2.6902869908268245684e-16 -> xyz=-0.059494699261975592108 -0.010983203527526907983 -0.01100000000000000977 rpy=-1.570796326794896558 -0.093507593570657396298 -3.1415926535897789051
- joint to_rotule_free_triangle4: child rode_foot_2 -> part_19_3; origin xyz=-0.041015624251386273436 -0.047709805194671606188 -0.047187499999999826805 rpy=-1.57079632679489678 -0.095087883447032894857 3.141592653589793116 -> xyz=-0.035854717888628179212 -0.041706584673487867576 -0.041249999999999786837 rpy=1.57079632679489678 -0.55222488425847393589 -2.6036272167158010406e-15
- joint to_rotule_free_trianle3: child rode_foot -> part_19_2; origin xyz=-0.041015624251385912613 0.047709805194671939255 -0.047187500000000021094 rpy=1.5707963267948961139 -1.4687456221646373322 3.141592653589658557 -> xyz=-0.035854717888627957167 0.041706584673487867576 -0.041250000000000008882 rpy=-1.5707963267949172081 1.56644625480537103 1.0966850609177858196e-13
