Commit message: Adding new robot with two legs

File: robots/robot_marcheur_two_leg/robot.urdf (robot description, URDF)
Before this commit: robot onshape, 46 links, 44 joints
Joints:
- added joint to_rotule_servo_gauche_2: type revolute, parent molet_4, child toe_b_1/2_4, origin xyz=2.2204460492503130808e-16 0.057000000000000494715 0.0025000000000004185541 rpy=-1.570796326794896558 -1.866329740155221443e-16 1.5707963267948970021, axis 0 0 1, limit effort=1 velocity=20
- joint to_rotule_servo_gauche_1: child toe_b_1/2_4 -> toe_b_2/2_4; origin xyz=2.2204460492503130808e-16 0.057000000000000494715 0.0025000000000004185541 rpy=-1.570796326794896558 -1.866329740155221443e-16 1.5707963267948970021 -> xyz=-5.5511151231257827021e-17 0.057000000000000050626 0.0025000000000000022204 rpy=-1.57079632679489678 -6.1989581036318994383e-14 -1.570796326794896558; parent molet_4 -> molet_3
