Commit message: Update robots

File: robots/disney_like/robot.urdf (robot description, URDF)
Before this commit: robot onshape, 26 links, 25 joints
Links:
- link bloc_moteur: mass 11.246937103837286287 -> 11.246937103837288063
- link bloc_moteur2: mass 11.246937103837179706 -> 11.246937103837177929
- link tibias_mirror2: mass 0.50944821011060748006 -> 0.50944821011060736904
