Commit message: Update robots

File: robots/kangaroo_like/robot.urdf (robot description, URDF)
Before this commit: robot onshape, 67 links, 66 joints
Links:
- removed link part_18
- removed link part_19
- removed link part_19_2
- removed link part_19_3
- removed link part_19_4
- removed link part_19_5
- removed link part_19_6
- removed link renvois_hanche
- removed link renvois_hanche_2
- removed link rode_tarsus
- removed link rode_tarsus_2
- removed link rode_tarsus_3
- removed link rode_tarsus_4
- removed link tarsus
- removed link tibias
- added link fermeture11_A, mass 1e-9
- added link fermeture11_B, mass 1e-9
- added link part_1, mass 0.48864348852726857686; collision mesh filename=package:///part_1.stl; visual mesh filename=package:///part_1.stl
- added link part_2, mass 0.7961294500674355179; collision mesh filename=package:///part_2.stl; visual mesh filename=package:///part_2.stl
- added link part_3, mass 0.40426961787931336989; collision mesh filename=package:///part_3.stl; visual mesh filename=package:///part_3.stl
- added link part_4, mass 0.022622071159599056733; collision mesh filename=package:///part_4.stl; visual mesh filename=package:///part_4.stl
- added link part_5, mass 0.022214201653533428155; collision mesh filename=package:///part_5.stl; visual mesh filename=package:///part_5.stl
- added link part_6, mass 0.067104419080678087695; collision mesh filename=package:///part_6.stl; visual mesh filename=package:///part_6.stl
- added link part_7, mass 0.062831853071795965016; collision mesh filename=package:///part_7.stl; visual mesh filename=package:///part_7.stl
- added link part_7_2, mass 0.062831853071795965016; collision mesh filename=package:///part_7.stl; visual mesh filename=package:///part_7.stl
- added link part_7_3, mass 0.062831853071795965016; collision mesh filename=package:///part_7.stl; visual mesh filename=package:///part_7.stl
- added link part_7_4, mass 0.062831853071795965016; collision mesh filename=package:///part_7.stl; visual mesh filename=package:///part_7.stl
- added link part_8, mass 0.012408180777254541535; collision mesh filename=package:///part_8.stl; visual mesh filename=package:///part_8.stl
- added link part_9, mass 0.012408180777254539801; collision mesh filename=package:///part_9.stl; visual mesh filename=package:///part_9.stl
- link attache_hanche: mass 0.012829478999097282399 -> 0.01282947899909727546
- link cardan_foot: mass 0.0064135211594024193679 -> 0.0064135211594024202353
- link cardan_foot_2: mass 0.0064135211594024193679 -> 0.0064135211594024202353
- link cardan_hache: mass 0.015608633111865832799 -> 0.015608633111865791165
- link cardan_hache_2: mass 0.015608633111865832799 -> 0.015608633111865791165
- link hanche: mass 0.14908820646980575075 -> 0.1490882064698049736
- link hanche_batis: mass 1.5865591647149874799 -> 1.5865591647149870358
- link moteur_hanche1: mass 0.17794962537636818678 -> 0.17794962537636810351
- link moteur_hanche1_2: mass 0.17794962537636818678 -> 0.17794962537636810351
- link motteur_rotation: mass 0.19339251676417071324 -> 0.19339251676417060222
- link motteur_rotation_2: mass 0.19339251676417071324 -> 0.19339251676417060222
- link motteur_rotation_3: mass 0.19339251676417071324 -> 0.19339251676417060222
- link motteur_rotation_4: mass 0.19339251676417071324 -> 0.19339251676417060222
- link renvois_cheville: mass 0.074310321213956573305 -> 0.074310321213953561825
- link renvois_cheville_2: mass 0.074310320490076631206 -> 0.074310320490072731547
Joints:
- removed joint ferme_genoux
- removed joint free_cardan_xhips
- removed joint free_cheville_cardany
- removed joint free_genoux
- removed joint free_renvois_hanche1
- removed joint free_renvois_hanche2
- removed joint free_triangle1_tibias
- removed joint free_triangle2_tibias
- removed joint moteur_genoux
- removed joint to_rotule_free_attache_genoux
- removed joint to_rotule_free_attache_hanche1
- removed joint to_rotule_free_attache_hanche2
- removed joint to_rotule_free_foot1
- removed joint to_rotule_free_goot2
- removed joint to_rotule_free_hanche_attache1
- removed joint to_rotule_free_hanche_attache2
- removed joint to_rotule_free_renvois_hanche3
- removed joint to_rotule_free_renvois_hanche4
- removed joint to_rotule_free_triangle1
- removed joint to_rotule_free_triangle2
- removed joint to_rotule_free_triangle4
- removed joint to_rotule_free_trianle3
- removed joint to_rotule_genoux
- removed joint to_rotule_genoux2
- removed joint to_rotule_moeur_cheville_1
- removed joint to_rotule_moeur_cheville_2
- removed joint to_rotule_test
- added joint 4barres_genoux: type revolute, parent part_2, child part_4, origin xyz=0.04604763173374630536 -0.01948372684352375761 2.0539125955565395998e-15 rpy=3.141592653589793116 2.0222313221252327283e-16 -1.2672660179279369164, axis 0 0 1, limit effort=1 velocity=20
- added joint cardans_foot_haut: type revolute, parent part_3, child cardan_foot_2, origin xyz=0.21747050071614926203 -0.33571800862966438839 -1.1102230246251565404e-16 rpy=-1.5707963267948958919 -1.4835298641951772947 1.5707963267949329733, axis 0 0 1, limit effort=1 velocity=20
- added joint fermeture11_A_frame: type fixed, parent foot, child fermeture11_A, origin xyz=-0.054999999999999993339 -0.01100000000000000977 -0.038499999999999978684 rpy=1.570796326794896558 4.5855729041023846865e-17 -1.570796326794896336, axis 0 0 0
- added joint fermeture11_B_frame: type fixed, parent part_7_2, child fermeture11_B, origin xyz=-1.1102230246251565404e-16 -2.7755575615628913511e-17 -0.4000000000000000222 rpy=3.1415926535897891192 -3.9070079812037976252e-16 1.570796326794896558, axis 0 0 0
- added joint frame_moeur_genoux: type revolute, parent part_2, child motteur_rotation, origin xyz=-0.061655078133537426222 -0.018724201373191751152 4.2974512837190559367e-12 rpy=-1.570796326794896558 1.2771385194773072769 -0.60601731071218312152, axis 0 0 1, limit effort=1 velocity=20
- added joint frame_moeur_pied1: type revolute, parent part_1, child motteur_rotation_2, origin xyz=0.054086706326755044916 0.014047405294960735311 -0.11824999999999977196 rpy=-1.57079632679489678 0.73498046737731359546 0.28589337779932527672, axis 0 0 1, limit effort=1 velocity=20
- added joint frame_moeur_pied2: type revolute, parent part_1, child motteur_rotation_3, origin xyz=0.054086706326755183694 0.014047405294960735311 -0.024749999999999966471 rpy=1.570796326794896558 -0.17956569756706253216 -2.8556992757904753333, axis 0 0 1, limit effort=1 velocity=20
- added joint genoux_bas: type revolute, parent part_2, child part_3, origin xyz=-0.21747050071615248168 -0.33571800862966205692 2.0539125955565395998e-15 rpy=2.0331986601504280136e-17 3.4472742402185754406e-17 0.89630439304597653294, axis 0 0 1, limit effort=1 velocity=20
- added joint genoux_haut: type revolute, parent part_1, child part_2, origin xyz=-1.4918621893400541012e-16 0.046752000000001070479 -0.071499999999995539346 rpy=-3.1415926535897851224 -4.177940397166871663e-15 0.55885062184425926546, axis 0 0 1, limit effort=1 velocity=20
- added joint hanche_bas: type revolute, parent cardan_foot, child part_1, origin xyz=6.600000000017702817e-05 -2.7755575615628913511e-17 -6.5999999999974065523e-05 rpy=-1.5707963267949276442 -1.531769381031934163 -1.570796326794891451, axis 0 0 1, limit effort=1 velocity=20
- added joint mot_genoux: type prismatic, parent motteur_rotation, child piston_3, origin xyz=-2.7755575615628913511e-17 -2.7755575615628913511e-17 -0.015328902570172664444 rpy=3.141592653589793116 1.4125255666875108451e-15 -4.0832512369930491999e-15, axis 0 0 1, limit effort=1 velocity=20
- added joint renvois_genoux_1: type revolute, parent part_2, child renvois_cheville_2, origin xyz=-0.21747050071615156575 -0.33571800862966272305 0.010000000000000064393 rpy=3.1415926535897926719 1.6415409336565314963e-15 2.9857006913335375486, axis 0 0 1, limit effort=1 velocity=20
- added joint renvois_genoux_2: type revolute, parent part_2, child renvois_cheville, origin xyz=-0.21747050071615153799 -0.33571800862966283407 -0.0099999999999999533706 rpy=3.141592653589793116 1.4899689001647264157e-15 3.0109455540470038137, axis 0 0 1, limit effort=1 velocity=20
- added joint renvois_hanche_1: type revolute, parent part_1, child part_8, origin xyz=-7.9797279894933126343e-17 0.046751999999999960256 -0.087999999999999994893 rpy=6.1903321544647517205e-15 -7.8041542465741715794e-15 1.1519622146724590728, axis 0 0 1, limit effort=1 velocity=20
- added joint renvois_hanche_2: type revolute, parent part_1, child part_9, origin xyz=-6.0715321659188248304e-17 0.046752000000000043523 -0.055000000000000076605 rpy=-3.1415926535897864547 -8.0378052466654680077e-15 1.1213209623233275636, axis 0 0 1, limit effort=1 velocity=20
- added joint to_rotule_4barres: type revolute, parent part_4, child part_5, origin xyz=0.0194837268435249511 -0.046047631733748373151 0 rpy=-1.57079632679489678 0.033617431841821705796 -1.5707963267948954478, axis 0 0 1, limit effort=1 velocity=20
- added joint to_rotule_barres_tibias: type revolute, parent part_3, child part_6, origin xyz=0.038967453687049569133 -0.092095263467498161836 -5.5511151231257827021e-17 rpy=-1.57079632679489678 -1.7877918082017555513e-15 1.5707963267948970021, axis 0 0 1, limit effort=1 velocity=20
- added joint to_rotule_hanche_bas1: type revolute, parent part_1, child piston, origin xyz=-0.060500000000000032918 -1.1102230246251565404e-16 -0.038500000000000034195 rpy=1.57079632679489678 -0.083114644637937176719 -3.1415926535897846783, axis 0 0 1, limit effort=1 velocity=20
- added joint to_rotule_hanche_bas2: type revolute, parent part_1, child piston_2, origin xyz=-0.060500000000000088429 8.3266726846886740532e-17 0.038499999999999978684 rpy=-1.57079632679489678 0.09010970645432067605 -5.2356120935469576439e-14, axis 0 0 1, limit effort=1 velocity=20
- added joint to_rotule_moeur_action_genoux: type revolute, parent part_1, child piston_6, origin xyz=-0.013749999999999944558 0.002500000000000029976 -0.071999999999999980682 rpy=-1.57079632679489678 -0.99860729712136486746 -1.5707963267949038855, axis 0 0 1, limit effort=1 velocity=20
- added joint to_rotule_renvois_hanche3: type revolute, parent part_8, child part_7_3, origin xyz=0.041074543378118916204 0.036577067764912929437 -0.0050000000000000044409 rpy=-1.570796326794896558 0.088927611054570185334 -3.1415926535897922278, axis 0 0 1, limit effort=1 velocity=20
- added joint to_rotule_renvois_hanche4: type revolute, parent part_9, child part_7_4, origin xyz=0.041074543378118888448 -0.036577067764912998826 -0.005000000000000059952 rpy=1.5707963267948972241 1.4581066266007882692 3.1415926535897522598, axis 0 0 1, limit effort=1 velocity=20
- added joint to_rotule_renvois_hanche_moeur1: type revolute, parent part_8, child piston_4, origin xyz=0.043531328479973763201 0.0032046566522408725941 -0.025000000000000022204 rpy=-1.5707963267948981123 -1.2175171882697095604 -1.4253980587447095076e-14, axis 0 0 1, limit effort=1 velocity=20
- added joint to_rotule_renvois_hanche_moeur2: type revolute, parent part_9, child piston_5, origin xyz=0.043531328479973624423 -0.0032046566522409697386 -0.025000000000000022204 rpy=-1.570796326794896336 -1.3137217724347112213 -3.1415926535897789051, axis 0 0 1, limit effort=1 velocity=20
- added joint to_rotule_renvois_pied1: type revolute, parent renvois_cheville, child part_7_2, origin xyz=-0.059494699261975425575 0.01098320352752724105 0.022000000000000102807 rpy=1.570796326794896558 1.9627544666669624505e-30 1.57079632679489678, axis 0 0 1, limit effort=1 velocity=20
- added joint to_rotule_renvois_pied2: type revolute, parent renvois_cheville_2, child part_7, origin xyz=-0.059494699261975605986 0.010983203527527130028 -0.021999999999999908518 rpy=-1.57079632679489678 -2.0407188599509725859e-30 -1.57079632679489678, axis 0 0 1, limit effort=1 velocity=20
- joint bout_pied_frame: origin xyz=0.012016949221079924193 0.038500000000000089706 6.8117394502742456552e-09 rpy=1.570796326794896558 -8.8759669262812707343e-18 -1.5746176066600222494e-17 -> xyz=0.01201694922107987562 0.038499999999999923173 6.8117393670075188084e-09 rpy=1.5707963267948972241 5.1168880392112031481e-18 1.430103156860997354e-15
- joint centre_hanche_frame: origin xyz=-0.004747469922900492828 0.288611431583448097 -0.17250000000000004219 rpy=0 -2.5097998118986334965e-18 0 -> xyz=-0.0047474699228997607747 0.28861143158345337056 -0.17250000000000290101 rpy=2.6505726415425557215e-28 -8.3196567936654447285e-16 -1.1492717312938456553e-28
- joint fermeture0_A_frame: origin xyz=-6.9388939039072283776e-18 0 -0.16775000000000006573 rpy=3.141592653589793116 2.0456812790238454299e-17 -1.6970722323022375395e-17 -> xyz=-0.05500000000000004885 -0.011000000000000065281 0.038500000000000089706 rpy=1.570796326794896558 4.5855729041023846865e-17 -1.570796326794896336; parent rode_tarsus -> foot
- joint fermeture0_B_frame: origin xyz=4.1633363423443370266e-17 -2.2204460492503130808e-16 -0.16775000000000006573 rpy=2.215784695846231927e-16 -1.1515570310408801353e-15 -3.1415926535897926719 -> xyz=-1.1102230246251565404e-16 -5.5511151231257827021e-17 -0.40000000000000007772 rpy=3.1415926535897913396 1.2983444000664012896e-15 -1.570796326794896558; parent rode_tarsus_4 -> part_7
- joint fermeture10_A_frame: origin xyz=-1.1102230246251565404e-16 2.7755575615628913511e-16 -0.18149999999999993916 rpy=3.1415926535897895633 1.1988806635353361042e-15 1.570796326794896558 -> xyz=-5.5511151231257827021e-17 5.5511151231257827021e-17 -0.4000000000000000222 rpy=1.6746929915636827556e-16 7.6910124686008864173e-16 -4.1986914796458445699e-16; parent part_19 -> part_7_3
- joint fermeture10_B_frame: origin xyz=0 0 -0.18149999999999999467 rpy=-1.0968167807709025411e-17 2.3866997684138820983e-16 -1.570796326794896336 -> xyz=-0.035854717888628928613 -0.041706584673488200643 -0.052249999999999963141 rpy=-1.57079632679489678 4.2500725161430645989e-17 -4.1960373922009253948e-16; parent part_19_6 -> renvois_cheville_2
- joint fermeture1_A_frame: origin xyz=0 -5.5511151231257827021e-17 -0.02200000000000001954 rpy=-3.959506825411487895e-17 -7.4680728089459370449e-16 -1.5846631400359783918e-15 -> xyz=-5.5511151231257827021e-17 8.3266726846886740532e-17 -0.021999999999999936273 rpy=-3.2868927901766838794e-15 5.1204923623446968973e-18 1.9524242285054774848e-16; parent piston_6 -> piston_7
- joint fermeture1_B_frame: origin xyz=5.5511151231257827021e-17 -2.7755575615628913511e-17 -0.021999999999999964029 rpy=3.1415926535897917837 -7.7655014458189670937e-17 -2.0416603488612588362e-15 -> xyz=-4.1633363423443370266e-16 2.7755575615628913511e-16 -0.021999999999999672595 rpy=-3.1415926535897904515 2.1284558966151313971e-15 -1.570796326794896336; parent piston_2 -> piston_4
- joint fermeture2_A_frame: origin xyz=5.5511151231257827021e-17 0 -0.021999999999999936273 rpy=4.9690715383031197353e-17 4.2603243868850291555e-16 -5.3263942368229908787e-16 -> xyz=0 5.5511151231257827021e-17 -0.021999999999999825251 rpy=-1.3411941716656837909e-15 3.5740894156239343174e-15 -9.5189019721563840201e-18; parent piston_7 -> piston_8
- joint fermeture2_B_frame: origin xyz=2.7755575615628913511e-17 8.3266726846886740532e-17 -0.022000000000000186073 rpy=3.1415926535897926719 -5.2479628515099482691e-16 -1.3723223920406849876e-17 -> xyz=2.7755575615628913511e-17 0 -0.021999999999999977907 rpy=3.1415926535897926719 3.2188537522304998196e-15 -1.570796326794896558; parent piston_3 -> piston_5
- joint fermeture3_A_frame: origin xyz=-6.9388939039072283776e-18 0 -0.021999999999999853006 rpy=3.1415926535897926719 1.293306172054732989e-15 -4.6717186998541594878e-16 -> xyz=1.3877787807814456755e-17 2.7755575615628913511e-17 -0.022000000000000047296 rpy=-3.141592653589793116 -9.3190864752961032569e-16 5.8795219851960389588e-17; parent piston_4 -> piston
- joint fermeture3_B_frame: origin xyz=-1.3877787807814456755e-17 -2.7755575615628913511e-17 -0.021999999999999964029 rpy=-3.2790004170572019291e-17 -4.1488573318750657904e-16 -9.26667881393621338e-17 -> xyz=-1.3877787807814456755e-17 -2.7755575615628913511e-17 -0.022000000000000005662 rpy=-3.8393612983596291192e-15 1.2937396776246885914e-16 1.6310189255223409293e-17
- joint fermeture4_A_frame: origin xyz=6.9388939039072283776e-18 2.7755575615628913511e-17 -0.02200000000000001954 rpy=-3.141592653589793116 1.2349141206114597266e-15 -8.455101107506878145e-16 -> xyz=-6.9388939039072283776e-18 -5.5511151231257827021e-17 -0.022000000000000158318 rpy=-3.1415926535897895633 -5.879482808650320173e-14 -4.752353584724499202e-18; parent piston_5 -> piston_2
- joint fermeture4_B_frame: origin xyz=-2.2204460492503130808e-16 2.498001805406602216e-16 -0.022000000000000158318 rpy=3.1902612722872356481e-17 -2.8778139619308739268e-16 -2.5319202630018849146e-17 -> xyz=0 -5.5511151231257827021e-17 -0.021999999999999880762 rpy=-5.2438558616291848205e-14 8.0236260903567770327e-15 -3.9494143193115342685e-18
- joint fermeture5_A_frame: origin xyz=-6.2450045135165055399e-17 -1.6653345369377348106e-16 -0.022000000000000508732 rpy=6.1488129178166477185e-17 3.0252467436341876234e-16 -7.7795934687865175359e-17 -> xyz=0 0 -0.021999999999999943212 rpy=4.0939474033053051719e-16 2.1380466841413257505e-16 6.2026386493102164692e-16
- joint fermeture5_B_frame: origin xyz=0 -6.9388939039072283776e-18 -0.022000000000000196482 rpy=3.141592653589793116 1.0467333922877013405e-16 -1.570796326794896558 -> xyz=-2.7755575615628913511e-17 -1.3877787807814456755e-17 -0.022000000000000054234 rpy=3.1415926535897917837 9.3675067702748754064e-17 -1.570796326794896558
- joint fermeture6_A_frame: origin xyz=4.1633363423443370266e-17 0 -0.27950000000000013722 rpy=-1.1991301870057867169e-15 -5.853160761014184723e-16 -1.5707963267948972241 -> xyz=0.038967453687049680155 -0.09209526346749669079 0 rpy=1.570796326794896558 4.0264892340170650855e-23 -1.570796326794896336; parent piston_8 -> part_4
- joint fermeture6_B_frame: origin xyz=0 1.3877787807814456755e-17 -0.022000000000000130562 rpy=3.1415926535897913396 -1.5085411047121220284e-15 3.1415926535897922278 -> xyz=0 0 -0.42719999999999996865 rpy=-3.1415926535897926719 3.4015388199230806036e-16 -3.141592653589793116; parent piston -> part_6
- joint fermeture7_A_frame: origin xyz=0 1.1102230246251565404e-16 -0.18149999999999993916 rpy=3.141592653589793116 -4.7296854721327377417e-17 -1.570796326794896336 -> xyz=2.7755575615628913511e-17 5.5511151231257827021e-17 -0.14141999999999993465 rpy=-3.141592653589793116 -2.7996380004088288758e-16 1.5135314005004021884e-16; parent part_19_2 -> part_5
- joint fermeture7_B_frame: origin xyz=-1.0581813203458523276e-16 4.4408920985006261617e-16 -0.18149999999999999467 rpy=-1.3951262331068545128e-16 1.4509398861626273799e-16 3.141592653589793116 -> xyz=0.083867056794542413356 -0.0077119035015027481705 -0.07150000000000009126 rpy=1.570796326794896558 -2.9280526622159908463e-31 1.5240432853305341472e-17; parent part_19_5 -> part_1
- joint fermeture8_A_frame: origin xyz=-3.4694469519536141888e-17 -1.1102230246251565404e-16 -0.18149999999999988365 rpy=1.5201522409519212166e-16 1.085313861270160621e-16 -3.141592653589793116 -> xyz=-2.7755575615628913511e-17 2.7755575615628913511e-17 -0.022000000000000047296 rpy=-3.141592653589793116 -6.9328037721462276608e-17 -1.570796326794896336; parent part_19_4 -> piston_3
- joint fermeture8_B_frame: origin xyz=-6.9388939039072283776e-18 1.6653345369377348106e-16 -0.18150000000000005018 rpy=3.1415926535897846783 -1.0140744846491861695e-15 -1.1625422325305371465e-15 -> xyz=0 -3.8163916471489756077e-17 -0.022000000000000064643 rpy=1.0535930861243439876e-15 -3.8516451723504327238e-16 1.5707963267948974462; parent part_19_3 -> piston_6
- joint fermeture9_A_frame: origin xyz=0 -2.7755575615628913511e-16 -0.1677499999999999547 rpy=-1.1523283906495666322e-15 -9.4536328633458138758e-17 3.141592653589793116 -> xyz=5.5511151231257827021e-17 -5.5511151231257827021e-17 -0.39999999999999991118 rpy=-2.3885598000085227952e-15 -1.1434631702908988368e-15 -1.5707963267948972241; parent rode_tarsus_3 -> part_7_4
- joint fermeture9_B_frame: origin xyz=-1.3877787807814456755e-17 -1.1102230246251565404e-16 -0.16775000000000006573 rpy=3.1415926535897922278 -3.067931197502387186e-17 1.1955958917632822073e-17 -> xyz=-0.035854717888628928613 -0.041706584673488200643 0.052250000000000074163 rpy=1.570796326794896558 1.4111985271034697919e-31 -3.1415926535897908956; parent rode_tarsus_2 -> renvois_cheville
- joint free_attache_moeur_hanche_1: origin xyz=0.012500000000000042327 -0.037125000000000019096 -0.076999999999999638178 rpy=1.57079632679489678 0.14902323053831087463 -1.5707963267948958919 -> xyz=0.012500000000000028449 -0.037124999999999797051 -0.077000000000000096145 rpy=1.57079632679489678 -0.022633356279604249783 -1.5707963267948996666
- joint free_attache_moeur_hanche_2: origin xyz=-0.10299999999999835676 0.24349999999999996647 1.1102230246251565404e-16 rpy=1.2301416552510086425e-15 1.6805779747991881159e-15 3.1236367382145302507 -> xyz=-0.10299999999999821798 0.24350000000000304734 0 rpy=-1.0047518372857614626e-14 7.4933038271172496209e-15 3.1415926535897793492
- joint free_attache_moeur_hanche_3: origin xyz=0.012499999999999993755 0.03712499999999999134 -0.07700000000000019329 rpy=1.570796326794896558 0.054244509264703762164 -1.5707963267948950037 -> xyz=0.012499999999999993755 0.037125000000000352163 -0.077000000000000623501 rpy=-1.570796326794896558 -0.020560685438658014845 1.5707963267948950037
- joint free_attache_moeur_hanchexy: origin xyz=2.7755575615628913511e-17 1.1102230246251565404e-16 -0.055000000000000055789 rpy=1.5707963267948945596 -1.4670604085028031704 -1.570796326794886566 -> xyz=0 8.3266726846886740532e-17 -0.055000000000000007216 rpy=-1.5707963267948970021 1.4483016225560627621 1.5707963267949096586
- joint free_attache_moeur_hanchexy2: origin xyz=5.5511151231257827021e-17 0 -0.054999999999999972522 rpy=-1.570796326794896558 -1.2050105151969217054 1.570796326794896336 -> xyz=-8.3266726846886740532e-17 -9.7144514654701197287e-17 -0.054999999999999951705 rpy=-1.5707963267948794606 -1.4483070518912046776 1.5707963267948805708
- joint free_cardans_yhips: origin xyz=6.9388939039072283776e-18 2.7755575615628913511e-17 -0.16500000000000006328 rpy=-1.570796326794896558 0.050365505582155675746 1.570796326794896336 -> xyz=-1.7347234759768070944e-18 0 -0.1649999999999999245 rpy=1.570796326794896558 -9.6290805123406329139e-15 -1.5707963267948992225
- joint free_cheville_cardanx: origin xyz=6.6000000000010494716e-05 1.1102230246251565404e-16 -6.6000000000010494716e-05 rpy=-1.570796326794896558 -1.3771163353918778327 1.5707963267949180963 -> xyz=6.5999999999899472414e-05 -1.1102230246251565404e-16 6.6000000000010494716e-05 rpy=-1.570796326794896558 -1.2485224054081762723 -1.5707963267948990005
- joint free_zhips: origin xyz=0.012499999999999998959 0.20500000000000007105 -0.0050000000000000044409 rpy=3.9196334302860388858e-19 -2.3551738862908776961e-17 0.066174176975497225883 -> xyz=0.012500000000000170697 0.20500000000000265232 -0.0050000000000000044409 rpy=1.0057557210906877445e-14 -7.6592250448352642693e-15 2.7755575615630239783e-16
- joint mot_cheville1: child piston_7 -> piston_8; origin xyz=1.3877787807814456755e-17 -8.3266726846886740532e-17 -0.0018968975253284559024 rpy=3.141592653589793116 -5.0324302259697873069e-16 3.1415926535897908956 -> xyz=-2.0816681711721685133e-15 5.5511151231257827021e-17 0.04053320001699314834 rpy=3.141592653589793116 2.1142323365907498637e-15 3.1415926535897922278; parent motteur_rotation_2 -> motteur_rotation_3
- joint mot_cheville2: child piston_6 -> piston_7; origin xyz=0 0 0.0040954289115288644574 rpy=-3.1415926535897917837 -3.1962866481529558786e-15 -3.1415926535897922278 -> xyz=2.2204460492503130808e-16 -8.3266726846886740532e-17 0.043273532217195209704 rpy=-3.141592653589793116 1.9076867048264111618e-14 3.1415926535897806815; parent motteur_rotation -> motteur_rotation_2
- joint mot_hanchexy1: origin xyz=-2.7755575615628913511e-17 -0.057345015123782927535 -8.3266726846886740532e-17 rpy=-1.57079632679489678 -1.0429752318537573658e-15 1.4296832532537950495e-15 -> xyz=-1.3877787807814456755e-17 -0.042153192856970334024 -3.3306690738754696213e-16 rpy=-1.5707963267949502928 -7.9443295731949990133e-15 7.187450421670799897e-15
- joint mot_hanchexy2: origin xyz=5.5511151231257827021e-17 -0.044774431464078667808 8.3266726846886740532e-17 rpy=-1.570796326794896558 2.0664159541542064226e-17 2.4647545633750977575e-17 -> xyz=-4.1633363423443370266e-17 -0.042150363629083059669 3.8857805861880478915e-16 rpy=-1.5707963267948996666 2.5427641942030839963e-15 2.1759312088804703145e-15
- joint mot_hanchez: origin xyz=2.498001805406602216e-16 6.6613381477509392425e-16 -0.072355931990307195689 rpy=1.5538161385153811095e-15 -5.3149376727347829173e-16 -1.5707963267948990005 -> xyz=-1.0547118733938987134e-15 -8.7430063189231077558e-16 -0.071500000000001451284 rpy=-2.1233015345958489363e-15 4.1282117760629273878e-17 -1.5707963267949134334
- joint to_rotule_free_attache2_moeur_hanchez: origin xyz=1.8075818619678329924e-15 0.038500000000000006439 -0.046749999999999958256 rpy=1.570796326794896558 7.0078510672975474039e-15 1.570796326794896558 -> xyz=3.2508717939805364949e-15 0.038500000000000034195 -0.046750000000000013767 rpy=1.570796326794896558 0.051824161433129206644 1.5707963267948945596
- joint to_rotule_free_attache_moeur_hanche_z: origin xyz=-1.3877787807814456755e-17 -5.5511151231257827021e-17 -0.051749999999999997391 rpy=1.5707963267948970021 0.017795322282523534652 1.5707963267948972241 -> xyz=1.3877787807814456755e-17 2.7755575615628913511e-17 -0.051749999999999775346 rpy=1.5707963267948976682 -0.051824161433128575205 1.5707963267948943376
