Commit message: Update robots

File: robots/talos_like/robot.urdf (robot description, URDF)
Before this commit: robot onshape, 14 links, 13 joints
Links:
- link ankle: mass 0.4254692017315677699 -> 0.42546920173156782541
- link foot: mass 2.4399385078931685733 -> 2.4399385078931690174
- link knee: mass 3.1208537261855564537 -> 3.1208537261855555656
- link rode_1: mass 0.0097669214712453687049 -> 0.0097669214712453669702

File: robots/wl16_like/robot.urdf (robot description, URDF)
Before this commit: robot onshape, 31 links, 30 joints
Links:
- link foot: mass 1.2962021735874538209 -> 1.2962021735874540429
- link hips: mass 43.978349764609021122 -> 43.978349764609063755
