Commit message: update other robot

File: example_parallel_robots/robots/5bar_linkage/robot.urdf (robot description, URDF)
Before this commit: robot onshape, 8 links, 7 joints
Links:
- removed link barre
- removed link barre_2
- removed link barre_3
- removed link barre_bout
- removed link batie
- removed link effecteur
- added link built, mass 90.55799165500025083; collision mesh filename=package:///built.stl; visual mesh filename=package:///built.stl
- added link effector, mass 1e-9
- added link end_rod, mass 29.820293741250193165; collision mesh filename=package:///end_rod.stl; visual mesh filename=package:///end_rod.stl
- added link rod, mass 24.820995827500130559; collision mesh filename=package:///rod.stl; visual mesh filename=package:///rod.stl
- added link rod_2, mass 24.820995827500130559; collision mesh filename=package:///rod.stl; visual mesh filename=package:///rod.stl
- added link rod_3, mass 24.820995827500130559; collision mesh filename=package:///rod.stl; visual mesh filename=package:///rod.stl
Joints:
- removed joint effecteur_frame
- removed joint fermeture1_A
- removed joint fermeture1_B
- removed joint libre1
- removed joint libre2
- added joint closedloop1_A: type revolute, parent rod_2, child sphere, origin xyz=2.7755575615628913511e-17 -0.46000000000000001998 -2.7755575615628913511e-17 rpy=2.0436181652775820801e-30 6.9767163393490848699e-30 1.570796326794896558, axis 0 0 1, limit effort=1 velocity=20
- added joint closedloop1_B: type revolute, parent end_rod, child sphere_2, origin xyz=-5.5511151231257827021e-17 -0.45999999999999985345 0.050000000000000002776 rpy=-6.1152609076707444674e-30 1.2212640759497854267e-29 -2.9143354396410176762e-16, axis 0 0 1, limit effort=1 velocity=20
- added joint effector_frame: type fixed, parent end_rod, child effector, origin xyz=0 -0.52750000000000019096 1.3877787807814456755e-17 rpy=-1.5707963267948958919 -1.570796326794896558 0, axis 0 0 0
- added joint free1: type revolute, parent rod, child rod_2, origin xyz=2.7755575615628913511e-17 -0.45999999999999990896 0.050000000000000016653 rpy=-1.5128280870939263564e-40 -3.6734198463195946286e-40 -6.1876044703704446752e-78, axis 0 0 1, limit effort=1 velocity=20
- added joint free2: type revolute, parent rod_3, child end_rod, origin xyz=2.7755575615628913511e-17 0.45999999999999996447 0 rpy=3.7235323964476006137e-42 7.1746481373430608542e-42 -3.141592653589793116, axis 0 0 1, limit effort=1 velocity=20
- joint mot1: child barre -> rod; parent batie -> built
- joint mot2: child barre_3 -> rod_3; parent batie -> built

File: example_parallel_robots/robots/5bar_linkage_iso3d/robot.urdf (robot description, URDF)
Before this commit: robot onshape, 9 links, 8 joints
Links:
- removed link effecteur
- removed link fermeture3D_1A
- removed link fermeture3D_1B
- added link closedloop3D_1A, mass 1e-9
- added link closedloop3D_1B, mass 1e-9
- added link effector, mass 1e-9
Joints:
- removed joint effecteur_frame
- removed joint fermeture3D_1A_frame
- removed joint fermeture3D_1B_frame
- removed joint libre1
- removed joint libre2
- removed joint libreortho
- added joint closedloop3D_1A_frame: type fixed, parent part_4, child closedloop3D_1A, origin xyz=0 -0.18000000000000015987 -0.062500000000000166533 rpy=1.570796326794896558 -1.570796326794896336 0, axis 0 0 0
- added joint closedloop3D_1B_frame: type fixed, parent part_5, child closedloop3D_1B, origin xyz=-0.0025000000000001132427 -0.36500000000000010214 -0.024999999999999994449 rpy=1.570796326794896558 4.8549226442908764763e-28 -3.1415926535897926719, axis 0 0 0
- added joint effector_frame: type fixed, parent part_4, child effector, origin xyz=0.025000000000000022204 -0.18000000000000004885 -0.067500000000000115463 rpy=3.141592653589793116 -2.0243283558835282576e-16 -1.570796326794896558, axis 0 0 0
- added joint free1: type revolute, parent part_2, child part_3, origin xyz=1.9428902930940239457e-16 0.31500000000000022427 -0.04999999999999997502 rpy=3.3991432702649502991e-18 -8.5627342893293126743e-18 2.0318009336061488845, axis 0 0 1, limit effort=1 velocity=20
- added joint free2: type revolute, parent part_1, child part_2_2, origin xyz=0.15000000000000004996 -0.10000000000000001943 -1.249000902703301108e-16 rpy=1.570796326794896558 0.44184666170691727638 3.141592653589793116, axis 0 0 1, limit effort=1 velocity=20
- added joint freeortho: type revolute, parent part_3, child part_4, origin xyz=-0.06500000000000000222 -0.34500000000000008438 -0.024999999999999994449 rpy=-1.45215238593493469e-17 1.570796326794896558 0, axis 0 0 1, limit effort=1 velocity=20

File: example_parallel_robots/robots/5bar_linkage_iso6d/robot.urdf (robot description, URDF)
Before this commit: robot onshape, 10 links, 9 joints
Links:
- removed link effecteur
- removed link fermeture6D_1A
- removed link fermeture6D_1B
- added link closedloop6D_1A, mass 1e-9
- added link closedloop6D_1B, mass 1e-9
- added link effector, mass 1e-9
Joints:
- removed joint effecteur_frame
- removed joint fermeture6D_1A_frame
- removed joint fermeture6D_1B_frame
- removed joint libre1
- removed joint libre2
- removed joint libreortho
- removed joint to_rotule_libre3
- added joint closedloop6D_1A_frame: type fixed, parent part_6, child closedloop6D_1A, origin xyz=5.5511151231257827021e-17 -2.7755575615628913511e-17 -0.10249999999999981348 rpy=-3.141592653589793116 7.4909873354573750005e-16 -3.141592653589793116, axis 0 0 0
- added joint closedloop6D_1B_frame: type fixed, parent part_5, child closedloop6D_1B, origin xyz=-0.0025000000000001687539 -0.36500000000000010214 -0.024999999999999994449 rpy=1.57079632679489678 -1.195073737747987526e-16 -3.141592653589793116, axis 0 0 0
- added joint effector_frame: type fixed, parent part_4, child effector, origin xyz=0.025000000000000022204 -0.18000000000000015987 -0.067499999999999976685 rpy=-3.141592653589793116 -1.5132630134575502908e-16 -1.570796326794896558, axis 0 0 0
- added joint free1: type revolute, parent part_2, child part_3, origin xyz=0 0.31500000000000005773 -0.049999999999999961142 rpy=-4.2298279813785684808e-19 -4.639019543158211348e-18 2.3867293943822684987, axis 0 0 1, limit effort=1 velocity=20
- added joint free2: type revolute, parent part_1, child part_2_2, origin xyz=0.1500000000000000222 -0.10000000000000000555 -2.4112656316077618612e-16 rpy=1.570796326794896558 0.058234987822223291398 3.141592653589793116, axis 0 0 1, limit effort=1 velocity=20
- added joint freeortho: type revolute, parent part_3, child part_4, origin xyz=-0.065000000000000113243 -0.34500000000000008438 -0.024999999999999994449 rpy=2.3794305551220863726e-16 1.5707963267948954478 0, axis 0 0 1, limit effort=1 velocity=20
- added joint spherical_free3: type revolute, parent part_4, child part_6, origin xyz=0 -0.18000000000000015987 -0.064999999999999918954 rpy=7.808431419004548746e-16 0.87266462599716454474 -1.5707963267948956698, axis 0 0 1, limit effort=1 velocity=20

File: example_parallel_robots/robots/robot_delta/robot.urdf (robot description, URDF)
Before this commit: robot onshape, 16 links, 15 joints
Links:
- removed link barre1
- removed link barre2
- removed link bielle1
- removed link bielle2
- removed link effecteur
- removed link renvois
- removed link renvois_barre
- removed link renvois_bielle
- added link connecting_rod1, mass 0.0044599281198533617665; collision mesh filename=package:///connecting_rod1.stl; visual mesh filename=package:///connecting_rod1.stl
- added link connecting_rod2, mass 0.0044599281198533661033; collision mesh filename=package:///connecting_rod2.stl; visual mesh filename=package:///connecting_rod2.stl
- added link effector, mass 0.0038207811339355168476; collision mesh filename=package:///effector.stl; visual mesh filename=package:///effector.stl
- added link rod1, mass 0.0028399281198533575174; collision mesh filename=package:///rod1.stl; visual mesh filename=package:///rod1.stl
- added link rod2, mass 0.0028399281198533622879; collision mesh filename=package:///rod2.stl; visual mesh filename=package:///rod2.stl
- added link transmission, mass 0.0013380381830738910607; collision mesh filename=package:///transmission.stl; visual mesh filename=package:///transmission.stl
- added link transmission_connecting_rod, mass 0.0021658241231472083639; collision mesh filename=package:///transmission_connecting_rod.stl; visual mesh filename=package:///transmission_connecting_rod.stl
- added link transmission_rod, mass 0.0014908241231472102797; collision mesh filename=package:///transmission_rod.stl; visual mesh filename=package:///transmission_rod.stl
Joints:
- removed joint fermeture1_A
- removed joint fermeture1_B
- removed joint fermeture2_A
- removed joint fermeture2_B
- removed joint fermeture3_A
- removed joint fermeture3_B
- removed joint libre1_bras1
- removed joint libre1_bras2
- removed joint libre1_bras3
- removed joint libre2_bras1
- removed joint libre2_bras3
- removed joint libre3_bras3
- removed joint mot1_bras1
- removed joint mot1_bras2
- added joint closedloop1_A: type revolute, parent transmission, child sphere_6, origin xyz=1.7347234759768070944e-17 0.008000000000000003636 0 rpy=5.1342448982226077446e-17 2.2017968259951186298e-16 -1.5707963267949633934, axis 0 0 1, limit effort=1 velocity=20
- added joint closedloop1_B: type revolute, parent connecting_rod2, child sphere_3, origin xyz=0 0 -0.002499999999999998751 rpy=1.880473962268720761e-55 -4.0583476162763403791e-55 -1.9618098062391555736, axis 0 0 1, limit effort=1 velocity=20
- added joint closedloop2_A: type revolute, parent connecting_rod2, child sphere_4, origin xyz=5.2041704279304212832e-18 0.05999999999999999778 0 rpy=-3.141592653589793116 -0 1.570796326794896558, axis 0 0 1, limit effort=1 velocity=20
- added joint closedloop2_B: type revolute, parent effector, child sphere_2, origin xyz=-1.7347234759768070944e-18 6.9388939039072283776e-18 -0.0024999999999999996184 rpy=-3.141592653589793116 1.1122345866076180164e-28 3.1204220693644000306, axis 0 0 1, limit effort=1 velocity=20
- added joint closedloop3_A: type revolute, parent transmission_connecting_rod, child sphere_5, origin xyz=6.0715321659188248304e-18 0.05999999999999999778 1.7347234759768070944e-18 rpy=-3.141592653589793116 -1.6250533601386852917e-33 -3.141592653589793116, axis 0 0 1, limit effort=1 velocity=20
- added joint closedloop3_B: type revolute, parent effector, child sphere, origin xyz=-0.0096592582628906940162 -0.0025881904510252004559 -0.0074999999999999997224 rpy=3.141592653589793116 3.469446951952502881e-16 -0.021170584225393276195, axis 0 0 1, limit effort=1 velocity=20
- added joint free1_rod1: type revolute, parent rod1, child connecting_rod1, origin xyz=-1.7347234759768070944e-18 0.040000000000000007772 0 rpy=3.141592653589793116 -5.7397185098697670323e-42 -7.0922928823064416586e-19, axis 0 0 1, limit effort=1 velocity=20
- added joint free1_rod2: type revolute, parent rod2, child connecting_rod2, origin xyz=-5.2041704279304212832e-18 0.040000000000000000833 -0.0024999999999999996184 rpy=-2.5639079630131276433e-26 2.4799494635820430051e-26 1.6300352109594598639e-51, axis 0 0 1, limit effort=1 velocity=20
- added joint free1_rod3: type revolute, parent bati, child transmission_rod, origin xyz=0.0075000000000001766642 0.012070552360820205329 0.057727406610312198554 rpy=-1.570796326794896558 3.5527136788004875187e-15 1.570796326794896558, axis 0 0 1, limit effort=1 velocity=20
- added joint free2_rod1: type revolute, parent connecting_rod1, child effector, origin xyz=0 -0.059999999999999983902 0 rpy=-3.141592653589793116 7.0113230956924185612e-27 1.704204991525385563e-18, axis 0 0 1, limit lower=-1.570796326794896558 upper=1.570796326794896558 effort=1 velocity=20
- added joint free2_rod3: type revolute, parent transmission_rod, child transmission, origin xyz=-3.4694469519536141888e-18 0.040000000000000007772 -0.0025000000000000013531 rpy=-5.0342327325063659791e-26 7.3518619293218564457e-26 1.5707963267949036634, axis 0 0 1, limit effort=1 velocity=20
- added joint free3_rod3: type revolute, parent transmission, child transmission_connecting_rod, origin xyz=-0.0099999999999999915345 0.0080000000000000105749 -0.002499999999999998751 rpy=1.8201011498345231359e-16 -6.013629783791155957e-16 -1.5707963267949633934, axis 0 0 1, limit effort=1 velocity=20
- added joint mot1_rod1: type revolute, parent bati, child rod1, origin xyz=0.0050000000000004901635 -0.0099999999999999776568 0.049999999999999863998 rpy=-1.570796326794896558 0.021170584225393279665 1.570796326794896558, axis 0 0 1, limit effort=1 velocity=20
- added joint mot1_rod2: type revolute, parent bati, child rod2, origin xyz=0.0050000000000000001041 0.010000000000000001943 0.050000000000000002776 rpy=-1.570796326794896558 2.7817834526774081734e-52 1.570796326794896558, axis 0 0 1, limit effort=1 velocity=20
- joint eff_frame: parent effecteur -> effector
