Commit message: 5 bar iso6 modified

File: example_parallel_robots/robots/5bar_linkage_iso6d/robot.urdf (robot description, URDF)
Before this commit: robot onshape, 10 links, 9 joints
Links:
- added link part_4_int1_1, mass 0.0
- added link part_4_int2_1, mass 0.0
Joints:
- removed joint spherical_free3
- added joint part_4_part_6_rev0: type revolute, parent part_4, child part_4_int1_1, origin xyz=0 -0.18000000000000015987 -0.064999999999999918954, axis 1 0 0, limit effort=1 velocity=20
- added joint part_4_part_6_rev1: type revolute, parent part_4_int1_1, child part_4_int2_1, axis 0 1 0, limit effort=1 velocity=20
- added joint part_4_part_6_rev2: type revolute, parent part_4_int2_1, child part_6, axis 0 0 1, limit effort=1 velocity=20
