Commit message: update cassie to new standard

File: example_parallel_robots/robots/cassie_like/robot.urdf (robot description, URDF)
Before this commit: robot onshape, 18 links, 17 joints
Links:
- removed link bout_pied
- removed link centre_hanche
- removed link fermeture1_A
- removed link fermeture1_B
- removed link fermeture2_A
- removed link fermeture2_B
- added link closedloop1_A, mass 1e-9
- added link closedloop1_B, mass 1e-9
- added link closedloop2_A, mass 1e-9
- added link closedloop2_B, mass 1e-9
- added link foot, mass 1e-9
- added link hip, mass 1e-9
- link foot_2: mass 0.17448227435667074126 -> 0.17448227435667082452
- link hip_roll: mass 1.2959080246959102656 -> 1.2959080246959100435
- link tarsus: mass 1.9514091738133036991 -> 1.9514091738133039211
Joints:
- removed joint bout_pied_frame
- removed joint centre_hanche_frame
- removed joint fermeture1_A_frame
- removed joint fermeture1_B_frame
- removed joint fermeture2_A_frame
- removed joint fermeture2_B_frame
- removed joint libre_cheville
- removed joint libre_genoux
- removed joint mot_cheville
- removed joint mot_cuisse
- removed joint mot_genoux
- removed joint mot_hanche1
- removed joint mot_hanche2
- removed joint to_rotule_free_genoux
- removed joint to_rotule_free_hanche
- removed joint to_rotule_free_molet
- removed joint to_rotule_free_pied
- added joint closedloop1_A_frame: type fixed, parent half_planta_rode, child closedloop1_A, origin xyz=-1.2143064331837649661e-17 -5.5511151231257827021e-17 -0.17499999999999993339 rpy=-3.9998783488706165629e-16 -3.1371620499754781664e-16 -1.9299084021460934093e-16, axis 0 0 0
- added joint closedloop1_B_frame: type fixed, parent half_planta_rode_2, child closedloop1_B, origin xyz=-1.1102230246251565404e-16 0 -0.17499999999999993339 rpy=3.1415926535897926719 2.2472903567366436713e-16 1.9179309870310918033e-17, axis 0 0 0
- added joint closedloop2_A_frame: type fixed, parent half_hachil_rode, child closedloop2_A, origin xyz=7.6327832942979512154e-17 2.7755575615628913511e-17 -0.25100000000000000089 rpy=-3.141592653589793116 -6.2578735636897098849e-17 -5.5511151231110433291e-17, axis 0 0 0
- added joint closedloop2_B_frame: type fixed, parent half_hachil_rode_2, child closedloop2_B, origin xyz=0 0 -0.25100000000000000089 rpy=0 -0 -5.8367148812184334304e-33, axis 0 0 0
- added joint foot_frame: type fixed, parent foot_2, child foot, origin xyz=0.017437288551799601244 0.053494595659102195384 -5.5511151231257827021e-17 rpy=1.570796326794896558 -2.579690608625463243e-32 7.5189606883587088013e-17, axis 0 0 0
- added joint free_ankle: type revolute, parent tarsus, child foot_2, origin xyz=-0.40817321560878561115 -0.040051999999999754465 -8.3266726846886740532e-17 rpy=-4.8132115049734420068e-17 5.2714015325247162167e-17 3.0436779078917255426, axis 0 0 1, limit effort=1 velocity=20
- added joint free_knee: type revolute, parent shin, child tarsus, origin xyz=0.49538451785003045913 0.066440389713804448579 -0.025000000000000022204 rpy=3.141592653589793116 7.7855609943435923412e-32 -1.57079632679489678, axis 0 0 1, limit effort=1 velocity=20
- added joint hip_frame: type fixed, parent pelvis, child hip, origin xyz=2.4027501270446963816e-19 -8.0668890063688602149e-19 -8.6736173798840393239e-19 rpy=-3.141592653589793116 1.7136028460806416378e-59 8.2107331894032250249e-48, axis 0 0 0
- added joint motor_ankle: type revolute, parent tarsus, child servo_gauche, origin xyz=-0.059638215608785377642 -0.032907999999999826279 0.025499999999999869993 rpy=3.141592653589793116 -7.1015003008495024371e-17 0.7436019737804375751, axis 0 0 1, limit effort=1 velocity=20
- added joint motor_hip1: type revolute, parent pelvis, child hip_pitch, origin xyz=-0.019710351940020659489 -0.13804195854893208661 0.025308433594891127649 rpy=-3.141592653589793116 -1.570796326794896558 0, axis 0 0 1, limit effort=1 velocity=20
- added joint motor_hip2: type revolute, parent hip_pitch, child hip_roll, origin xyz=-0.019115999999999976761 4.5009618254709948815e-10 -0.037728323691212151125 rpy=-1.5707963267948961139 -8.3200173597528512219e-32 -1.570796326794896336, axis 0 0 1, limit effort=1 velocity=20
- added joint motor_knee: type revolute, parent tigh, child shin, origin xyz=0.11999999999999999556 0 0 rpy=3.141592653589793116 -1.2509380223995319123e-32 0.89341897777118783885, axis 0 0 1, limit effort=1 velocity=20
- added joint motor_tigh: type revolute, parent hip_roll, child tigh, origin xyz=-0.024999999999999994449 -6.9388939039072283776e-18 -0.069698146467463528708 rpy=1.9890235727123534246e-47 1.5707963267948961139 0, axis 0 0 1, limit effort=1 velocity=20
- added joint spherical_foot: type revolute, parent foot_2, child half_planta_rode_2, origin xyz=-0.044721183654949425712 0.032465595659102119974 0.0047499999999999764633 rpy=-1.57079632679489678 4.0889288827580028673e-17 -1.570796326794896558, axis 0 0 1, limit effort=1 velocity=20
- added joint spherical_hip: type revolute, parent tigh, child half_hachil_rode_2, origin xyz=0 0 0.071140999999999968151 rpy=-1.5707963267948958919 1.3877787807814427173e-16 1.5707963267948974462, axis 0 0 1, limit effort=1 velocity=20
- added joint spherical_knee: type revolute, parent tarsus, child half_hachil_rode, origin xyz=0.12533558857838403289 0.020589067772979641191 0 rpy=-1.570796326794896558 -1.2294649081564687934e-14 3.141592653589793116, axis 0 0 1, limit effort=1 velocity=20
- added joint spherical_shin: type revolute, parent servo_gauche, child half_planta_rode, origin xyz=-3.3306690738754696213e-16 0.061228364595627748912 0.0063374999999999820366 rpy=-1.57079632679489678 -1.3143067936387966554 -1.5707963267948981123, axis 0 0 1, limit effort=1 velocity=20

Commit message: cassie modified

File: example_parallel_robots/robots/cassie_like/robot.urdf (robot description, URDF)
Before this commit: robot onshape, 18 links, 17 joints
Links:
- added link foot_2_int1_2, mass 0.0
- added link foot_2_int2_2, mass 0.0
- added link servo_gauche_int1_1, mass 0.0
- added link servo_gauche_int2_1, mass 0.0
- added link tarsus_int1_3, mass 0.0
- added link tarsus_int2_3, mass 0.0
- added link tigh_int1_4, mass 0.0
- added link tigh_int2_4, mass 0.0
Joints:
- removed joint spherical_foot
- removed joint spherical_hip
- removed joint spherical_knee
- removed joint spherical_shin
- added joint foot_2_half_planta_rode_2_rev0: type revolute, parent foot_2, child foot_2_int1_2, origin xyz=-0.044721183654949425712 0.032465595659102119974 0.0047499999999999764633, axis 1 0 0, limit effort=1 velocity=20
- added joint foot_2_half_planta_rode_2_rev1: type revolute, parent foot_2_int1_2, child foot_2_int2_2, axis 0 1 0, limit effort=1 velocity=20
- added joint foot_2_half_planta_rode_2_rev2: type revolute, parent foot_2_int2_2, child half_planta_rode_2, axis 0 0 1, limit effort=1 velocity=20
- added joint servo_gauche_half_planta_rode_rev0: type revolute, parent servo_gauche, child servo_gauche_int1_1, origin xyz=-3.3306690738754696213e-16 0.061228364595627748912 0.0063374999999999820366, axis 1 0 0, limit effort=1 velocity=20
- added joint servo_gauche_half_planta_rode_rev1: type revolute, parent servo_gauche_int1_1, child servo_gauche_int2_1, axis 0 1 0, limit effort=1 velocity=20
- added joint servo_gauche_half_planta_rode_rev2: type revolute, parent servo_gauche_int2_1, child half_planta_rode, axis 0 0 1, limit effort=1 velocity=20
- added joint tarsus_half_hachil_rode_rev0: type revolute, parent tarsus, child tarsus_int1_3, origin xyz=0.12533558857838403289 0.020589067772979641191 0, axis 1 0 0, limit effort=1 velocity=20
- added joint tarsus_half_hachil_rode_rev1: type revolute, parent tarsus_int1_3, child tarsus_int2_3, axis 0 1 0, limit effort=1 velocity=20
- added joint tarsus_half_hachil_rode_rev2: type revolute, parent tarsus_int2_3, child half_hachil_rode, axis 0 0 1, limit effort=1 velocity=20
- added joint tigh_half_hachil_rode_2_rev0: type revolute, parent tigh, child tigh_int1_4, origin xyz=0 0 0.071140999999999968151, axis 1 0 0, limit effort=1 velocity=20
- added joint tigh_half_hachil_rode_2_rev1: type revolute, parent tigh_int1_4, child tigh_int2_4, axis 0 1 0, limit effort=1 velocity=20
- added joint tigh_half_hachil_rode_2_rev2: type revolute, parent tigh_int2_4, child half_hachil_rode_2, axis 0 0 1, limit effort=1 velocity=20
