Commit message: start correction robot

File: example_parallel_robots/robots/digit_like/robot.urdf (robot description, URDF)
Before this commit: robot onshape, 24 links, 23 joints
Links:
- removed link bout_pied
- removed link centre_hanche
- removed link fermeture1_A
- removed link fermeture1_B
- removed link fermeture2_A
- removed link fermeture2_B
- removed link fermeture3_A
- removed link fermeture3_B
- removed link molet
- removed link molet_2
- added link closedloop1_A, mass 1e-9
- added link closedloop1_B, mass 1e-9
- added link closedloop2_A, mass 1e-9
- added link closedloop2_B, mass 1e-9
- added link closedloop3_A, mass 1e-9
- added link closedloop3_B, mass 1e-9
- added link crank, mass 0.0045332434126214744829; collision mesh filename=package:///crank.stl; visual mesh filename=package:///crank.stl
- added link crank_2, mass 0.0045332434126214744829; collision mesh filename=package:///crank.stl; visual mesh filename=package:///crank.stl
- added link hip, mass 1e-9
- link foot: mass 0.3309516742025366276 -> 1e-9; geometry 
- link foot_roll: mass 0.0027067106871796991867 -> 0.0027067106871796996204
- link hip_x: mass 1.4197410037164885921 -> 1.4197410037164888141
- link shin: mass 0.5557814093331634453 -> 0.55578140933316355632
- link tarsus: mass 0.74284619422086206608 -> 0.7428461942208621771
Joints:
- removed joint bout_pied_frame
- removed joint centre_hanche_frame
- removed joint fermeture1_A_frame
- removed joint fermeture1_B_frame
- removed joint fermeture2_A_frame
- removed joint fermeture2_B_frame
- removed joint fermeture3_A_frame
- removed joint fermeture3_B_frame
- removed joint libre_genoux
- removed joint libre_pied1
- removed joint libre_pied_2
- removed joint mot_genoux
- removed joint mot_hanche_x
- removed joint mot_hanche_y
- removed joint mot_hanche_z
- removed joint mot_servo1
- removed joint mot_servo2
- removed joint to_rotule_libre_genoux
- removed joint to_rotule_libre_hanche
- removed joint to_rotule_libre_molet1
- removed joint to_rotule_libre_molet2
- removed joint to_rotule_libre_pied1
- removed joint to_rotule_libre_pied2
- added joint closedloop1_A_frame: type fixed, parent toe_a_2/2, child closedloop1_A, origin xyz=9.0205620750793968909e-17 0 -0.19994999999999990559 rpy=-3.7112781480334425034e-16 8.2442115866850430893e-18 1.0097912624895015577e-27, axis 0 0 0
- added joint closedloop1_B_frame: type fixed, parent toe_a_1/2, child closedloop1_B, origin xyz=0 1.3877787807814456755e-17 -0.1999500000000002109 rpy=3.141592653589793116 -9.7378114602005348959e-18 3.141592653589793116, axis 0 0 0
- added joint closedloop2_A_frame: type fixed, parent toe_b_2/2, child closedloop2_A, origin xyz=0 0 -0.11994999999999994555 rpy=6.1280808278935614477e-17 3.5225097907092313716e-17 -1.5770158750347860435e-21, axis 0 0 0
- added joint closedloop2_B_frame: type fixed, parent toe_b_1/2_2, child closedloop2_B, origin xyz=-4.1633363423443370266e-17 0 -0.11995000000000000107 rpy=3.141592653589793116 1.9682319780529215571e-17 1.570796326794896558, axis 0 0 0
- added joint closedloop3_A_frame: type fixed, parent toe_b_2/2_2, child closedloop3_A, origin xyz=0 0 -0.11994999999999983453 rpy=1.7991914157564876276e-16 3.9760952339837050232e-18 -2.1710651278743624535e-18, axis 0 0 0
- added joint closedloop3_B_frame: type fixed, parent toe_b_1/2, child closedloop3_B, origin xyz=0 -1.1102230246251565404e-16 -0.11995000000000022311 rpy=3.141592653589793116 5.765418484336821195e-17 1.570796326794896558, axis 0 0 0
- added joint foot_frame: type fixed, parent foot, child foot, origin xyz=-0.05589761960057737511 0 0.014375929767894424227 rpy=3.141592653589793116 1.0420837364882535869 3.141592653589793116, axis 0 0 0
- added joint free_foot1: type revolute, parent tarsus, child foot_roll, origin xyz=-0.32599840000000018803 -0.038657982377658606232 -0.014000000000000074885 rpy=3.141592653589793116 -2.7008077392723998759e-16 -2.8764747500822966941, axis 0 0 1, limit effort=1 velocity=20
- added joint free_foot2: type revolute, parent foot_roll, child foot, origin xyz=0 0.0090000000000000079936 -0.013999999999999998557 rpy=-1.570796326794896558 3.0369740063504090599e-05 -3.1415926535897926719, axis 0 0 1, limit effort=1 velocity=20
- added joint free_knee: type revolute, parent shin, child tarsus, origin xyz=0.39567486363081372236 0.053875166733171692135 -0.025000000000000015266 rpy=3.141592653589793116 1.8170376977777737139e-18 -1.6910768536229012771, axis 0 0 1, limit effort=1 velocity=20
- added joint hip_frame: type fixed, parent torso, child hip, origin xyz=-2.4027501270446886779e-19 1.626303258728255688e-19 0.0024999999999999996184 rpy=2.8421709430404007435e-14 3.0814879110196404233e-31 3.141592653589793116, axis 0 0 0
- added joint motor_hip_x: type revolute, parent torso, child hip_y, origin xyz=0.02999999999999999889 0.072799999999999975842 0.059867854479678822566 rpy=-3.141592653589793116 1.570796326794896558 0, axis 0 0 1, limit effort=1 velocity=20
- added joint motor_hip_y: type revolute, parent hip_y, child hip_x, origin xyz=0.052665792973456596049 0 -0.035200000000000009059 rpy=1.570796326794896558 9.2157185462955552578e-18 -1.570796326794896558, axis 0 0 1, limit effort=1 velocity=20
- added joint motor_hip_z: type revolute, parent hip_x, child hip_z, origin xyz=-0.026000000000000002276 0 -0.054400000000000010847 rpy=-1.570796326794896558 -1.1931918349460191031 -1.5707963267948970021, axis 0 0 1, limit effort=1 velocity=20
- added joint motor_knee: type revolute, parent hip_z, child shin, origin xyz=-0.11999999999999998168 -1.3877787807814456755e-17 0 rpy=3.141592653589793116 1.6140181441454188796e-16 -2.6828651102102365478, axis 0 0 1, limit effort=1 velocity=20
- added joint motor_shin1: type revolute, parent tarsus, child crank, origin xyz=-0.088800000000000045564 -0.026113982377658551126 0.029999999999999985012 rpy=-3.141592653589793116 5.2844134501331837538e-18 0.085487820950950324517, axis 0 0 1, limit effort=1 velocity=20
- added joint motor_shin2: type revolute, parent tarsus, child crank_2, origin xyz=-0.088800000000000045564 -0.026113982377658551126 -0.030000000000000019706 rpy=-7.2028754011234369278e-17 -2.0682911281837146378e-18 -3.0334710307071497404, axis 0 0 1, limit effort=1 velocity=20
- added joint spherical_free_foot1: type revolute, parent foot, child toe_b_1/2, origin xyz=-0.0091288304490430016713 -0.014275999999999990087 0.052813599999999960577 rpy=1.57079632679489678 -8.3440173426621114272e-05 -1.570796326794896558, axis 0 0 1, limit effort=1 velocity=20
- added joint spherical_free_foot2: type revolute, parent foot, child toe_b_1/2_2, origin xyz=-0.0091288304490430016713 0.014276000000000010903 0.052813599999999960577 rpy=1.5707963267948970021 -8.3440173426648856295e-05 -1.570796326794896558, axis 0 0 1, limit effort=1 velocity=20
- added joint spherical_free_hip: type revolute, parent hip_x, child toe_a_2/2, origin xyz=0.033685999999999993726 0 -0.054399999999999996969 rpy=1.57079632679489678 -1.570796326794896336 0, axis 0 0 1, limit effort=1 velocity=20
- added joint spherical_free_knee: type revolute, parent tarsus, child toe_a_1/2, origin xyz=0.11418993498637036721 0.036206749731294507466 0 rpy=-1.57079632679489678 -1.2731099122301607895 -3.1415926535897926719, axis 0 0 1, limit effort=1 velocity=20
- added joint spherical_free_shin1: type revolute, parent crank_2, child toe_b_2/2_2, origin xyz=0 0.056999999999999995115 0.0025000000000000022204 rpy=1.5707963267948970021 -1.438335209354334232 -1.5707963267948930053, axis 0 0 1, limit effort=1 velocity=20
- added joint spherical_free_shin2: type revolute, parent crank, child toe_b_2/2, origin xyz=0 0.057000000000000050626 0.0025000000000000022204 rpy=1.570796326794896558 -0.00025864959668214364567 1.57079632679489678, axis 0 0 1, limit effort=1 velocity=20

File: example_parallel_robots/robots/talos_like/robot.urdf (robot description, URDF)
Before this commit: robot onshape, 14 links, 13 joints
Links:
- removed link bout_pied
- removed link centre_hanche
- removed link fermeture1_A
- removed link fermeture1_B
- removed link rode_1
- removed link rode_2
- added link closedloop1_A, mass 1e-9
- added link closedloop1_B, mass 1e-9
- added link hip, mass 1e-9
- added link rod_1, mass 0.0097669214712453687049; collision mesh filename=package:///rod_1.stl; visual mesh filename=package:///rod_1.stl
- added link rod_2, mass 0.010715370571438426195; collision mesh filename=package:///rod_2.stl; visual mesh filename=package:///rod_2.stl
- link foot: mass 2.4399385078931690174 -> 1e-9; geometry 
- link hip_x: mass 0.79889634230491624045 -> 0.79889634230491601841
- link hip_z: mass 5.8694864970653579661 -> 5.8694864970653588543
- link knee: mass 3.1208537261855555656 -> 3.1208537261855564537
Joints:
- removed joint bout_pied_frame
- removed joint centre_hanche_frame
- removed joint fermeture1_A_frame
- removed joint fermeture1_B_frame
- removed joint free_cheville
- removed joint free_to_rotule_molet
- removed joint free_to_rotule_pied
- removed joint mot_cheville
- removed joint mot_genoux
- removed joint mot_hanch_y
- removed joint mot_hanche_x
- removed joint mot_hanche_z
- removed joint mot_molet
- added joint closedloop1_A_frame: type fixed, parent rod_1, child closedloop1_A, origin xyz=-1.1102230246251565404e-16 0 -0.09766921471245393338 rpy=-3.0473731582998980835e-17 -0.052380185283905734972 -7.432341433572684695e-18, axis 0 0 0
- added joint closedloop1_B_frame: type fixed, parent rod_2, child closedloop1_B, origin xyz=-0.0056101647180723385189 -1.6653345369377348106e-16 -0.10700674137717214318 rpy=-3.0892124683058885815 9.926167565595004985e-24 1.5707963267948958919, axis 0 0 0
- added joint foot_frame: type fixed, parent foot, child foot, origin xyz=0.0037180509068605455125 -0.10113711488645749093 0.026634499999999991515 rpy=-1.570796326794896336 -1.570796326794896558 0, axis 0 0 0
- added joint free_ankle: type revolute, parent knee, child ankle, origin xyz=-2.7755575615628913511e-16 0.32492300000000001736 0.1211999999999999883 rpy=-3.3681081625124890998e-16 1.5434403186069809791e-16 -0.39124082415745392582, axis 0 0 1, limit effort=1 velocity=20
- added joint free_spherical_foot: type revolute, parent ankle, child rod_2, origin xyz=-0.071653553385825186073 -0.020555800061897611108 -0.0096809999999999951648 rpy=-1.5707963267948970021 0.21638278784128975318 -4.9155172359768353702e-16, axis 0 0 1, limit effort=1 velocity=20
- added joint free_spherical_shin: type revolute, parent moteur, child rod_1, origin xyz=-0.071653553385825130562 0.020555800061899054398 -0.0096810000000000506759 rpy=-1.570796326794896558 -9.3594596865425342696e-17 -3.1415926535897926719, axis 0 0 1, limit effort=1 velocity=20
- added joint hip_frame: type fixed, parent buste, child hip, origin xyz=2.4027501270446963816e-19 0.074999999999999997224 -0.097500000000000003331 rpy=0 -0 0, axis 0 0 0
- added joint motor_ankle: type revolute, parent ankle, child foot, origin xyz=-0.026499999999999676592 0.001371350934377235653 -0.10499999999999996836 rpy=3.141592653589793116 -1.5707963255260641855 0, axis 0 0 1, limit effort=1 velocity=20
- added joint motor_hip_x: type revolute, parent hip_x, child hip_y, origin xyz=-0.025999999999999998807 2.7755575615628913511e-17 -0.0934999999999999859 rpy=1.570796326794896558 4.3603698957148256544e-17 -1.570796326794896558, axis 0 0 1, limit effort=1 velocity=20
- added joint motor_hip_y: type revolute, parent hip_y, child hip_z, origin xyz=-0.0780000000000000554 1.3877787807814456755e-17 -0.025999999999999967581 rpy=-1.5707963267948970021 -0.99311814123129293908 -1.5707963267948961139, axis 0 0 1, limit effort=1 velocity=20
- added joint motor_hip_z: type revolute, parent buste, child hip_x, origin xyz=0.02371448658186565972 0.084999999999999992228 -0.010000000000000008882 rpy=0 -0 0, axis 0 0 1, limit effort=1 velocity=20
- added joint motor_knee: type revolute, parent hip_z, child knee, origin xyz=0.018186673545849449396 0.37956454642832049284 0.096000000000000029754 rpy=-3.141592653589793116 3.7503479430427692051e-17 2.1726736438687357378, axis 0 0 1, limit effort=1 velocity=20
- added joint motor_shin: type revolute, parent knee, child moteur, origin xyz=0.010729000000000044057 0.12028099999999997127 0.12120000000000001605 rpy=-1.7163581602055608654e-16 3.2833637602275228514e-16 0.26818340469683032978, axis 0 0 1, limit effort=1 velocity=20

Commit message: update digit to new standard

File: example_parallel_robots/robots/digit_like/robot.urdf (robot description, URDF)
Before this commit: robot onshape, 23 links, 23 joints
Links:
- added link foot_part, mass 0.33095167420253657209; collision mesh filename=package:///foot_part.stl; visual mesh filename=package:///foot_part.stl
- link hip_z: mass 3.8932756153047387571 -> 3.893275615304738313
- link tarsus: mass 0.7428461942208621771 -> 0.74284619422086228813
Joints:
- joint foot_frame: parent foot -> foot_part
- joint free_foot2: child foot -> foot_part
- joint spherical_free_foot1: parent foot -> foot_part
- joint spherical_free_foot2: parent foot -> foot_part

Commit message: dgit modified

File: example_parallel_robots/robots/digit_like/robot.urdf (robot description, URDF)
Before this commit: robot onshape, 24 links, 23 joints
Links:
- added link crank_2_int1_4, mass 0.0
- added link crank_2_int2_4, mass 0.0
- added link crank_int1_3, mass 0.0
- added link crank_int2_3, mass 0.0
- added link foot_part_int1_1, mass 0.0
- added link foot_part_int1_2, mass 0.0
- added link foot_part_int2_1, mass 0.0
- added link foot_part_int2_2, mass 0.0
- added link hip_x_int1_6, mass 0.0
- added link hip_x_int2_6, mass 0.0
- added link tarsus_int1_5, mass 0.0
- added link tarsus_int2_5, mass 0.0
Joints:
- removed joint spherical_free_foot1
- removed joint spherical_free_foot2
- removed joint spherical_free_hip
- removed joint spherical_free_knee
- removed joint spherical_free_shin1
- removed joint spherical_free_shin2
- added joint crank_2_toe_b_2/2_2_rev0: type revolute, parent crank_2, child crank_2_int1_4, origin xyz=0 0.056999999999999995115 0.0025000000000000022204, axis 1 0 0, limit effort=1 velocity=20
- added joint crank_2_toe_b_2/2_2_rev1: type revolute, parent crank_2_int1_4, child crank_2_int2_4, axis 0 1 0, limit effort=1 velocity=20
- added joint crank_2_toe_b_2/2_2_rev2: type revolute, parent crank_2_int2_4, child toe_b_2/2_2, axis 0 0 1, limit effort=1 velocity=20
- added joint crank_toe_b_2/2_rev0: type revolute, parent crank, child crank_int1_3, origin xyz=0 0.057000000000000050626 0.0025000000000000022204, axis 1 0 0, limit effort=1 velocity=20
- added joint crank_toe_b_2/2_rev1: type revolute, parent crank_int1_3, child crank_int2_3, axis 0 1 0, limit effort=1 velocity=20
- added joint crank_toe_b_2/2_rev2: type revolute, parent crank_int2_3, child toe_b_2/2, axis 0 0 1, limit effort=1 velocity=20
- added joint foot_part_toe_b_1/2_2_rev0: type revolute, parent foot_part, child foot_part_int1_2, origin xyz=-0.0091288304490430016713 0.014276000000000010903 0.052813599999999960577, axis 1 0 0, limit effort=1 velocity=20
- added joint foot_part_toe_b_1/2_2_rev1: type revolute, parent foot_part_int1_2, child foot_part_int2_2, axis 0 1 0, limit effort=1 velocity=20
- added joint foot_part_toe_b_1/2_2_rev2: type revolute, parent foot_part_int2_2, child toe_b_1/2_2, axis 0 0 1, limit effort=1 velocity=20
- added joint foot_part_toe_b_1/2_rev0: type revolute, parent foot_part, child foot_part_int1_1, origin xyz=-0.0091288304490430016713 -0.014275999999999990087 0.052813599999999960577, axis 1 0 0, limit effort=1 velocity=20
- added joint foot_part_toe_b_1/2_rev1: type revolute, parent foot_part_int1_1, child foot_part_int2_1, axis 0 1 0, limit effort=1 velocity=20
- added joint foot_part_toe_b_1/2_rev2: type revolute, parent foot_part_int2_1, child toe_b_1/2, axis 0 0 1, limit effort=1 velocity=20
- added joint hip_x_toe_a_2/2_rev0: type revolute, parent hip_x, child hip_x_int1_6, origin xyz=0.033685999999999993726 0 -0.054399999999999996969, axis 1 0 0, limit effort=1 velocity=20
- added joint hip_x_toe_a_2/2_rev1: type revolute, parent hip_x_int1_6, child hip_x_int2_6, axis 0 1 0, limit effort=1 velocity=20
- added joint hip_x_toe_a_2/2_rev2: type revolute, parent hip_x_int2_6, child toe_a_2/2, axis 0 0 1, limit effort=1 velocity=20
- added joint tarsus_toe_a_1/2_rev0: type revolute, parent tarsus, child tarsus_int1_5, origin xyz=0.11418993498637036721 0.036206749731294507466 0, axis 1 0 0, limit effort=1 velocity=20
- added joint tarsus_toe_a_1/2_rev1: type revolute, parent tarsus_int1_5, child tarsus_int2_5, axis 0 1 0, limit effort=1 velocity=20
- added joint tarsus_toe_a_1/2_rev2: type revolute, parent tarsus_int2_5, child toe_a_1/2, axis 0 0 1, limit effort=1 velocity=20
