Commit message: digit 2 legs  modified

File: example_parallel_robots/robots/digit_like_2legs/robot.urdf (robot description, URDF)
Before this commit: robot onshape, 46 links, 45 joints
Links:
- added link crank_2_int1_4, mass 0.0
- added link crank_2_int2_4, mass 0.0
- added link crank_3_int1_9, mass 0.0
- added link crank_3_int2_9, mass 0.0
- added link crank_4_int1_10, mass 0.0
- added link crank_4_int2_10, mass 0.0
- added link crank_int1_3, mass 0.0
- added link crank_int2_3, mass 0.0
- added link foot_part_2_int1_7, mass 0.0
- added link foot_part_2_int1_8, mass 0.0
- added link foot_part_2_int2_7, mass 0.0
- added link foot_part_2_int2_8, mass 0.0
- added link foot_part_int1_1, mass 0.0
- added link foot_part_int1_2, mass 0.0
- added link foot_part_int2_1, mass 0.0
- added link foot_part_int2_2, mass 0.0
- added link hip_x_2_int1_12, mass 0.0
- added link hip_x_2_int2_12, mass 0.0
- added link hip_x_int1_6, mass 0.0
- added link hip_x_int2_6, mass 0.0
- added link tarsus_2_int1_11, mass 0.0
- added link tarsus_2_int2_11, mass 0.0
- added link tarsus_int1_5, mass 0.0
- added link tarsus_int2_5, mass 0.0
Joints:
- removed joint spherical_free_foot1
- removed joint spherical_free_foot1_left
- removed joint spherical_free_foot2
- removed joint spherical_free_foot2_left
- removed joint spherical_free_hip
- removed joint spherical_free_hip_left
- removed joint spherical_free_knee
- removed joint spherical_free_knee_left
- removed joint spherical_free_shin1
- removed joint spherical_free_shin1_left
- removed joint spherical_free_shin2
- removed joint spherical_free_shin2_left
- added joint crank_2_toe_b_2/2_2_rev0: type revolute, parent crank_2, child crank_2_int1_4, origin xyz=5.5511151231257827021e-17 0.056999999999999939604 0.0024999999999999883427, axis 1 0 0, limit effort=1 velocity=20
- added joint crank_2_toe_b_2/2_2_rev1: type revolute, parent crank_2_int1_4, child crank_2_int2_4, axis 0 1 0, limit effort=1 velocity=20
- added joint crank_2_toe_b_2/2_2_rev2: type revolute, parent crank_2_int2_4, child toe_b_2/2_2, axis 0 0 1, limit effort=1 velocity=20
- added joint crank_3_toe_b_2/2_4_rev0: type revolute, parent crank_3, child crank_3_int1_9, origin xyz=-5.5511151231257827021e-17 0.057000000000000050626 0.0025000000000000022204, axis 1 0 0, limit effort=1 velocity=20
- added joint crank_3_toe_b_2/2_4_rev1: type revolute, parent crank_3_int1_9, child crank_3_int2_9, axis 0 1 0, limit effort=1 velocity=20
- added joint crank_3_toe_b_2/2_4_rev2: type revolute, parent crank_3_int2_9, child toe_b_2/2_4, axis 0 0 1, limit effort=1 velocity=20
- added joint crank_4_toe_b_1/2_4_rev0: type revolute, parent crank_4, child crank_4_int1_10, origin xyz=2.2204460492503130808e-16 0.057000000000000494715 0.0025000000000004185541, axis 1 0 0, limit effort=1 velocity=20
- added joint crank_4_toe_b_1/2_4_rev1: type revolute, parent crank_4_int1_10, child crank_4_int2_10, axis 0 1 0, limit effort=1 velocity=20
- added joint crank_4_toe_b_1/2_4_rev2: type revolute, parent crank_4_int2_10, child toe_b_1/2_4, axis 0 0 1, limit effort=1 velocity=20
- added joint crank_toe_b_2/2_rev0: type revolute, parent crank, child crank_int1_3, origin xyz=5.5511151231257827021e-17 0.057000000000000050626 0.002499999999999967526, axis 1 0 0, limit effort=1 velocity=20
- added joint crank_toe_b_2/2_rev1: type revolute, parent crank_int1_3, child crank_int2_3, axis 0 1 0, limit effort=1 velocity=20
- added joint crank_toe_b_2/2_rev2: type revolute, parent crank_int2_3, child toe_b_2/2, axis 0 0 1, limit effort=1 velocity=20
- added joint foot_part_2_toe_b_1/2_3_rev0: type revolute, parent foot_part_2, child foot_part_2_int1_7, origin xyz=-0.0091288304490432237159 -0.014276000000000010903 -0.034653600000000173154, axis 1 0 0, limit effort=1 velocity=20
- added joint foot_part_2_toe_b_1/2_3_rev1: type revolute, parent foot_part_2_int1_7, child foot_part_2_int2_7, axis 0 1 0, limit effort=1 velocity=20
- added joint foot_part_2_toe_b_1/2_3_rev2: type revolute, parent foot_part_2_int2_7, child toe_b_1/2_3, axis 0 0 1, limit effort=1 velocity=20
- added joint foot_part_2_toe_b_2/2_3_rev0: type revolute, parent foot_part_2, child foot_part_2_int1_8, origin xyz=-0.0091288304490432237159 0.014275999999999927637 -0.034653600000000284176, axis 1 0 0, limit effort=1 velocity=20
- added joint foot_part_2_toe_b_2/2_3_rev1: type revolute, parent foot_part_2_int1_8, child foot_part_2_int2_8, axis 0 1 0, limit effort=1 velocity=20
- added joint foot_part_2_toe_b_2/2_3_rev2: type revolute, parent foot_part_2_int2_8, child toe_b_2/2_3, axis 0 0 1, limit effort=1 velocity=20
- added joint foot_part_toe_b_1/2_2_rev0: type revolute, parent foot_part, child foot_part_int1_2, origin xyz=-0.009128830449042890649 0.014276000000000017842 0.052813599999999794044, axis 1 0 0, limit effort=1 velocity=20
- added joint foot_part_toe_b_1/2_2_rev1: type revolute, parent foot_part_int1_2, child foot_part_int2_2, axis 0 1 0, limit effort=1 velocity=20
- added joint foot_part_toe_b_1/2_2_rev2: type revolute, parent foot_part_int2_2, child toe_b_1/2_2, axis 0 0 1, limit effort=1 velocity=20
- added joint foot_part_toe_b_1/2_rev0: type revolute, parent foot_part, child foot_part_int1_1, origin xyz=-0.0091288304490431126936 -0.014275999999999927637 0.052813599999999960577, axis 1 0 0, limit effort=1 velocity=20
- added joint foot_part_toe_b_1/2_rev1: type revolute, parent foot_part_int1_1, child foot_part_int2_1, axis 0 1 0, limit effort=1 velocity=20
- added joint foot_part_toe_b_1/2_rev2: type revolute, parent foot_part_int2_1, child toe_b_1/2, axis 0 0 1, limit effort=1 velocity=20
- added joint hip_x_2_toe_a_2/2_2_rev0: type revolute, parent hip_x_2, child hip_x_2_int1_12, origin xyz=0.030568773343218405558 0 -0.054400000000000003908, axis 1 0 0, limit effort=1 velocity=20
- added joint hip_x_2_toe_a_2/2_2_rev1: type revolute, parent hip_x_2_int1_12, child hip_x_2_int2_12, axis 0 1 0, limit effort=1 velocity=20
- added joint hip_x_2_toe_a_2/2_2_rev2: type revolute, parent hip_x_2_int2_12, child toe_a_2/2_2, axis 0 0 1, limit effort=1 velocity=20
- added joint hip_x_toe_a_2/2_rev0: type revolute, parent hip_x, child hip_x_int1_6, origin xyz=0.033686000000000014543 -4.1633363423443370266e-17 -0.054400000000000017786, axis 1 0 0, limit effort=1 velocity=20
- added joint hip_x_toe_a_2/2_rev1: type revolute, parent hip_x_int1_6, child hip_x_int2_6, axis 0 1 0, limit effort=1 velocity=20
- added joint hip_x_toe_a_2/2_rev2: type revolute, parent hip_x_int2_6, child toe_a_2/2, axis 0 0 1, limit effort=1 velocity=20
- added joint tarsus_2_toe_a_1/2_2_rev0: type revolute, parent tarsus_2, child tarsus_2_int1_11, origin xyz=0.1141899349863718105 0.03620674973129278662 7.3552275381416620803e-16, axis 1 0 0, limit effort=1 velocity=20
- added joint tarsus_2_toe_a_1/2_2_rev1: type revolute, parent tarsus_2_int1_11, child tarsus_2_int2_11, axis 0 1 0, limit effort=1 velocity=20
- added joint tarsus_2_toe_a_1/2_2_rev2: type revolute, parent tarsus_2_int2_11, child toe_a_1/2_2, axis 0 0 1, limit effort=1 velocity=20
- added joint tarsus_toe_a_1/2_rev0: type revolute, parent tarsus, child tarsus_int1_5, origin xyz=0.1141899349863703117 0.036206749731294562977 0, axis 1 0 0, limit effort=1 velocity=20
- added joint tarsus_toe_a_1/2_rev1: type revolute, parent tarsus_int1_5, child tarsus_int2_5, axis 0 1 0, limit effort=1 velocity=20
- added joint tarsus_toe_a_1/2_rev2: type revolute, parent tarsus_int2_5, child toe_a_1/2, axis 0 0 1, limit effort=1 velocity=20
