Commit message: update disney

File: example_parallel_robots/robots/disney_like/robot.urdf (robot description, URDF)
Before this commit: robot onshape, 26 links, 25 joints
Links:
- removed link bout_pied
- removed link centre_hanche
- removed link fermeture1_A
- removed link fermeture1_B
- removed link fermeture2_A
- removed link fermeture2_B
- removed link fermeture3_A
- removed link fermeture3_B
- added link closedloop1_A, mass 1e-9
- added link closedloop1_B, mass 1e-9
- added link closedloop2_A, mass 1e-9
- added link closedloop2_B, mass 1e-9
- added link closedloop3_A, mass 1e-9
- added link closedloop3_B, mass 1e-9
- added link hip, mass 1e-9
- link bloc_moteur: mass 11.246937103837288063 -> 11.246937103837284511
- link cheville: mass 0.33045817880272942979 -> 0.33045817880272937428
- link foot: mass 9.775601923935292703 -> 1e-9; geometry 
Joints:
- removed joint bout_pied_frame
- removed joint centre_hanche_frame
- removed joint fermeture1_A_frame
- removed joint fermeture1_B_frame
- removed joint fermeture2_A_frame
- removed joint fermeture2_B_frame
- removed joint fermeture3_A_frame
- removed joint fermeture3_B_frame
- removed joint free_4link5
- removed joint free_4link6
- removed joint free_cardan1
- removed joint free_cardan2
- removed joint free_cardan3_to_rotule
- removed joint free_hipsx
- removed joint free_to_rotule_4link3
- removed joint free_to_rotule_4link4
- removed joint mot_4link1
- removed joint mot_4link2
- removed joint mot_4link3
- removed joint mot_4link4
- removed joint mot_cheville
- removed joint mot_hipsx
- removed joint to_rotule_1
- removed joint to_rotule_2
- added joint closedloop1_A_frame: type fixed, parent tibias_mirror, child closedloop1_A, origin xyz=1.1102230246251565404e-16 -5.5511151231257827021e-17 -0.10666666666666652086 rpy=-7.0826551989213637361e-16 5.0108442370046637999e-16 8.3199342453526548535e-17, axis 0 0 0
- added joint closedloop1_B_frame: type fixed, parent tibias_mirror2, child closedloop1_B, origin xyz=-1.1102230246251565404e-16 0.27066923076923060654 2.7755575615628913511e-16 rpy=-1.570796326794896558 -6.9533746316801810132e-17 1.8765245027468448435e-17, axis 0 0 0
- added joint closedloop2_A_frame: type fixed, parent cuiqqe_22, child closedloop2_A, origin xyz=-0.098047014809141019853 -0.36591500633661799835 -8.9052723362126329221e-08 rpy=1.570796326794896336 3.9766546240696217832e-16 3.141592653589793116, axis 0 0 0
- added joint closedloop2_B_frame: type fixed, parent cuiqqe_2, child closedloop2_B, origin xyz=0.018726579856343239516 0.069889981937422795966 8.9052723445393056068e-08 rpy=1.57079632679489678 6.2116731977486425824e-17 3.1415926535897806815, axis 0 0 0
- added joint closedloop3_A_frame: type fixed, parent cuiqqe_22_2, child closedloop3_A, origin xyz=-0.09804663044632583313 -0.36591500633661810937 5.5511151231257827021e-17 rpy=1.5707963267948956698 -8.7456685035717067728e-18 3.1415926535897922278, axis 0 0 0
- added joint closedloop3_B_frame: type fixed, parent cuiqqe_2_2, child closedloop3_B, origin xyz=0.018726579856343239516 0.069889981937422795966 8.9052723417637480452e-08 rpy=1.570796326794896336 -6.6744906857665710867e-17 -3.1415926535897926719, axis 0 0 0
- added joint foot_frame: type fixed, parent foot, child foot, origin xyz=0.02871794871794855486 0.10256410256410286586 0 rpy=1.570796326794896558 -6.9388939039056606707e-18 -2.8965986363544974793e-31, axis 0 0 0
- added joint free_4barlink5: type revolute, parent cuisse_1, child tibias, origin xyz=6.9388939039072283776e-17 -0.37743589743589744945 0 rpy=-4.5155172960891913228e-17 -4.4892155809767338609e-16 -1.439300600469447744, axis 0 0 1, limit effort=1 velocity=20
- added joint free_4barlink6: type revolute, parent cuisse_1_2, child tibias_mirror2, origin xyz=1.3877787807814456755e-16 0.37743589743589756047 0 rpy=-2.7475810661940926133e-16 -2.1857764558124863903e-16 1.3398696506926415228, axis 0 0 1, limit effort=1 velocity=20
- added joint free_hip_x: type revolute, parent part_9, child bloc_moteur, origin xyz=0.061538461538461514122 -0.41641025641025630755 -0.024615384615384594547 rpy=-1.570796326794896558 -0.034665069869454112617 1.570796326794896558, axis 0 0 1, limit effort=1 velocity=20
- added joint free_universal1: type revolute, parent tibias, child cardan, origin xyz=0 -0.37743589743589733843 2.7755575615628913511e-17 rpy=1.570796326794896558 0.0050482419228041449169 1.6594171315849655033e-15, axis 0 0 1, limit effort=1 velocity=20
- added joint free_universal2: type revolute, parent cardan, child cheville, origin xyz=-0.00029538461538458626876 5.5511151231257827021e-17 -0.00029538461538464177991 rpy=1.57079632679489678 0.0088312852163830307672 -1.5707963267948970021, axis 0 0 1, limit effort=1 velocity=20
- added joint hip_frame: type fixed, parent part_9, child hip, origin xyz=0.20000312504882905573 -0.35064297879654365842 -0.015450280473132521272 rpy=1.2764350627171105268e-14 -0 -6.1232339957367438492e-17, axis 0 0 0
- added joint motor_4barlink1: type revolute, parent bloc_moteur2, child part_6, origin xyz=0.034871794871794675741 -0.10666666666666652086 -0.13538461538461535327 rpy=1.570796326794896558 0.95118241861191532571 -1.570796326794896336, axis 0 0 1, limit effort=1 velocity=20
- added joint motor_4barlink2: type revolute, parent bloc_moteur, child part_6_2, origin xyz=-0.034871794871794925541 -0.10666666666666653474 -0.13538461538461535327 rpy=-1.570796326794896558 0.81155647644717276989 -1.57079632679489678, axis 0 0 1, limit effort=1 velocity=20
- added joint motor_4barlink3: type revolute, parent bloc_moteur2, child cuisse_1, origin xyz=0.034871794871794703496 3.8163916471489756077e-17 -0.049230769230769216849 rpy=1.570796326794896558 0.65078186773195378922 -1.570796326794896336, axis 0 0 1, limit effort=1 velocity=20
- added joint motor_4barlink4: type revolute, parent bloc_moteur, child cuisse_1_2, origin xyz=-0.034871794871794981052 -8.6736173798840354721e-18 -0.049230769230769216849 rpy=-1.570796326794896558 0.75635458602387717342 -1.570796326794896558, axis 0 0 1, limit effort=1 velocity=20
- added joint motor_ankle: type revolute, parent cheville, child foot, origin xyz=-0.11076923076923070322 1.6653345369377348106e-16 -5.5511151231257827021e-17 rpy=-1.570796326794896558 1.0514878939640439626 -1.5707963267948961139, axis 0 0 1, limit effort=1 velocity=20
- added joint motor_hip_x: type revolute, parent part_9, child bloc_moteur2, origin xyz=0.061538461538461514122 -0.26461538461538441913 -0.024615384615384483524 rpy=-1.570796326794896558 0.010172299766896189879 1.570796326794896558, axis 0 0 1, limit effort=1 velocity=20
- added joint spherical_free_4barlink1: type revolute, parent part_6_2, child cuiqqe_22_2, origin xyz=0.16410256410256410242 -2.7755575615628913511e-17 -5.5511151231257827021e-17 rpy=-3.141592653589793116 2.6020322225198728799e-16 -0.017899381364008804668, axis 0 0 1, limit effort=1 velocity=20
- added joint spherical_free_4barlink2: type revolute, parent part_6, child cuiqqe_22, origin xyz=0.16410256410256421344 -1.3877787807814456755e-17 -5.5511151231257827021e-17 rpy=-1.8001705999122800977e-17 1.23480581994850213e-16 0.29559516206773489566, axis 0 0 1, limit effort=1 velocity=20
- added joint spherical_free_4barlink3: type revolute, parent tibias_mirror2, child cuiqqe_2_2, origin xyz=0.12024806843488550223 -0.12907742097056101871 5.5511151231257827021e-17 rpy=-3.141592653589793116 3.4952106738054546811e-16 -0.99380518745195023378, axis 0 0 1, limit effort=1 velocity=20
- added joint spherical_free_4barlink4: type revolute, parent tibias, child cuiqqe_2, origin xyz=0.12024806843488550223 0.12907742097056090769 8.3266726846886740532e-17 rpy=3.101675607867788693e-16 -1.6442897688707137481e-16 1.0221182606507059898, axis 0 0 1, limit effort=1 velocity=20
- added joint spherical_free_foot: type revolute, parent cheville, child cardan_2, origin xyz=-0.2215384615384614897 1.1102230246251565404e-16 0 rpy=1.018762015073934528e-16 6.8533423168462731645e-16 3.1404277272486473827, axis 0 0 1, limit effort=1 velocity=20

Commit message: update disney to new standard

File: example_parallel_robots/robots/disney_like/robot.urdf (robot description, URDF)
Before this commit: robot onshape, 25 links, 25 joints
Links:
- removed link bloc_moteur
- removed link bloc_moteur2
- removed link cardan
- removed link cardan_2
- removed link cheville
- removed link cuiqqe_2
- removed link cuiqqe_22
- removed link cuiqqe_22_2
- removed link cuiqqe_2_2
- removed link cuisse_1
- removed link cuisse_1_2
- removed link part_6
- removed link part_6_2
- removed link part_9
- removed link tibias
- removed link tibias_mirror
- removed link tibias_mirror2
- added link ankle, mass 0.33045817880272942979; collision mesh filename=package:///ankle.stl; visual mesh filename=package:///ankle.stl
- added link foot_part, mass 9.775601923935292703; collision mesh filename=package:///foot_part.stl; visual mesh filename=package:///foot_part.stl
- added link hip_part, mass 8.9064002264242461138; collision mesh filename=package:///hip_part.stl; visual mesh filename=package:///hip_part.stl
- added link motor_1, mass 11.246937103837177929; collision mesh filename=package:///motor_1.stl; visual mesh filename=package:///motor_1.stl
- added link motor_2, mass 11.246937103837284511; collision mesh filename=package:///motor_2.stl; visual mesh filename=package:///motor_2.stl
- added link motor_link, mass 0.28186684374163423206; collision mesh filename=package:///motor_link.stl; visual mesh filename=package:///motor_link.stl
- added link motor_link_2, mass 0.28186684374163423206; collision mesh filename=package:///motor_link.stl; visual mesh filename=package:///motor_link.stl
- added link shin, mass 0.59977356844858531471; collision mesh filename=package:///shin.stl; visual mesh filename=package:///shin.stl
- added link shin_mirror1, mass 0.090242128488126502339; collision mesh filename=package:///shin_mirror1.stl; visual mesh filename=package:///shin_mirror1.stl
- added link shin_mirror2, mass 0.50944821011060736904; collision mesh filename=package:///shin_mirror2.stl; visual mesh filename=package:///shin_mirror2.stl
- added link tigh_1, mass 0.4623509198917738483; collision mesh filename=package:///tigh_1.stl; visual mesh filename=package:///tigh_1.stl
- added link tigh_1_2, mass 0.4623509198917738483; collision mesh filename=package:///tigh_1.stl; visual mesh filename=package:///tigh_1.stl
- added link tigh_mirror1, mass 0.13272969052998584427; collision mesh filename=package:///tigh_mirror1.stl; visual mesh filename=package:///tigh_mirror1.stl
- added link tigh_mirror1_2, mass 0.13272969052998584427; collision mesh filename=package:///tigh_mirror1.stl; visual mesh filename=package:///tigh_mirror1.stl
- added link tigh_mirror2, mass 0.39199504768219411988; collision mesh filename=package:///tigh_mirror2.stl; visual mesh filename=package:///tigh_mirror2.stl
- added link tigh_mirror2_2, mass 0.39199504768219411988; collision mesh filename=package:///tigh_mirror2.stl; visual mesh filename=package:///tigh_mirror2.stl
- added link universal, mass 0.14303170725627573079; collision mesh filename=package:///universal.stl; visual mesh filename=package:///universal.stl
- added link universal_2, mass 0.14303170725627573079; collision mesh filename=package:///universal.stl; visual mesh filename=package:///universal.stl
Joints:
- removed joint free_cardan4
- added joint free_universal4: type revolute, parent universal_2, child shin_mirror1, origin xyz=0.00029538461538458626876 1.1102230246251565404e-16 -0.00029538461538464177991 rpy=1.5707963267948958919 1.4006235050832673839 1.5707963267948972241, axis 0 0 1, limit effort=1 velocity=20
- joint closedloop1_A_frame: parent tibias_mirror -> shin_mirror1
- joint closedloop1_B_frame: parent tibias_mirror2 -> shin_mirror2
- joint closedloop2_A_frame: parent cuiqqe_22 -> tigh_mirror2
- joint closedloop2_B_frame: parent cuiqqe_2 -> tigh_mirror1
- joint closedloop3_A_frame: parent cuiqqe_22_2 -> tigh_mirror2_2
- joint closedloop3_B_frame: parent cuiqqe_2_2 -> tigh_mirror1_2
- joint foot_frame: parent foot -> foot_part
- joint free_4barlink5: child tibias -> shin; parent cuisse_1 -> tigh_1
- joint free_4barlink6: child tibias_mirror2 -> shin_mirror2; parent cuisse_1_2 -> tigh_1_2
- joint free_hip_x: child bloc_moteur -> motor_2; parent part_9 -> hip_part
- joint free_universal1: child cardan -> universal; parent tibias -> shin
- joint free_universal2: child cheville -> ankle; parent cardan -> universal
- joint hip_frame: parent part_9 -> hip_part
- joint motor_4barlink1: child part_6 -> motor_link; parent bloc_moteur2 -> motor_1
- joint motor_4barlink2: child part_6_2 -> motor_link_2; parent bloc_moteur -> motor_2
- joint motor_4barlink3: child cuisse_1 -> tigh_1; parent bloc_moteur2 -> motor_1
- joint motor_4barlink4: child cuisse_1_2 -> tigh_1_2; parent bloc_moteur -> motor_2
- joint motor_ankle: child foot -> foot_part; parent cheville -> ankle
- joint motor_hip_x: child bloc_moteur2 -> motor_1; parent part_9 -> hip_part
- joint spherical_free_4barlink1: child cuiqqe_22_2 -> tigh_mirror2_2; parent part_6_2 -> motor_link_2
- joint spherical_free_4barlink2: child cuiqqe_22 -> tigh_mirror2; parent part_6 -> motor_link
- joint spherical_free_4barlink3: child cuiqqe_2_2 -> tigh_mirror1_2; parent tibias_mirror2 -> shin_mirror2
- joint spherical_free_4barlink4: child cuiqqe_2 -> tigh_mirror1; parent tibias -> shin
- joint spherical_free_foot: child cardan_2 -> universal_2; parent cheville -> ankle

Commit message: disney modified

File: example_parallel_robots/robots/disney_like/robot.urdf (robot description, URDF)
Before this commit: robot onshape, 26 links, 25 joints
Links:
- added link ankle_int1_2, mass 0.0
- added link ankle_int2_2, mass 0.0
- added link motor_link_2_int1_4, mass 0.0
- added link motor_link_2_int2_4, mass 0.0
- added link motor_link_int1_1, mass 0.0
- added link motor_link_int2_1, mass 0.0
- added link shin_int1_3, mass 0.0
- added link shin_int2_3, mass 0.0
- added link shin_mirror2_int1_5, mass 0.0
- added link shin_mirror2_int2_5, mass 0.0
Joints:
- removed joint spherical_free_4barlink1
- removed joint spherical_free_4barlink2
- removed joint spherical_free_4barlink3
- removed joint spherical_free_4barlink4
- removed joint spherical_free_foot
- added joint ankle_universal_2_rev0: type revolute, parent ankle, child ankle_int1_2, origin xyz=-0.2215384615384614897 1.1102230246251565404e-16 0, axis 1 0 0, limit effort=1 velocity=20
- added joint ankle_universal_2_rev1: type revolute, parent ankle_int1_2, child ankle_int2_2, axis 0 1 0, limit effort=1 velocity=20
- added joint ankle_universal_2_rev2: type revolute, parent ankle_int2_2, child universal_2, axis 0 0 1, limit effort=1 velocity=20
- added joint motor_link_2_tigh_mirror2_2_rev0: type revolute, parent motor_link_2, child motor_link_2_int1_4, origin xyz=0.16410256410256410242 -2.7755575615628913511e-17 -5.5511151231257827021e-17, axis 1 0 0, limit effort=1 velocity=20
- added joint motor_link_2_tigh_mirror2_2_rev1: type revolute, parent motor_link_2_int1_4, child motor_link_2_int2_4, axis 0 1 0, limit effort=1 velocity=20
- added joint motor_link_2_tigh_mirror2_2_rev2: type revolute, parent motor_link_2_int2_4, child tigh_mirror2_2, axis 0 0 1, limit effort=1 velocity=20
- added joint motor_link_tigh_mirror2_rev0: type revolute, parent motor_link, child motor_link_int1_1, origin xyz=0.16410256410256421344 -1.3877787807814456755e-17 -5.5511151231257827021e-17, axis 1 0 0, limit effort=1 velocity=20
- added joint motor_link_tigh_mirror2_rev1: type revolute, parent motor_link_int1_1, child motor_link_int2_1, axis 0 1 0, limit effort=1 velocity=20
- added joint motor_link_tigh_mirror2_rev2: type revolute, parent motor_link_int2_1, child tigh_mirror2, axis 0 0 1, limit effort=1 velocity=20
- added joint shin_mirror2_tigh_mirror1_2_rev0: type revolute, parent shin_mirror2, child shin_mirror2_int1_5, origin xyz=0.12024806843488550223 -0.12907742097056101871 5.5511151231257827021e-17, axis 1 0 0, limit effort=1 velocity=20
- added joint shin_mirror2_tigh_mirror1_2_rev1: type revolute, parent shin_mirror2_int1_5, child shin_mirror2_int2_5, axis 0 1 0, limit effort=1 velocity=20
- added joint shin_mirror2_tigh_mirror1_2_rev2: type revolute, parent shin_mirror2_int2_5, child tigh_mirror1_2, axis 0 0 1, limit effort=1 velocity=20
- added joint shin_tigh_mirror1_rev0: type revolute, parent shin, child shin_int1_3, origin xyz=0.12024806843488550223 0.12907742097056090769 8.3266726846886740532e-17, axis 1 0 0, limit effort=1 velocity=20
- added joint shin_tigh_mirror1_rev1: type revolute, parent shin_int1_3, child shin_int2_3, axis 0 1 0, limit effort=1 velocity=20
- added joint shin_tigh_mirror1_rev2: type revolute, parent shin_int2_3, child tigh_mirror1, axis 0 0 1, limit effort=1 velocity=20
