Commit message: update kangaroo to new standard

File: example_parallel_robots/robots/kangaroo_like/robot.urdf (robot description, URDF)
Before this commit: robot onshape, 66 links, 65 joints
Links:
- removed link attache_hanche
- removed link bout_pied
- removed link cardan_foot
- removed link cardan_foot_2
- removed link cardan_hache
- removed link cardan_hache_2
- removed link centre_hanche
- removed link fermeture0_A
- removed link fermeture0_B
- removed link fermeture10_A
- removed link fermeture10_B
- removed link fermeture11_A
- removed link fermeture11_B
- removed link fermeture1_A
- removed link fermeture1_B
- removed link fermeture2_A
- removed link fermeture2_B
- removed link fermeture3_A
- removed link fermeture3_B
- removed link fermeture4_A
- removed link fermeture4_B
- removed link fermeture5_A
- removed link fermeture5_B
- removed link fermeture6_A
- removed link fermeture6_B
- removed link fermeture7_A
- removed link fermeture7_B
- removed link fermeture8_A
- removed link fermeture8_B
- removed link fermeture9_A
- removed link fermeture9_B
- removed link hanche
- removed link hanche_batis
- removed link moteur_hanche1
- removed link moteur_hanche1_2
- removed link motteur_rotation
- removed link motteur_rotation_2
- removed link motteur_rotation_3
- removed link motteur_rotation_4
- removed link piston
- removed link piston_10
- removed link piston_11
- removed link piston_12
- removed link piston_2
- removed link piston_3
- removed link piston_4
- removed link piston_5
- removed link piston_6
- removed link piston_7
- removed link piston_8
- removed link piston_9
- removed link renvois_cheville
- removed link renvois_cheville_2
- added link closedloop0_A, mass 1e-9
- added link closedloop0_B, mass 1e-9
- added link closedloop10_A, mass 1e-9
- added link closedloop10_B, mass 1e-9
- added link closedloop11_A, mass 1e-9
- added link closedloop11_B, mass 1e-9
- added link closedloop1_A, mass 1e-9
- added link closedloop1_B, mass 1e-9
- added link closedloop2_A, mass 1e-9
- added link closedloop2_B, mass 1e-9
- added link closedloop3_A, mass 1e-9
- added link closedloop3_B, mass 1e-9
- added link closedloop4_A, mass 1e-9
- added link closedloop4_B, mass 1e-9
- added link closedloop5_A, mass 1e-9
- added link closedloop5_B, mass 1e-9
- added link closedloop6_A, mass 1e-9
- added link closedloop6_B, mass 1e-9
- added link closedloop7_A, mass 1e-9
- added link closedloop7_B, mass 1e-9
- added link closedloop8_A, mass 1e-9
- added link closedloop8_B, mass 1e-9
- added link closedloop9_A, mass 1e-9
- added link closedloop9_B, mass 1e-9
- added link cylinder, mass 0.0047041422996690132607; collision mesh filename=package:///cylinder.stl; visual mesh filename=package:///cylinder.stl
- added link cylinder_10, mass 0.0047041422996690132607; collision mesh filename=package:///cylinder.stl; visual mesh filename=package:///cylinder.stl
- added link cylinder_11, mass 0.0047041422996690132607; collision mesh filename=package:///cylinder.stl; visual mesh filename=package:///cylinder.stl
- added link cylinder_12, mass 0.0047041422996690132607; collision mesh filename=package:///cylinder.stl; visual mesh filename=package:///cylinder.stl
- added link cylinder_2, mass 0.0047041422996690132607; collision mesh filename=package:///cylinder.stl; visual mesh filename=package:///cylinder.stl
- added link cylinder_3, mass 0.0047041422996690132607; collision mesh filename=package:///cylinder.stl; visual mesh filename=package:///cylinder.stl
- added link cylinder_4, mass 0.0047041422996690132607; collision mesh filename=package:///cylinder.stl; visual mesh filename=package:///cylinder.stl
- added link cylinder_5, mass 0.0047041422996690132607; collision mesh filename=package:///cylinder.stl; visual mesh filename=package:///cylinder.stl
- added link cylinder_6, mass 0.0047041422996690132607; collision mesh filename=package:///cylinder.stl; visual mesh filename=package:///cylinder.stl
- added link cylinder_7, mass 0.0047041422996690132607; collision mesh filename=package:///cylinder.stl; visual mesh filename=package:///cylinder.stl
- added link cylinder_8, mass 0.0047041422996690132607; collision mesh filename=package:///cylinder.stl; visual mesh filename=package:///cylinder.stl
- added link cylinder_9, mass 0.0047041422996690132607; collision mesh filename=package:///cylinder.stl; visual mesh filename=package:///cylinder.stl
- added link foot_part, mass 0.31091298222930213724; collision mesh filename=package:///foot_part.stl; visual mesh filename=package:///foot_part.stl
- added link hip_center, mass 1e-9
- added link hip_ground, mass 1.5865591647149870358; collision mesh filename=package:///hip_ground.stl; visual mesh filename=package:///hip_ground.stl
- added link hip_part, mass 0.1490882064698049736; collision mesh filename=package:///hip_part.stl; visual mesh filename=package:///hip_part.stl
- added link holder_hip, mass 0.01282947899909727546; collision mesh filename=package:///holder_hip.stl; visual mesh filename=package:///holder_hip.stl
- added link motor_hip1, mass 0.17794962537636810351; collision mesh filename=package:///motor_hip1.stl; visual mesh filename=package:///motor_hip1.stl
- added link motor_hip1_2, mass 0.17794962537636810351; collision mesh filename=package:///motor_hip1.stl; visual mesh filename=package:///motor_hip1.stl
- added link rotation_motor, mass 0.19339251676417062997; collision mesh filename=package:///rotation_motor.stl; visual mesh filename=package:///rotation_motor.stl
- added link rotation_motor_2, mass 0.19339251676417062997; collision mesh filename=package:///rotation_motor.stl; visual mesh filename=package:///rotation_motor.stl
- added link rotation_motor_3, mass 0.19339251676417062997; collision mesh filename=package:///rotation_motor.stl; visual mesh filename=package:///rotation_motor.stl
- added link rotation_motor_4, mass 0.19339251676417062997; collision mesh filename=package:///rotation_motor.stl; visual mesh filename=package:///rotation_motor.stl
- added link transmission_ankle, mass 0.074310321213953561825; collision mesh filename=package:///transmission_ankle.stl; visual mesh filename=package:///transmission_ankle.stl
- added link transmission_ankle2, mass 0.074310320490072731547; collision mesh filename=package:///transmission_ankle2.stl; visual mesh filename=package:///transmission_ankle2.stl
- added link universal_foot, mass 0.0064135211594024193679; collision mesh filename=package:///universal_foot.stl; visual mesh filename=package:///universal_foot.stl
- added link universal_foot_2, mass 0.0064135211594024193679; collision mesh filename=package:///universal_foot.stl; visual mesh filename=package:///universal_foot.stl
- added link universal_hip, mass 0.015608633111865791165; collision mesh filename=package:///universal_hip.stl; visual mesh filename=package:///universal_hip.stl
- added link universal_hip_2, mass 0.015608633111865791165; collision mesh filename=package:///universal_hip.stl; visual mesh filename=package:///universal_hip.stl
- link foot: mass 0.3109129822293019707 -> 1e-9; geometry 
- link part_1: mass 0.48864348852726857686 -> 0.24432174426363428843
- link part_2: mass 0.7961294500674355179 -> 0.39806472503371775895
- link part_3: mass 0.40426961787931336989 -> 0.20213480893965668495
- link part_4: mass 0.022622071159599056733 -> 0.011311035579799526632
- link part_5: mass 0.022214201653533428155 -> 0.011107100826766714077
- link part_6: mass 0.067104419080678087695 -> 0.033552209540339043847
- link part_7: mass 0.062831853071795965016 -> 0.031415926535897982508
- link part_7_2: mass 0.062831853071795965016 -> 0.031415926535897982508
- link part_7_3: mass 0.062831853071795965016 -> 0.031415926535897982508
- link part_7_4: mass 0.062831853071795965016 -> 0.031415926535897982508
- link part_8: mass 0.012408180777254541535 -> 0.0062040903886272707676
- link part_9: mass 0.012408180777254539801 -> 0.0062040903886272699003
Joints:
- removed joint 4barres_genoux
- removed joint bout_pied_frame
- removed joint cardans_foot_haut
- removed joint centre_hanche_frame
- removed joint fermeture0_A_frame
- removed joint fermeture0_B_frame
- removed joint fermeture10_A_frame
- removed joint fermeture10_B_frame
- removed joint fermeture11_A_frame
- removed joint fermeture11_B_frame
- removed joint fermeture1_A_frame
- removed joint fermeture1_B_frame
- removed joint fermeture2_A_frame
- removed joint fermeture2_B_frame
- removed joint fermeture3_A_frame
- removed joint fermeture3_B_frame
- removed joint fermeture4_A_frame
- removed joint fermeture4_B_frame
- removed joint fermeture5_A_frame
- removed joint fermeture5_B_frame
- removed joint fermeture6_A_frame
- removed joint fermeture6_B_frame
- removed joint fermeture7_A_frame
- removed joint fermeture7_B_frame
- removed joint fermeture8_A_frame
- removed joint fermeture8_B_frame
- removed joint fermeture9_A_frame
- removed joint fermeture9_B_frame
- removed joint frame_moeur_genoux
- removed joint frame_moeur_pied1
- removed joint frame_moeur_pied2
- removed joint free_attache_moeur_hanche_1
- removed joint free_attache_moeur_hanche_2
- removed joint free_attache_moeur_hanche_3
- removed joint free_attache_moeur_hanchexy
- removed joint free_attache_moeur_hanchexy2
- removed joint free_cardans_yhips
- removed joint free_cheville_cardanx
- removed joint free_zhips
- removed joint genoux_bas
- removed joint genoux_haut
- removed joint hanche_bas
- removed joint mot_cheville1
- removed joint mot_cheville2
- removed joint mot_genoux
- removed joint mot_hanchexy1
- removed joint mot_hanchexy2
- removed joint mot_hanchez
- removed joint renvois_genoux_1
- removed joint renvois_genoux_2
- removed joint renvois_hanche_1
- removed joint renvois_hanche_2
- removed joint to_rotule_4barres
- removed joint to_rotule_barres_tibias
- removed joint to_rotule_free_attache2_moeur_hanchez
- removed joint to_rotule_free_attache_moeur_hanche_z
- removed joint to_rotule_hanche_bas1
- removed joint to_rotule_hanche_bas2
- removed joint to_rotule_moeur_action_genoux
- removed joint to_rotule_renvois_hanche3
- removed joint to_rotule_renvois_hanche4
- removed joint to_rotule_renvois_hanche_moeur1
- removed joint to_rotule_renvois_hanche_moeur2
- removed joint to_rotule_renvois_pied1
- removed joint to_rotule_renvois_pied2
- added joint 4barlink_knee: type revolute, parent part_2, child part_4, origin xyz=0.046047631733746000049 -0.019483726843523341277 0 rpy=3.141592653589793116 -2.0953369411995213608e-17 -1.2672660179279418013, axis 0 0 1, limit effort=1 velocity=20
- added joint closedloop0_A_frame: type fixed, parent foot_part, child closedloop0_A, origin xyz=-0.054999999999999993339 -0.01100000000000000977 0.038500000000000006439 rpy=1.570796326794896558 7.0549938242594490701e-17 -1.570796326794896558, axis 0 0 0
- added joint closedloop0_B_frame: type fixed, parent part_7, child closedloop0_B, origin xyz=0 0 -0.40000000000000007772 rpy=3.1415926535897913396 1.2983444000664018813e-15 -1.570796326794896558, axis 0 0 0
- added joint closedloop10_A_frame: type fixed, parent part_7_3, child closedloop10_A, origin xyz=0 0 -0.4000000000000000222 rpy=1.4735023840744858996e-16 6.8620917561167023512e-16 -4.2558792724255830793e-16, axis 0 0 0
- added joint closedloop10_B_frame: type fixed, parent transmission_ankle2, child closedloop10_B, origin xyz=-0.035854717888628970246 -0.041706584673488089621 -0.052249999999999963141 rpy=-1.57079632679489678 4.2500725161430664477e-17 -3.7753854610413260056e-16, axis 0 0 0
- added joint closedloop11_A_frame: type fixed, parent foot_part, child closedloop11_A, origin xyz=-0.054999999999999965583 -0.010999999999999898748 -0.038500000000000006439 rpy=1.570796326794896558 7.0549938242594490701e-17 -1.570796326794896558, axis 0 0 0
- added joint closedloop11_B_frame: type fixed, parent part_7_2, child closedloop11_B, origin xyz=0 2.7755575615628913511e-17 -0.39999999999999996669 rpy=3.1415926535897895633 -3.9070079812038025555e-16 1.570796326794896558, axis 0 0 0
- added joint closedloop1_A_frame: type fixed, parent cylinder_7, child closedloop1_A, origin xyz=0 0 -0.02200000000000001954 rpy=-2.7819127417443369016e-15 4.1538050120666868689e-17 -7.0215725374297579137e-17, axis 0 0 0
- added joint closedloop1_B_frame: type fixed, parent cylinder_4, child closedloop1_B, origin xyz=-5.5511151231257827021e-17 -5.5511151231257827021e-17 -0.02200000000000001954 rpy=-3.1415926535897904515 2.0111125192863830092e-15 -1.570796326794896336, axis 0 0 0
- added joint closedloop2_A_frame: type fixed, parent cylinder_8, child closedloop2_A, origin xyz=-1.3877787807814456755e-17 -2.7755575615628913511e-17 -0.021999999999999880762 rpy=-1.3082333062209864418e-15 3.1484991343763797587e-15 5.5969162711631674861e-17, axis 0 0 0
- added joint closedloop2_B_frame: type fixed, parent cylinder_5, child closedloop2_B, origin xyz=2.7755575615628913511e-17 0 -0.02200000000000001954 rpy=3.1415926535897917837 3.0726606491544917811e-15 -1.570796326794896558, axis 0 0 0
- added joint closedloop3_A_frame: type fixed, parent cylinder, child closedloop3_A, origin xyz=2.7755575615628913511e-17 -5.5511151231257827021e-17 -0.021999999999999964029 rpy=-3.141592653589793116 -1.4810179096329776666e-15 -2.2307564621250647706e-17, axis 0 0 0
- added joint closedloop3_B_frame: type fixed, parent cylinder_10, child closedloop3_B, origin xyz=2.7755575615628913511e-17 -5.5511151231257827021e-17 -0.021999999999999964029 rpy=-3.7983807026823699256e-15 -3.1724293295329463046e-16 -2.1021659879463730673e-17, axis 0 0 0
- added joint closedloop4_A_frame: type fixed, parent cylinder_2, child closedloop4_A, origin xyz=-2.7755575615628913511e-17 2.7755575615628913511e-17 -0.021999999999999991784 rpy=-3.1415926535897895633 -5.9339792050261044152e-14 -2.0808136697909534971e-18, axis 0 0 0
- added joint closedloop4_B_frame: type fixed, parent cylinder_9, child closedloop4_B, origin xyz=0 0 -0.021999999999999866884 rpy=-5.2342383182449044881e-14 8.2074296634245360986e-15 1.4117770487744005312e-18, axis 0 0 0
- added joint closedloop5_A_frame: type fixed, parent cylinder_12, child closedloop5_A, origin xyz=0 0 -0.021999999999999943212 rpy=4.0939474033053051719e-16 2.1380466841413257505e-16 6.2026386493102164692e-16, axis 0 0 0
- added joint closedloop5_B_frame: type fixed, parent cylinder_11, child closedloop5_B, origin xyz=-2.7755575615628913511e-17 -1.3877787807814456755e-17 -0.022000000000000054234 rpy=3.1415926535897917837 9.3675067702748754064e-17 -1.570796326794896558, axis 0 0 0
- added joint closedloop6_A_frame: type fixed, parent part_4, child closedloop6_A, origin xyz=0.038967453687049763422 -0.092095263467496704668 0 rpy=1.570796326794896558 -5.7748320244677594273e-24 -1.570796326794896336, axis 0 0 0
- added joint closedloop6_B_frame: type fixed, parent part_6, child closedloop6_B, origin xyz=5.5511151231257827021e-17 5.5511151231257827021e-17 -0.42720000000000002416 rpy=-3.1415926535897926719 3.4737141109842255094e-16 -3.141592653589793116, axis 0 0 0
- added joint closedloop7_A_frame: type fixed, parent part_5, child closedloop7_A, origin xyz=0 5.5511151231257827021e-17 -0.14141999999999999016 rpy=-3.141592653589793116 -1.2232281396413594261e-16 1.505751559102670748e-16, axis 0 0 0
- added joint closedloop7_B_frame: type fixed, parent part_1, child closedloop7_B, origin xyz=0.083867056794542357845 -0.0077119035015027481705 -0.071500000000000035749 rpy=1.570796326794896558 -2.1742890467508124463e-30 -1.3975154895155261838e-14, axis 0 0 0
- added joint closedloop8_A_frame: type fixed, parent cylinder_3, child closedloop8_A, origin xyz=0 5.5511151231257827021e-17 -0.022000000000000213829 rpy=-3.141592653589793116 -6.0722954362721615853e-17 -1.570796326794896336, axis 0 0 0
- added joint closedloop8_B_frame: type fixed, parent cylinder_6, child closedloop8_B, origin xyz=5.5511151231257827021e-17 1.4745149545802860303e-17 -0.022000000000000061173 rpy=9.260101808175594684e-16 -6.0667578152815541166e-16 1.5707963267948974462, axis 0 0 0
- added joint closedloop9_A_frame: type fixed, parent part_7_4, child closedloop9_A, origin xyz=0 -8.3266726846886740532e-17 -0.4000000000000000222 rpy=-2.3952719085374775399e-15 -9.8359338965770896915e-16 -1.5707963267948972241, axis 0 0 0
- added joint closedloop9_B_frame: type fixed, parent transmission_ankle, child closedloop9_B, origin xyz=-0.035854717888629011879 -0.041706584673488200643 0.052249999999999990896 rpy=1.570796326794896558 -3.2748092031556818832e-31 -3.1415926535897913396, axis 0 0 0
- added joint foot_frame: type fixed, parent foot_part, child foot, origin xyz=0.012016949221079820109 0.038499999999999978684 6.8117394502742456552e-09 rpy=1.5707963267948972241 1.0529999139445015132e-16 9.3156790618841999074e-16, axis 0 0 0
- added joint frame_motor_foot1: type revolute, parent part_1, child rotation_motor_2, origin xyz=0.054086706326755197571 0.014047405294960763067 -0.118249999999999994 rpy=-1.570796326794896558 0.70569698106852796204 0.2858933777993261649, axis 0 0 1, limit effort=1 velocity=20
- added joint frame_motor_foot2: type revolute, parent part_1, child rotation_motor_3, origin xyz=0.054086706326755190632 0.014047405294960790823 -0.024749999999999966471 rpy=1.570796326794896558 -0.16946695988620705253 -2.8556992757904748892, axis 0 0 1, limit effort=1 velocity=20
- added joint frame_motor_knee: type revolute, parent part_2, child rotation_motor, origin xyz=-0.061655078133537342955 -0.018724201373191751152 4.2972847502653621632e-12 rpy=-1.5707963267948970021 1.2771385194773068328 -0.60601731071218267743, axis 0 0 1, limit effort=1 velocity=20
- added joint free_ankle_universalx: type revolute, parent universal_foot_2, child foot_part, origin xyz=6.6000000000010494716e-05 1.1102230246251565404e-16 6.5999999999954983565e-05 rpy=1.5707963267949303088 -1.5331629223910492321 1.570796326794896336, axis 0 0 1, limit effort=1 velocity=20
- added joint free_motor_holder_hip_1: type revolute, parent hip_part, child universal_hip, origin xyz=0.012500000000000035388 -0.037124999999999769296 -0.077000000000000096145 rpy=1.57079632679489678 -0.020021707956276633966 -1.5707963267948994446, axis 0 0 1, limit effort=1 velocity=20
- added joint free_motor_holder_hip_2: type revolute, parent hip_ground, child holder_hip, origin xyz=-0.10299999999999821798 0.24350000000000304734 0 rpy=-1.0047518372857614626e-14 7.4933038271172496209e-15 3.1415926535897793492, axis 0 0 1, limit effort=1 velocity=20
- added joint free_motor_holder_hip_3: type revolute, parent hip_part, child universal_hip_2, origin xyz=0.012499999999999965999 0.037125000000000268896 -0.077000000000000956568 rpy=-1.570796326794896558 -0.018188083207083823034 1.5707963267948941155, axis 0 0 1, limit effort=1 velocity=20
- added joint free_motor_holder_hip_xy1: type revolute, parent universal_hip_2, child motor_hip1_2, origin xyz=5.5511151231257827021e-17 -2.7755575615628913511e-17 -0.055000000000000007216 rpy=-1.5707963267948972241 1.5002236252432261665 1.5707963267949194286, axis 0 0 1, limit effort=1 velocity=20
- added joint free_motor_holder_hip_xy2: type revolute, parent universal_hip, child motor_hip1, origin xyz=-5.5511151231257827021e-17 -1.9428902930940239457e-16 -0.054999999999999979461 rpy=-1.570796326794866804 -1.5002260895475847402 1.5707963267948659158, axis 0 0 1, limit effort=1 velocity=20
- added joint free_universal_yhip: type revolute, parent hip_part, child universal_foot, origin xyz=-1.7347234759768070944e-18 0 -0.1649999999999999245 rpy=1.570796326794896558 -9.6290805123406329139e-15 -1.5707963267948992225, axis 0 0 1, limit effort=1 velocity=20
- added joint free_zhip: type revolute, parent hip_ground, child hip_part, origin xyz=0.012500000000000170697 0.20500000000000265232 -0.0050000000000000044409 rpy=1.0057557210906877445e-14 -7.6592250448352642693e-15 2.7755575615630239783e-16, axis 0 0 1, limit effort=1 velocity=20
- added joint hip_center_frame: type fixed, parent hip_ground, child hip_center, origin xyz=-0.0047474699228997607747 0.28861143158345337056 -0.17250000000000290101 rpy=2.6505726415425557215e-28 -8.3196567936654447285e-16 -1.1492717312938456553e-28, axis 0 0 0
- added joint hip_transmission_1: type revolute, parent part_1, child part_8, origin xyz=-6.9388939039072283776e-17 0.046751999999999988011 -0.087999999999999994893 rpy=7.0625044874992382189e-15 -6.8120459426221159297e-15 1.0736013892061464503, axis 0 0 1, limit effort=1 velocity=20
- added joint hip_transmission_2: type revolute, parent part_1, child part_9, origin xyz=-6.2450045135165055399e-17 0.046751999999999988011 -0.055000000000000021094 rpy=-3.1415926535897860106 -7.0534351170114349528e-15 1.0500864465451529295, axis 0 0 1, limit effort=1 velocity=20
- added joint knee_transmission_1: type revolute, parent part_2, child transmission_ankle2, origin xyz=-0.21747050071615148248 -0.33571800862966283407 0.0099999999999999533706 rpy=3.1415926535897926719 2.3487564121428828494e-15 3.0459021140380468928, axis 0 0 1, limit effort=1 velocity=20
- added joint knee_transmission_2: type revolute, parent part_2, child transmission_ankle, origin xyz=-0.21747050071615170452 -0.33571800862966272305 -0.010000000000000064393 rpy=3.141592653589793116 2.1953367209117600024e-15 3.0659322643825968058, axis 0 0 1, limit effort=1 velocity=20
- added joint lower_hip: type revolute, parent universal_foot, child part_1, origin xyz=6.6000000000010494716e-05 -8.3266726846886740532e-17 -6.5999999999998351652e-05 rpy=1.5707963267949149877 -1.4738036229882285344 1.5707963267948861219, axis 0 0 1, limit effort=1 velocity=20
- added joint lower_knee: type revolute, parent part_2, child part_3, origin xyz=-0.21747050071615151023 -0.33571800862966272305 5.5511151231257827021e-17 rpy=-1.7726512667869372285e-16 -4.9802783514596252578e-17 0.89630439304597708805, axis 0 0 1, limit effort=1 velocity=20
- added joint motor_ankle1: type prismatic, parent rotation_motor_3, child cylinder_8, origin xyz=9.7144514654701197287e-17 1.6653345369377348106e-16 0.048590062929759286758 rpy=3.141592653589793116 6.5278587787792881949e-16 3.1415926535897922278, axis 0 0 1, limit effort=1 velocity=20
- added joint motor_ankle2: type prismatic, parent rotation_motor_2, child cylinder_7, origin xyz=-5.5511151231257827021e-17 -8.3266726846886740532e-17 0.051330395129961847722 rpy=3.141592653589793116 1.8208947195106360443e-14 3.1415926535897815697, axis 0 0 1, limit effort=1 velocity=20
- added joint motor_hip_xy1: type prismatic, parent motor_hip1, child cylinder_9, origin xyz=4.1633363423443370266e-17 -0.050156290972289171992 -4.1633363423443370266e-16 rpy=-1.5707963267949502928 -8.1160902808362363988e-15 5.5693133426199995086e-15, axis 0 0 1, limit effort=1 velocity=20
- added joint motor_hip_xy2: type prismatic, parent motor_hip1_2, child cylinder_10, origin xyz=1.3877787807814456755e-17 -0.050153775555251425833 3.6082248300317587564e-16 rpy=-1.5707963267948996666 2.6021963268559055545e-15 1.4416055078510302742e-15, axis 0 0 1, limit effort=1 velocity=20
- added joint motor_hipz: type prismatic, parent rotation_motor_4, child cylinder_12, origin xyz=-1.0547118733938987134e-15 -8.7430063189231077558e-16 -0.071500000000001451284 rpy=-2.1233015345958489363e-15 4.1282117760629273878e-17 -1.5707963267949134334, axis 0 0 1, limit effort=1 velocity=20
- added joint motor_knee: type prismatic, parent rotation_motor, child cylinder_3, origin xyz=-2.7755575615628913511e-17 2.7755575615628913511e-17 -0.022568234725387908979 rpy=3.141592653589793116 1.6075711619745091793e-15 -4.0446422624590046478e-15, axis 0 0 1, limit effort=1 velocity=20
- added joint sherical_4bar: type revolute, parent part_4, child part_5, origin xyz=0.019483726843524923344 -0.046047631733748387028 0 rpy=-1.57079632679489678 0.033617431841822156824 -1.5707963267948954478, axis 0 0 1, limit effort=1 velocity=20
- added joint spherical_lower_hip1: type revolute, parent part_1, child cylinder, origin xyz=-0.060500000000000039857 -1.9428902930940239457e-16 -0.03850000000000006195 rpy=1.57079632679489678 -0.083114644637935983229 -3.141592653589783346, axis 0 0 1, limit effort=1 velocity=20
- added joint spherical_lower_hip2: type revolute, parent part_1, child cylinder_2, origin xyz=-0.060499999999999998224 -5.5511151231257827021e-17 0.038500000000000006439 rpy=-1.57079632679489678 0.090109706454319454805 -5.2162867703289486806e-14, axis 0 0 1, limit effort=1 velocity=20
- added joint spherical_motor_holder_1_hip_z: type revolute, parent holder_hip, child rotation_motor_4, origin xyz=1.3877787807814456755e-17 2.7755575615628913511e-17 -0.051749999999999775346 rpy=1.5707963267948976682 -0.051824161433128575205 1.5707963267948943376, axis 0 0 1, limit effort=1 velocity=20
- added joint spherical_motor_holder_2_hip_z: type revolute, parent hip_part, child cylinder_11, origin xyz=3.2508717939805364949e-15 0.038500000000000034195 -0.046750000000000013767 rpy=1.570796326794896558 0.051824161433129206644 1.5707963267948945596, axis 0 0 1, limit effort=1 velocity=20
- added joint spherical_motor_transmission_hip1: type revolute, parent part_8, child cylinder_4, origin xyz=0.043531328479973735446 0.0032046566522409281053 -0.025000000000000077716 rpy=-1.57079632679489678 -1.2175171882697088943 -1.3995157029259762656e-14, axis 0 0 1, limit effort=1 velocity=20
- added joint spherical_motor_transmission_hip2: type revolute, parent part_9, child cylinder_5, origin xyz=0.043531328479973624423 -0.003204656652241011372 -0.024999999999999994449 rpy=-1.570796326794896336 -1.3137217724347107772 -3.1415926535897784611, axis 0 0 1, limit effort=1 velocity=20
- added joint spherical_shin: type revolute, parent part_3, child part_6, origin xyz=0.038967453687049680155 -0.092095263467496885079 -1.1102230246251565404e-16 rpy=-1.57079632679489678 -1.2130896351314029502e-15 1.5707963267948972241, axis 0 0 1, limit effort=1 velocity=20
- added joint spherical_transmission_foot1: type revolute, parent transmission_ankle, child part_7_2, origin xyz=-0.059494699261975675375 0.010983203527527130028 0.021999999999999964029 rpy=1.570796326794896558 -4.2017171180584709161e-17 1.57079632679489678, axis 0 0 1, limit effort=1 velocity=20
- added joint spherical_transmission_foot2: type revolute, parent transmission_ankle2, child part_7, origin xyz=-0.059494699261975494964 0.01098320352752724105 -0.021999999999999964029 rpy=-1.57079632679489678 4.0432982165859767957e-17 -1.5707963267948972241, axis 0 0 1, limit effort=1 velocity=20
- added joint spherical_transmission_hip3: type revolute, parent part_8, child part_7_3, origin xyz=0.041074543378118888448 0.036577067764912846171 -0.0050000000000000044409 rpy=-1.570796326794896558 0.088927611054569727367 -3.1415926535897917837, axis 0 0 1, limit effort=1 velocity=20
- added joint spherical_transmission_hip4: type revolute, parent part_9, child part_7_4, origin xyz=0.041074543378118943959 -0.036577067764912957193 -0.0050000000000000044409 rpy=1.5707963267948972241 1.4581066266007887133 3.1415926535897527039, axis 0 0 1, limit effort=1 velocity=20
- added joint spherical_transmission_knee: type revolute, parent part_1, child cylinder_6, origin xyz=-0.013749999999999946293 0.0024999999999999744649 -0.072000000000000036193 rpy=-1.57079632679489678 -0.99860729712136064862 -1.5707963267949054398, axis 0 0 1, limit effort=1 velocity=20
- added joint universal_foot_up: type revolute, parent part_3, child universal_foot_2, origin xyz=0.2174705007161493453 -0.33571800862966416634 0 rpy=-1.5707963267948972241 -1.4835298641951775167 1.5707963267949347497, axis 0 0 1, limit effort=1 velocity=20
- added joint upper_knee: type revolute, parent part_1, child part_2, origin xyz=-6.5919492087118669588e-17 0.046751999999999988011 -0.07150000000000009126 rpy=-3.1415926535897855665 -5.4851651532674043147e-15 0.72447699933333153943, axis 0 0 1, limit effort=1 velocity=20
