Commit message: kangaroo modified

File: example_parallel_robots/robots/kangaroo_like/robot.urdf (robot description, URDF)
Before this commit: robot onshape, 66 links, 65 joints
Links:
- added link hip_part_int1_11, mass 0.0
- added link hip_part_int2_11, mass 0.0
- added link holder_hip_int1_12, mass 0.0
- added link holder_hip_int2_12, mass 0.0
- added link part_1_int1_1, mass 0.0
- added link part_1_int1_10, mass 0.0
- added link part_1_int1_2, mass 0.0
- added link part_1_int2_1, mass 0.0
- added link part_1_int2_10, mass 0.0
- added link part_1_int2_2, mass 0.0
- added link part_3_int1_3, mass 0.0
- added link part_3_int2_3, mass 0.0
- added link part_8_int1_6, mass 0.0
- added link part_8_int1_7, mass 0.0
- added link part_8_int2_6, mass 0.0
- added link part_8_int2_7, mass 0.0
- added link part_9_int1_8, mass 0.0
- added link part_9_int1_9, mass 0.0
- added link part_9_int2_8, mass 0.0
- added link part_9_int2_9, mass 0.0
- added link transmission_ankle2_int1_4, mass 0.0
- added link transmission_ankle2_int2_4, mass 0.0
- added link transmission_ankle_int1_5, mass 0.0
- added link transmission_ankle_int2_5, mass 0.0
Joints:
- removed joint spherical_lower_hip1
- removed joint spherical_lower_hip2
- removed joint spherical_motor_holder_1_hip_z
- removed joint spherical_motor_holder_2_hip_z
- removed joint spherical_motor_transmission_hip1
- removed joint spherical_motor_transmission_hip2
- removed joint spherical_shin
- removed joint spherical_transmission_foot1
- removed joint spherical_transmission_foot2
- removed joint spherical_transmission_hip3
- removed joint spherical_transmission_hip4
- removed joint spherical_transmission_knee
- added joint hip_part_cylinder_11_rev0: type revolute, parent hip_part, child hip_part_int1_11, origin xyz=3.2508717939805364949e-15 0.038500000000000034195 -0.046750000000000013767, axis 1 0 0, limit effort=1 velocity=20
- added joint hip_part_cylinder_11_rev1: type revolute, parent hip_part_int1_11, child hip_part_int2_11, axis 0 1 0, limit effort=1 velocity=20
- added joint hip_part_cylinder_11_rev2: type revolute, parent hip_part_int2_11, child cylinder_11, axis 0 0 1, limit effort=1 velocity=20
- added joint holder_hip_rotation_motor_4_rev0: type revolute, parent holder_hip, child holder_hip_int1_12, origin xyz=1.3877787807814456755e-17 2.7755575615628913511e-17 -0.051749999999999775346, axis 1 0 0, limit effort=1 velocity=20
- added joint holder_hip_rotation_motor_4_rev1: type revolute, parent holder_hip_int1_12, child holder_hip_int2_12, axis 0 1 0, limit effort=1 velocity=20
- added joint holder_hip_rotation_motor_4_rev2: type revolute, parent holder_hip_int2_12, child rotation_motor_4, axis 0 0 1, limit effort=1 velocity=20
- added joint part_1_cylinder_2_rev0: type revolute, parent part_1, child part_1_int1_2, origin xyz=-0.060499999999999998224 -5.5511151231257827021e-17 0.038500000000000006439, axis 1 0 0, limit effort=1 velocity=20
- added joint part_1_cylinder_2_rev1: type revolute, parent part_1_int1_2, child part_1_int2_2, axis 0 1 0, limit effort=1 velocity=20
- added joint part_1_cylinder_2_rev2: type revolute, parent part_1_int2_2, child cylinder_2, axis 0 0 1, limit effort=1 velocity=20
- added joint part_1_cylinder_6_rev0: type revolute, parent part_1, child part_1_int1_10, origin xyz=-0.013749999999999946293 0.0024999999999999744649 -0.072000000000000036193, axis 1 0 0, limit effort=1 velocity=20
- added joint part_1_cylinder_6_rev1: type revolute, parent part_1_int1_10, child part_1_int2_10, axis 0 1 0, limit effort=1 velocity=20
- added joint part_1_cylinder_6_rev2: type revolute, parent part_1_int2_10, child cylinder_6, axis 0 0 1, limit effort=1 velocity=20
- added joint part_1_cylinder_rev0: type revolute, parent part_1, child part_1_int1_1, origin xyz=-0.060500000000000039857 -1.9428902930940239457e-16 -0.03850000000000006195, axis 1 0 0, limit effort=1 velocity=20
- added joint part_1_cylinder_rev1: type revolute, parent part_1_int1_1, child part_1_int2_1, axis 0 1 0, limit effort=1 velocity=20
- added joint part_1_cylinder_rev2: type revolute, parent part_1_int2_1, child cylinder, axis 0 0 1, limit effort=1 velocity=20
- added joint part_3_part_6_rev0: type revolute, parent part_3, child part_3_int1_3, origin xyz=0.038967453687049680155 -0.092095263467496885079 -1.1102230246251565404e-16, axis 1 0 0, limit effort=1 velocity=20
- added joint part_3_part_6_rev1: type revolute, parent part_3_int1_3, child part_3_int2_3, axis 0 1 0, limit effort=1 velocity=20
- added joint part_3_part_6_rev2: type revolute, parent part_3_int2_3, child part_6, axis 0 0 1, limit effort=1 velocity=20
- added joint part_8_cylinder_4_rev0: type revolute, parent part_8, child part_8_int1_6, origin xyz=0.043531328479973735446 0.0032046566522409281053 -0.025000000000000077716, axis 1 0 0, limit effort=1 velocity=20
- added joint part_8_cylinder_4_rev1: type revolute, parent part_8_int1_6, child part_8_int2_6, axis 0 1 0, limit effort=1 velocity=20
- added joint part_8_cylinder_4_rev2: type revolute, parent part_8_int2_6, child cylinder_4, axis 0 0 1, limit effort=1 velocity=20
- added joint part_8_part_7_3_rev0: type revolute, parent part_8, child part_8_int1_7, origin xyz=0.041074543378118888448 0.036577067764912846171 -0.0050000000000000044409, axis 1 0 0, limit effort=1 velocity=20
- added joint part_8_part_7_3_rev1: type revolute, parent part_8_int1_7, child part_8_int2_7, axis 0 1 0, limit effort=1 velocity=20
- added joint part_8_part_7_3_rev2: type revolute, parent part_8_int2_7, child part_7_3, axis 0 0 1, limit effort=1 velocity=20
- added joint part_9_cylinder_5_rev0: type revolute, parent part_9, child part_9_int1_8, origin xyz=0.043531328479973624423 -0.003204656652241011372 -0.024999999999999994449, axis 1 0 0, limit effort=1 velocity=20
- added joint part_9_cylinder_5_rev1: type revolute, parent part_9_int1_8, child part_9_int2_8, axis 0 1 0, limit effort=1 velocity=20
- added joint part_9_cylinder_5_rev2: type revolute, parent part_9_int2_8, child cylinder_5, axis 0 0 1, limit effort=1 velocity=20
- added joint part_9_part_7_4_rev0: type revolute, parent part_9, child part_9_int1_9, origin xyz=0.041074543378118943959 -0.036577067764912957193 -0.0050000000000000044409, axis 1 0 0, limit effort=1 velocity=20
- added joint part_9_part_7_4_rev1: type revolute, parent part_9_int1_9, child part_9_int2_9, axis 0 1 0, limit effort=1 velocity=20
- added joint part_9_part_7_4_rev2: type revolute, parent part_9_int2_9, child part_7_4, axis 0 0 1, limit effort=1 velocity=20
- added joint transmission_ankle2_part_7_rev0: type revolute, parent transmission_ankle2, child transmission_ankle2_int1_4, origin xyz=-0.059494699261975494964 0.01098320352752724105 -0.021999999999999964029, axis 1 0 0, limit effort=1 velocity=20
- added joint transmission_ankle2_part_7_rev1: type revolute, parent transmission_ankle2_int1_4, child transmission_ankle2_int2_4, axis 0 1 0, limit effort=1 velocity=20
- added joint transmission_ankle2_part_7_rev2: type revolute, parent transmission_ankle2_int2_4, child part_7, axis 0 0 1, limit effort=1 velocity=20
- added joint transmission_ankle_part_7_2_rev0: type revolute, parent transmission_ankle, child transmission_ankle_int1_5, origin xyz=-0.059494699261975675375 0.010983203527527130028 0.021999999999999964029, axis 1 0 0, limit effort=1 velocity=20
- added joint transmission_ankle_part_7_2_rev1: type revolute, parent transmission_ankle_int1_5, child transmission_ankle_int2_5, axis 0 1 0, limit effort=1 velocity=20
- added joint transmission_ankle_part_7_2_rev2: type revolute, parent transmission_ankle_int2_5, child part_7_2, axis 0 0 1, limit effort=1 velocity=20
