Commit message: debug kangaroo

File: example_parallel_robots/robots/kangaroo_like_2legs/robot.urdf (robot description, URDF)
Before this commit: robot onshape, 131 links, 130 joints
Links:
- link foot: mass 0.3109129822293019707 -> 0.31091298222930185968
- link foot_2: mass 0.3109129822293019707 -> 0.31091298222930185968
- link hanche_batis_gauche: mass 1.5865591647149872578 -> 1.5865591647149870358
- link moteur_hanche1: mass 0.17794962537636810351 -> 0.17794962537636813127
- link moteur_hanche1_2: mass 0.17794962537636810351 -> 0.17794962537636813127
- link moteur_hanche1_3: mass 0.17794962537636810351 -> 0.17794962537636813127
- link moteur_hanche1_4: mass 0.17794962537636810351 -> 0.17794962537636813127
- link part_1: mass 0.24432174426363423292 -> 0.24432174426363428843
- link part_2: mass 0.39806472503371786997 -> 0.39806472503371781446
- link part_2_2: mass 0.39806472503371786997 -> 0.39806472503371781446
- link part_3: mass 0.20213480893965668495 -> 0.2021348089396567127
- link part_3_2: mass 0.20213480893965668495 -> 0.2021348089396567127
- link part_4: mass 0.011311035579799526632 -> 0.011311035579799528367
- link part_4_2: mass 0.011311035579799526632 -> 0.011311035579799528367
- link part_9: mass 0.0062040903886272707676 -> 0.0062040903886272699003
- link part_9_2: mass 0.0062040903886272707676 -> 0.0062040903886272699003
