Commit message: new initial conf

File: example_parallel_robots/robots/kangaroo_like_2legs/robot.urdf (robot description, URDF)
Before this commit: robot onshape, 131 links, 130 joints
Links:
- link cardan_foot: mass 0.0064135211594024202353 -> 0.0064135211594024193679
- link cardan_foot_2: mass 0.0064135211594024202353 -> 0.0064135211594024193679
- link cardan_foot_3: mass 0.0064135211594024202353 -> 0.0064135211594024193679
- link cardan_foot_4: mass 0.0064135211594024202353 -> 0.0064135211594024193679
- link foot: mass 0.31091298222930185968 -> 0.3109129822293019707
- link foot_2: mass 0.31091298222930185968 -> 0.3109129822293019707
- link hanche_batis: mass 1.5865591647149870358 -> 1.5865591647149872578
- link moteur_hanche1: mass 0.17794962537636813127 -> 0.17794962537636810351
- link moteur_hanche1_2: mass 0.17794962537636813127 -> 0.17794962537636810351
- link moteur_hanche1_3: mass 0.17794962537636813127 -> 0.17794962537636810351
- link moteur_hanche1_4: mass 0.17794962537636813127 -> 0.17794962537636810351
- link motteur_rotation: mass 0.19339251676417060222 -> 0.19339251676417062997
- link motteur_rotation_2: mass 0.19339251676417060222 -> 0.19339251676417062997
- link motteur_rotation_3: mass 0.19339251676417060222 -> 0.19339251676417062997
- link motteur_rotation_4: mass 0.19339251676417060222 -> 0.19339251676417062997
- link motteur_rotation_5: mass 0.19339251676417060222 -> 0.19339251676417062997
- link motteur_rotation_6: mass 0.19339251676417060222 -> 0.19339251676417062997
- link motteur_rotation_7: mass 0.19339251676417060222 -> 0.19339251676417062997
- link motteur_rotation_8: mass 0.19339251676417060222 -> 0.19339251676417062997
- link part_1_gauche: mass 0.24432174482850427255 -> 0.24432174482850421704
- link part_4: mass 0.011311035579799528367 -> 0.011311035579799526632
- link part_4_2: mass 0.011311035579799528367 -> 0.011311035579799526632
- link part_8: mass 0.0062040903886272725024 -> 0.0062040903886272707676
- link part_8_2: mass 0.0062040903886272725024 -> 0.0062040903886272707676
- link renvois_cheville: mass 0.074310321213953547947 -> 0.074310321213953561825
- link renvois_cheville_2: mass 0.074310321213953547947 -> 0.074310321213953561825
Joints:
- joint 4rod_knee: origin xyz=0.046047631733745958416 -0.019483726843523313521 -1.1102230246251565404e-16 rpy=3.141592653589793116 2.0222300709208235426e-16 -1.2672660179279322534 -> xyz=0.046047631733745986171 -0.019483726843523341277 -1.1102230246251565404e-16 rpy=3.141592653589793116 2.0222300709208235426e-16 -1.2672660179279322534
- joint 4rof_knee_left: origin xyz=0.046047631733746000049 -0.019483726843523313521 -1.7347234759768070944e-17 rpy=3.141592653589793116 4.5795419413634097813e-17 -0.96785189103621938056 -> xyz=0.04604763173374580576 -0.01948372684352350781 7.6327832942979512154e-17 rpy=3.141592653589793116 4.4057711130820799237e-17 -1.2499268310990352404
- joint closedloop0_A_3D_frame: origin xyz=-0.054999999999999715783 -0.010999999999999843237 0.038500000000000006439 rpy=1.570796326794896558 6.2711683153062856565e-17 -1.5707963267948958919 -> xyz=-0.054999999999999882316 -0.01100000000000000977 0.038500000000000006439 rpy=1.570796326794896558 6.2711683153062856565e-17 -1.5707963267948958919
- joint closedloop0_B_3D_frame: origin xyz=-1.1102230246251565404e-16 5.5511151231257827021e-17 -0.40000000000000007772 rpy=3.1415926535897913396 1.3110944058270872971e-15 -1.570796326794896558 -> xyz=0 -5.5511151231257827021e-17 -0.40000000000000007772 rpy=3.1415926535897913396 1.3110944058270872971e-15 -1.570796326794896558
- joint closedloop10_A_3D_frame: origin xyz=-8.6736173798840354721e-17 -1.1102230246251565404e-16 -0.40000000000000007772 rpy=1.4121142989576800076e-16 6.455226355074138767e-16 -4.8615344150257609708e-16 -> xyz=-2.5695591487906455086e-17 0 -0.4000000000000000222 rpy=1.4121142989576800076e-16 6.455226355074138767e-16 -4.8615344150257609708e-16
- joint closedloop10_B_3D_frame: origin xyz=-0.035854717888629136779 -0.041706584673488200643 -0.052249999999999963141 rpy=-1.57079632679489678 4.2500725161430485751e-17 -2.5782405335516153514e-16 -> xyz=-0.03585471788862894249 -0.041706584673488089621 -0.052249999999999963141 rpy=-1.57079632679489678 4.2500725161430485751e-17 -2.5782405335516153514e-16
- joint closedloop11_A_3D_frame: origin xyz=-0.054999999999999826805 -0.010999999999999954259 -0.038500000000000034195 rpy=1.570796326794896558 6.2711683153062856565e-17 -1.5707963267948958919 -> xyz=-0.054999999999999826805 -0.01100000000000000977 -0.038500000000000006439 rpy=1.570796326794896558 6.2711683153062856565e-17 -1.5707963267948958919
- joint closedloop11_B_3D_frame: origin xyz=0 1.3877787807814456755e-17 -0.40000000000000013323 rpy=3.1415926535897895633 -3.5435748969399307641e-16 1.570796326794896558 -> xyz=0 2.7755575615628913511e-17 -0.40000000000000013323 rpy=3.1415926535897895633 -3.5435748969399307641e-16 1.570796326794896558
- joint closedloop12_B_3D_frame: origin xyz=0.038967453687049735667 -0.09209526346749669079 -6.9388939039072283776e-18 rpy=-1.57079632679489678 -6.0039660859700073265e-22 -3.141592653589793116 -> xyz=0.038967453687049680155 -0.092095263467496718546 3.8163916471489756077e-17 rpy=-1.57079632679489678 1.342843395992826004e-18 3.141592653589793116
- joint closedloop13_A_3D_frame: origin xyz=-1.3877787807814456755e-17 -3.4694469519536141888e-18 -0.14141999999999999016 rpy=-3.141592653589793116 1.2734996606920880132e-19 8.5029346353481308663e-18 -> xyz=0 8.6736173798840354721e-19 -0.14142000000000001791 rpy=3.141592653589793116 4.0907557778710928219e-17 -5.6977393277845192855e-18
- joint closedloop13_B_3D_frame: origin xyz=0.083867056794542482745 0.0077119035015027481705 -0.071500000000000007994 rpy=1.570796326794896558 2.8360520648029955147e-19 -3.141592653589793116 -> xyz=0.083867056794542510501 0.007711903501502720415 -0.071500000000000021871 rpy=1.570796326794896558 -3.7484973866353497179e-19 3.141592653589793116
- joint closedloop14_A_6D_frame: origin xyz=-6.9388939039072283776e-18 0 -0.022000000000000033418 rpy=-3.141592653589793116 8.9294959238987079639e-17 -1.570796326794896558 -> xyz=2.0816681711721685133e-17 -2.7755575615628913511e-17 -0.022000000000000088929 rpy=-3.141592653589793116 -1.0072885720893678228e-17 -1.570796326794896558
- joint closedloop14_B_6D_frame: origin xyz=2.7755575615628913511e-17 0 -0.022000000000000047296 rpy=-1.8505714609404598692e-19 -1.6770242961476544053e-17 -3.141592653589793116 -> xyz=-1.3877787807814456755e-17 -4.1633363423443370266e-17 -0.021999999999999991784 rpy=-2.2581636180355804894e-19 -6.9441320598627267313e-17 3.141592653589793116
- joint closedloop15_A_6D_frame: origin xyz=-2.7755575615628913511e-17 -1.3877787807814456755e-17 -0.021999999999999964029 rpy=6.3846877427644474244e-19 -1.6649989410368488151e-17 1.05387434053115508e-20 -> xyz=6.9388939039072283776e-17 -1.3877787807814456755e-17 -0.022000000000000102807 rpy=-3.1415926535897922278 1.2136429784084949567e-18 1.8454263175901755748e-19
- joint closedloop15_B_6D_frame: origin xyz=6.9388939039072283776e-18 0 -0.022000000000000047296 rpy=2.9668696099179873576e-15 -1.6282746472828449155e-16 1.570796326794896558 -> xyz=0 2.7755575615628913511e-17 -0.021999999999999977907 rpy=2.9668696099179873576e-15 -4.3043349733024282915e-15 1.570796326794896558
- joint closedloop16_A_6D_frame: origin xyz=0 3.1225022567582527699e-17 -0.022000000000000012601 rpy=-1.1895523874969165944e-18 2.1422087479376391186e-18 -6.3367552503614883775e-20 -> xyz=0 -3.4694469519536141888e-18 -0.022000000000000088929 rpy=-1.8504633983418571518e-19 -6.260850223067403694e-19 -4.7624303933662426292e-20
- joint closedloop17_A_6D_frame: origin xyz=1.3877787807814456755e-17 3.6429192995512948983e-17 -0.022000000000000075051 rpy=-3.141592653589793116 2.3850006220383799507e-18 -3.141592653589793116 -> xyz=-2.7755575615628913511e-17 -1.3877787807814456755e-17 -0.022000000000000186073 rpy=3.141592653589793116 -7.3264322513918817262e-18 -3.141592653589793116
- joint closedloop17_B_6D_frame: origin xyz=-2.7755575615628913511e-17 2.7755575615628913511e-17 -0.02199999999999989464 rpy=5.9407647068876257037e-19 -1.5422740935228754604e-17 -3.141592653589793116 -> xyz=-8.3266726846886740532e-17 1.1449174941446926823e-16 -0.021999999999999755862 rpy=-1.0432559969542629084e-18 7.3670874017545408448e-18 3.141592653589793116
- joint closedloop18_A_6D_frame: origin xyz=-2.7755575615628913511e-17 1.3877787807814456755e-17 -0.021999999999999964029 rpy=-3.141592653589793116 -7.7893742605831685744e-18 1.5311910373604695636e-18 -> xyz=-1.3877787807814456755e-17 1.3877787807814456755e-17 -0.022000000000000047296 rpy=-3.141592653589793116 -9.9855164538881929072e-18 -1.8871733321435959936e-16
- joint closedloop18_B_6D_frame: origin xyz=2.7755575615628913511e-17 2.7755575615628913511e-17 -0.021999999999999991784 rpy=2.8720513250545159028e-18 5.0069198964034734906e-17 -1.195602383648069109e-18 -> xyz=6.9388939039072283776e-17 0 -0.021999999999999908518 rpy=2.6914833269231957991e-18 3.6319536955476601562e-17 1.9081360785855584273e-18
- joint closedloop19_A_6D_frame: origin xyz=-2.4286128663675299322e-17 1.3877787807814456755e-17 -0.021999999999999981376 rpy=-9.4645443920224450633e-16 4.3138963368770645641e-15 -1.570796326794896558 -> xyz=0 1.3877787807814456755e-17 -0.022000000000000071582 rpy=-9.4224279476490090478e-16 4.313236932270966082e-15 -1.570796326794896558
- joint closedloop1_A_6D_frame: origin xyz=-1.6653345369377348106e-16 -8.3266726846886740532e-17 -0.02200000000000001954 rpy=-3.5035493923141009984e-15 1.2814418519762241213e-14 7.7830227665322737198e-18 -> xyz=0 -1.1102230246251565404e-16 -0.021999999999999964029 rpy=-3.5598665453424719627e-15 -1.9052153454978073203e-17 3.3163568929996116003e-17
- joint closedloop1_B_6D_frame: origin xyz=5.5511151231257827021e-17 -5.5511151231257827021e-17 -0.021999999999999964029 rpy=-3.1415926535897900074 2.0244592807192931317e-15 -1.570796326794896336 -> xyz=1.1102230246251565404e-16 -5.5511151231257827021e-17 -0.021999999999999908518 rpy=-3.1415926535897900074 2.0244592807192931317e-15 -1.570796326794896336
- joint closedloop23_A_3D_frame: origin xyz=-5.5511151231257827021e-17 -5.5511151231257827021e-17 -0.39999999999999991118 rpy=2.0595706521359607965e-16 6.9689394429105795176e-16 -3.8311948294342778263e-16 -> xyz=5.5511151231257827021e-17 5.5511151231257827021e-17 -0.39999999999999996669 rpy=1.9591181760418772481e-16 6.806829491380363508e-16 -5.9600644535927175492e-16
- joint closedloop2_A_6D_frame: origin xyz=-5.5511151231257827021e-17 -2.7755575615628913511e-17 -0.021999999999999964029 rpy=-1.3603990467924331356e-15 3.4203648913185160548e-15 4.0022067353557518153e-17 -> xyz=0 2.7755575615628913511e-17 -0.021999999999999991784 rpy=-1.3602385390666154951e-15 3.5897601158671507726e-15 -2.9774527545974381583e-17
- joint closedloop2_B_6D_frame: origin xyz=0 -8.3266726846886740532e-17 -0.021999999999999977907 rpy=3.1415926535897926719 3.2544751110174058161e-15 -1.570796326794896558 -> xyz=0 -8.3266726846886740532e-17 -0.021999999999999936273 rpy=3.1415926535897926719 3.2183378182619466957e-15 -1.570796326794896558
- joint closedloop3_A_6D_frame: origin xyz=-2.4286128663675299322e-17 0 -0.022000000000000158318 rpy=-3.141592653589793116 -8.9238004832296958299e-16 2.3469316244365445958e-17 -> xyz=-2.7755575615628913511e-17 -2.7755575615628913511e-17 -0.022000000000000130562 rpy=-3.141592653589793116 -9.9990740856057949295e-16 -3.7021204681756544686e-17
- joint closedloop3_B_6D_frame: origin xyz=-4.1633363423443370266e-17 -8.3266726846886740532e-17 -0.022000000000000005662 rpy=-3.8323071526180824844e-15 1.9454298298622066299e-16 1.4021234671943678824e-17 -> xyz=0 2.7755575615628913511e-17 -0.022000000000000047296 rpy=-3.8418763942784059345e-15 1.8594444041235966788e-16 1.1399726909584655164e-17
- joint closedloop4_A_6D_frame: origin xyz=1.7347234759768070944e-17 0 -0.02200000000000001954 rpy=-3.1415926535897895633 -5.8631330626161750329e-14 -2.5740459072486076896e-17 -> xyz=-2.7755575615628913511e-17 0 -0.022000000000000075051 rpy=-3.1415926535897895633 -5.8588589039601575851e-14 -8.1060924113090465019e-18
- joint closedloop4_B_6D_frame: origin xyz=5.5511151231257827021e-17 0 -0.021999999999999887701 rpy=-5.2397508177699997199e-14 7.9985639615515115397e-15 -6.9853190798646948938e-18 -> xyz=0 -2.7755575615628913511e-17 -0.022000000000000172196 rpy=-6.0488890030723583321e-14 2.4688424028795064476e-15 -1.0953694299338978907e-18
- joint closedloop5_A_6D_frame: origin xyz=-2.0816681711721685133e-17 0 -0.021999999999999936273 rpy=4.0939474033052918599e-16 2.1380466841413380764e-16 6.2026386493102164692e-16 -> xyz=0 0 -0.021999999999999929334 rpy=4.093947403305292846e-16 2.1380466841413412812e-16 4.0514340995891024666e-16
- joint closedloop6_A_3D_frame: origin xyz=0.038967453687049735667 -0.092095263467496704668 -5.5511151231257827021e-17 rpy=1.570796326794896558 4.0264892381777355687e-23 -1.570796326794896336 -> xyz=0.038967453687049735667 -0.092095263467496676912 -5.5511151231257827021e-17 rpy=1.570796326794896558 4.0264892381777355687e-23 -1.570796326794896336
- joint closedloop6_B_3D_frame: origin xyz=-2.7755575615628913511e-17 0 -0.42720000000000007967 rpy=-3.1415926535897926719 4.3171515544792239751e-16 3.141592653589793116 -> xyz=2.7755575615628913511e-17 -5.5511151231257827021e-17 -0.42719999999999991314 rpy=-3.1415926535897926719 4.3962922511980055669e-16 3.141592653589793116
- joint closedloop7_A_3D_frame: origin xyz=2.7755575615628913511e-17 -5.5511151231257827021e-17 -0.14142000000000004567 rpy=-3.141592653589793116 -2.5701272669893044796e-16 1.5487482446605287392e-16 -> xyz=1.3877787807814456755e-17 -5.5511151231257827021e-17 -0.14142000000000001791 rpy=-3.141592653589793116 -2.5701272669893044796e-16 1.5487482446605287392e-16
- joint closedloop7_B_3D_frame: origin xyz=0.083867056794542343967 -0.0077119035015027481705 -0.071500000000000063505 rpy=1.570796326794896558 -1.3655413196735760511e-30 -1.3856394439909555038e-14 -> xyz=0.083867056794542371723 -0.007711903501502720415 -0.071500000000000063505 rpy=1.570796326794896558 -2.0564927122134184515e-32 -1.3872350632051290567e-14
- joint closedloop8_A_6D_frame: origin xyz=-2.7755575615628913511e-17 -2.7755575615628913511e-17 -0.021999999999999991784 rpy=-3.141592653589793116 -7.5767938905805758326e-17 -1.570796326794896336 -> xyz=-8.3266726846886740532e-17 8.3266726846886740532e-17 -0.022000000000000075051 rpy=-3.141592653589793116 -7.5767938905805758326e-17 -1.570796326794896336
- joint closedloop8_B_6D_frame: origin xyz=0 -1.3877787807814456755e-17 -0.022000000000000047296 rpy=9.6232195658333659591e-16 -1.7756561743236490927e-16 1.5707963267948978903 -> xyz=-5.5511151231257827021e-17 -1.1275702593849246114e-17 -0.021999999999999950151 rpy=1.0351578883266661055e-15 -3.0410359695203482574e-16 1.5707963267948981123
- joint closedloop9_A_3D_frame: origin xyz=0 6.2450045135165055399e-17 -0.40000000000000013323 rpy=-2.3882228318976020147e-15 -1.0948393169349909809e-15 -1.5707963267948972241 -> xyz=0 5.2041704279304212832e-17 -0.40000000000000013323 rpy=-2.3882228318976020147e-15 -1.0948393169349909809e-15 -1.5707963267948972241
- joint closedloop9_B_3D_frame: origin xyz=-0.035854717888628991063 -0.041706584673488089621 0.052250000000000074163 rpy=1.570796326794896558 7.4525120443701586197e-31 -3.1415926535897908956 -> xyz=-0.035854717888628921674 -0.041706584673488200643 0.052250000000000046407 rpy=1.570796326794896558 7.4525120443701586197e-31 -3.1415926535897908956
- joint foot_right_frame: origin xyz=0.01201694922107987562 0.038499999999999923173 6.8117393392519431927e-09 rpy=1.5707963267948972241 4.1530747501458917702e-18 1.4689606375488657859e-15 -> xyz=0.01201694922107987562 0.038499999999999923173 6.8117394225186700396e-09 rpy=1.5707963267948972241 4.1530747501458917702e-18 1.4689606375488657859e-15
- joint frame_motor_ankle1: origin xyz=0.054086706326755232266 0.014047405294960763067 -0.11825000000000002176 rpy=-1.570796326794896558 0.73498046737731748124 0.2858933777993256653 -> xyz=0.054086706326755218388 0.014047405294960790823 -0.11824999999999985523 rpy=-1.57079632679489678 0.73498046737729960665 0.2858933777993256653
- joint frame_motor_ankle1_left: origin xyz=0.054086706326755308594 -0.014047405294960818578 -0.11824999999999991074 rpy=1.570796326794896558 0.014238452528742229219 -0.28589337779933110539 -> xyz=0.054086706326755322471 -0.014047405294960790823 -0.118249999999999994 rpy=1.570796326794896558 0.014238452528749003315 -0.28589337779933121642
- joint frame_motor_ankle2: origin xyz=0.054086706326755190632 0.014047405294960790823 -0.024750000000000021982 rpy=1.570796326794896558 -0.17956569756706666774 -2.8556992757904748892 -> xyz=0.054086706326755190632 0.014047405294960846334 -0.024750000000000133005 rpy=1.57079632679489678 -0.17956569756705714758 -2.855699275790474001
- joint frame_motor_ankle2_left: origin xyz=0.054086706326755280838 -0.014047405294960763067 -0.024750000000000119127 rpy=-1.570796326794896558 -0.014238452528742286465 2.8556992757904868796 -> xyz=0.054086706326755301655 -0.014047405294960763067 -0.024750000000000056677 rpy=-1.570796326794896558 -0.014238452528749060561 2.8556992757904868796
- joint frame_motor_knee: origin xyz=-0.061655078133537336016 -0.018724201373191806663 4.297340261416593421e-12 rpy=-1.570796326794896558 1.2771385194773066107 -0.60601731071218278846 -> xyz=-0.061655078133537280505 -0.018724201373191778908 4.297340261416593421e-12 rpy=-1.570796326794896558 1.2771385194773066107 -0.60601731071218278846
- joint free_ankle_universalx: origin xyz=6.6000000007115922074e-05 -1.1102230246251565404e-16 6.6000000002341963068e-05 rpy=-1.570796326794896558 -0.95882611835293629632 -1.570796326794896558 -> xyz=6.5999999999899472414e-05 -9.9920072216264088638e-16 6.6000000001481540224e-05 rpy=-1.5707963267948978903 -0.95882611835293851676 -1.5707963267948956698
- joint free_motor_holder_1: origin xyz=0.012499999999999998959 -0.037124999999999658273 -0.077000000000000151656 rpy=1.57079632679489678 -0.033001070205816974978 -1.5707963267948974462 -> xyz=0.012500000000000047531 -0.037124999999999713785 -0.077000000000000262679 rpy=1.57079632679489678 -0.021206259450686756884 -1.5707963267948974462
- joint free_motor_holder_1_left: origin xyz=0.012500000000000007633 -0.037125000000000123179 -0.07700000000000006839 rpy=1.570796326794896558 -0.019211068168970831666 -1.5707963267948918951 -> xyz=0.012499999999999990286 -0.037124999999999915012 -0.076999999999999957367 rpy=1.57079632679489678 -0.026529746372805688981 -1.5707963267948961139
- joint free_motor_holder_2_left: origin xyz=0.012500000000000007633 0.037124999999999908074 -0.076999999999999971245 rpy=-1.570796326794896558 -0.021147767637937589513 1.5707963267948983344 -> xyz=0.012499999999999990286 0.037124999999999880318 -0.076999999999999860223 rpy=-1.570796326794896558 -0.026024394633311673242 1.5707963267948956698
- joint free_motor_holder_3: origin xyz=0.012499999999999998959 0.037125000000000019096 -0.077000000000000151656 rpy=-1.570796326794896558 -0.029979973678264791592 1.5707963267948958919 -> xyz=0.01249999999999999549 0.03712499999999999134 -0.07699999999999981859 rpy=-1.570796326794896558 -0.019264206118359661346 1.5707963267948950037
- joint free_motor_holder_hip_xy1_left: origin xyz=4.1633363423443370266e-17 4.1633363423443370266e-17 -0.054999999999999993339 rpy=-1.570796326794896558 1.4797294953454118716 1.5707963267949098807 -> xyz=2.7755575615628913511e-17 3.6082248300317587564e-16 -0.054999999999999979461 rpy=-1.5707963267948974462 1.4812643203298270222 1.5707963267949103248
- joint free_motor_holder_hip_xy2_left: origin xyz=5.2041704279304212832e-18 1.8041124150158793782e-16 -0.054999999999999993339 rpy=-1.570796326794896558 -1.4803191601263148147 1.5707963267948810149 -> xyz=-2.7755575615628913511e-17 5.5511151231257827021e-17 -0.055000000000000021094 rpy=-1.5707963267948961139 -1.4802679079841647436 1.5707963267948805708
- joint free_motor_holder_hipxy1: origin xyz=-2.7755575615628913511e-17 1.6653345369377348106e-16 -0.054999999999999979461 rpy=-1.57079632679489678 1.1267886452730790925 1.5707963267949007768 -> xyz=-5.5511151231257827021e-17 5.5511151231257827021e-17 -0.055000000000000007216 rpy=-1.5707963267948976682 1.4788923407475595972 1.5707963267949134334
- joint free_motor_holder_hipxy2: origin xyz=-2.7755575615628913511e-17 -6.9388939039072283776e-17 -0.055000000000000062728 rpy=-1.570796326794896558 -1.1268255606165180627 1.5707963267948938935 -> xyz=2.7755575615628913511e-17 5.5511151231257827021e-17 -0.054999999999999944766 rpy=-1.570796326794876796 -1.4788959325009420898 1.570796326794836606
- joint free_spherical_hip_xy_1_left: origin xyz=-0.060499999999999970468 -2.7755575615628913511e-17 -0.038500000000000013378 rpy=1.570796326794896558 9.8397440977066039283e-15 -9.8885767237220441916e-16 -> xyz=-0.060499999999999991285 -2.7755575615628913511e-17 -0.038499999999999985623 rpy=1.570796326794896558 1.6842724911847358392e-14 -9.8608513340270172252e-16
- joint free_spherical_hipxy_2_left: origin xyz=-0.060499999999999984346 1.1102230246251565404e-16 0.038500000000000013378 rpy=-1.57079632679489678 -1.021615604280151078e-14 3.1415926535897908956 -> xyz=-0.060499999999999991285 0 0.038499999999999964806 rpy=-1.570796326794896558 0.17430796725364161581 3.1415926535897917837
- joint free_spherical_motor_holder_1: origin xyz=1.3877787807814456755e-17 -8.3266726846886740532e-17 -0.051749999999999775346 rpy=1.5707963267948976682 -0.051824161433118527686 1.5707963267948943376 -> xyz=-1.3877787807814456755e-17 5.5511151231257827021e-17 -0.051749999999999886369 rpy=1.570796326794896558 -0.094549574280562209694 1.5707963267948903408
- joint free_universal_y_hip_left: origin xyz=-6.5999999999961922459e-05 -2.7755575615628913511e-17 -6.5999999999998351652e-05 rpy=-1.5707963267951692288 -1.5358146150088003434 1.5707963267951787767 -> xyz=-6.5999999999961922459e-05 -2.7755575615628913511e-17 -6.5999999999998351652e-05 rpy=-1.570796326795369291 -1.5358146150088136661 1.5707963267953790609
- joint lower_hip: origin xyz=6.6000000000010494716e-05 -2.7755575615628913511e-17 -6.6000000000000086375e-05 rpy=-1.5707963267949025532 -1.1595523542658980887 -1.5707963267948952257 -> xyz=6.6000000000038250292e-05 0 -6.6000000000003555822e-05 rpy=1.5707963267949520692 -1.5388859775012673214 1.5707963267948683583
- joint lower_knee: origin xyz=-0.21747050071615142697 -0.33571800862966272305 -5.5511151231257827021e-17 rpy=2.0331881193927353103e-17 3.4472918726955580133e-17 0.89630439304597731009 -> xyz=-0.21747050071615126043 -0.3357180086296619459 -2.2204460492503130808e-16 rpy=-1.2825270953943237956e-16 -5.2913746228227154917e-16 0.89630439304597941952
- joint motor_ankle1: origin xyz=3.0531133177191804862e-16 -2.7755575615628913511e-17 0.018399835965480559885 rpy=-3.141592653589793116 2.2946682489661683897e-15 3.1415926535897926719 -> xyz=0 1.6653345369377348106e-16 0.043564478507036985544 rpy=3.1415926535897891192 2.698026123213506634e-15 3.1415926535897926719
- joint motor_ankle1_left: origin xyz=-6.8001160258290838101e-16 1.249000902703301108e-16 0.041658869056533737174 rpy=3.141592653589793116 1.0794107117225389546e-14 -3.1415926535897873428 -> xyz=-1.3877787807814456755e-17 1.0408340855860842566e-17 0.041658869056532793484 rpy=3.1415926535897820138 -6.6815401904784765465e-15 -3.1415926535897873428
- joint motor_ankle2: origin xyz=4.2743586448068526806e-15 7.5772721430666933884e-15 0.021140168165682704515 rpy=3.1415926535897926719 1.8047950485096526647e-14 3.1415926535897802374 -> xyz=1.1102230246251565404e-16 2.2204460492503130808e-16 0.046304810707238769352 rpy=3.1415926535897926719 1.8282399324537366167e-14 3.1415926535897797933
- joint motor_ankle2_left: origin xyz=-6.9388939039072283776e-16 -5.5511151231257827021e-17 0.036860927393517817219 rpy=-3.141592653589793116 -2.3101201183360073099e-15 -3.1415926535897829019 -> xyz=6.9388939039072283776e-17 2.7755575615628913511e-17 0.036860927393517151085 rpy=-3.141592653589793116 1.5408374369357243975e-14 -3.1415926535897824579
- joint motor_hip_xy_1: origin xyz=5.5511151231257827021e-17 -0.026357933593704453712 2.7755575615628913511e-17 rpy=-1.5707963267948994446 2.6524860729722982745e-15 1.8903718014666384216e-15 -> xyz=0 -0.046242052428871111003 5.5511151231257827021e-17 rpy=-1.5707963267948996666 2.6244546298293282002e-15 1.7228045307915577077e-15
- joint motor_hip_xy_1_left: origin xyz=1.3877787807814456755e-17 -0.049224876560801336667 1.3877787807814456755e-17 rpy=-1.570796326794896558 -8.4128073089814322834e-15 7.43963769432937431e-15 -> xyz=1.3877787807814456755e-17 -0.044933728103784820185 -3.6602665343110629692e-16 rpy=-1.5707963267949507369 -8.3077011567330338006e-15 7.4116426331934598049e-15
- joint motor_hip_xy_2: origin xyz=0 -0.026361686710175066817 -1.9428902930940239457e-16 rpy=-1.5707963267949502928 -7.9875720912898989692e-15 7.040089964984604181e-15 -> xyz=-5.5511151231257827021e-17 -0.046244712027414175415 -4.1633363423443370266e-16 rpy=-1.5707963267949494046 -7.6308472951699595211e-15 7.1448122585686606186e-15
- joint motor_hip_xy_2_left: origin xyz=0 -0.04333782624542449613 4.1633363423443370266e-17 rpy=-1.570796326794896558 2.612321956315469991e-15 2.3456370119822959644e-15 -> xyz=1.3877787807814456755e-17 -0.046444953521771831229 1.249000902703301108e-16 rpy=-1.5707963267948994446 2.6395580239470105185e-15 2.7853195712080230793e-15
- joint motor_hip_z_left: origin xyz=5.5511151231257827021e-17 3.4694469519536141888e-18 -0.070937073864986127658 rpy=-2.3978477236838945599e-15 -1.3376382854703311896e-16 -1.570796326794871467 -> xyz=-1.4398204850607498884e-16 1.5265566588595902431e-16 -0.070937073864986155414 rpy=-2.3897270858110496043e-15 -1.556724709680402787e-16 -1.5707963267948730213
- joint motor_hipz: origin xyz=-1.3877787807814456755e-16 -3.8163916471489756077e-16 -0.07149999999999984146 rpy=-2.1233015345958434142e-15 4.128211776064302964e-17 -1.5707963267949134334 -> xyz=-4.9960036108132044319e-16 -1.5959455978986625269e-16 -0.071499999999999813705 rpy=-6.0620461731129641165e-15 1.521560350042941006e-15 -1.5707963267949132113
- joint motor_knee: origin xyz=-8.2434059578417873126e-15 -1.8873791418627661187e-15 -0.0023309791397017609604 rpy=3.141592653589793116 1.4510931439305401901e-15 -4.1052068437918848451e-15 -> xyz=5.5511151231257827021e-17 1.6653345369377348106e-16 -0.020205644373555181614 rpy=3.141592653589793116 1.4510931439305401901e-15 -4.1052068437918848451e-15
- joint spherical_4rod: origin xyz=0.0194837268435249511 -0.046047631733748414784 0 rpy=1.57079632679489678 0.15824418733945430637 1.5707963267948958919 -> xyz=0.0194837268435249511 -0.046047631733748387028 0 rpy=1.57079632679489678 0.15824418733945430637 1.5707963267948958919
- joint spherical_4rod_left: origin xyz=0.0194837268435249511 -0.046047631733748352334 -6.9388939039072283776e-18 rpy=1.57079632679489678 0.15824418733945430637 1.5707963267948952257 -> xyz=0.019483726843525006611 -0.046047631733748345395 1.0408340855860842566e-17 rpy=1.57079632679489678 0.15824418733945425086 1.5707963267948952257
- joint spherical_actuation_knee_left: origin xyz=-0.013749999999999866496 -0.0024999999999999467093 -0.070874999999999993561 rpy=1.570796326794896558 8.9605786434077115269e-17 1.570796326794896558 -> xyz=-0.01374999999999977629 -0.0024999999999999467093 -0.070875000000000007438 rpy=1.570796326794896558 3.5095903105758312051e-17 1.570796326794896558
- joint spherical_lower_hip1: origin xyz=-0.060500000000000137002 2.7755575615628913511e-17 -0.038499999999999978684 rpy=1.57079632679489678 -0.083114644637941520466 -3.1415926535897846783 -> xyz=-0.060500000000000109246 2.7755575615628913511e-17 -0.038499999999999978684 rpy=1.57079632679489678 -0.083114644637934484428 -3.1415926535897846783
- joint spherical_lower_hip2: origin xyz=-0.060500000000000150879 2.7755575615628913511e-17 0.03850000000000006195 rpy=-1.57079632679489678 0.090109706454325047553 -5.2539072764179264277e-14 -> xyz=-0.06050000000000008149 -8.3266726846886740532e-17 0.038500000000000006439 rpy=-1.57079632679489678 -0.044003745446504607952 -5.158214291223756956e-14
- joint spherical_motor_holder_hip_z_left: origin xyz=-1.3877787807814456755e-17 -5.5511151231257827021e-17 -0.051749999999999823919 rpy=1.570796326794896336 1.3223675276875890283 1.5707963267949045516 -> xyz=-1.3877787807814456755e-17 2.7755575615628913511e-17 -0.051749999999999934941 rpy=1.5707963267948961139 -0.14866879169792945881 1.5707963267948972241
- joint spherical_motor_knee_holder: origin xyz=-0.013749999999999956701 0.0024999999999999744649 -0.072000000000000008438 rpy=-1.57079632679489678 -0.99860729712136542258 -1.5707963267949036634 -> xyz=-0.013750000000000071193 0.0024999999999999744649 -0.072000000000000008438 rpy=-1.57079632679489678 -0.99860729712135265501 -1.5707963267949038855
- joint spherical_motor_transmission_hip1_left: origin xyz=0.043531328479973735446 0.0032046566522410946387 -0.025000000000000001388 rpy=1.5707963267948970021 -1.3881446540757400587 -3.1415926535897527039 -> xyz=0.043531328479973513401 0.0032046566522406227939 -0.02500000000000011241 rpy=1.5707963267948970021 -1.3881446540757382824 -3.1415926535897527039
- joint spherical_shin_rod1: origin xyz=0.038967453687049735667 -0.092095263467496524257 0 rpy=-1.57079632679489678 -1.3380503778517247593 1.5707963267948987784 -> xyz=0.038967453687049735667 -0.092095263467496718546 1.1102230246251565404e-16 rpy=-1.57079632679489678 -1.3380503778517249813 1.5707963267948987784
- joint spherical_transmission_foot1: origin xyz=-0.059494699261975536597 0.010983203527527130028 0.022000000000000047296 rpy=1.570796326794896558 -0.30096768397183631949 1.5707963267948981123 -> xyz=-0.059494699261975467208 0.010983203527527130028 0.02200000000000001954 rpy=1.570796326794896558 -0.30096768397183631949 1.5707963267948981123
- joint spherical_transmission_foot2: origin xyz=-0.059494699261975703131 0.010983203527527130028 -0.021999999999999964029 rpy=-1.57079632679489678 0.2674961218464166901 -1.570796326794896558 -> xyz=-0.059494699261975467208 0.01098320352752724105 -0.021999999999999964029 rpy=-1.57079632679489678 0.2674961218464166901 -1.570796326794896558
- joint spherical_transmission_hip3: origin xyz=0.041074543378118832937 0.036577067764912832293 -0.005000000000000059952 rpy=-1.570796326794896558 0.67303436723393439411 3.141592653589793116 -> xyz=0.041074543378118805181 0.036577067764912860048 -0.0050000000000000044409 rpy=-1.570796326794896558 0.67303436723393439411 3.141592653589793116
- joint spherical_transmission_hip3_left: origin xyz=0.041074543378118943959 0.03657706776491291556 -0.0049999999999999888284 rpy=-1.570796326794896558 0.6730343672339298422 3.1415926535897922278 -> xyz=0.041074543378118194559 0.03657706776491259637 -0.00499999999999997842 rpy=-1.570796326794896558 0.67303436723393150753 3.1415926535897922278
- joint spherical_transmission_hip4: origin xyz=0.041074543378118888448 -0.036577067764912901682 -0.0050000000000000044409 rpy=1.570796326794896558 0.73924967494907445342 3.1415926535897851224 -> xyz=0.041074543378118943959 -0.036577067764912887804 -0.005000000000000059952 rpy=1.570796326794896558 0.73924967494907445342 3.1415926535897851224
- joint spherical_transmission_motor_hip1: origin xyz=0.043531328479973679935 0.0032046566522409558608 -0.025000000000000077716 rpy=1.5707963267948992225 -1.3881446540757451658 -3.1415926535897669147 -> xyz=0.043531328479973735446 0.0032046566522409003497 -0.025000000000000077716 rpy=1.5707963267948992225 -1.3881446540757451658 -3.1415926535897669147
- joint spherical_transmission_motor_hip2: origin xyz=0.043531328479973679935 -0.0032046566522410668831 -0.024999999999999938938 rpy=1.570796326794896558 -1.0520766825141583123 -1.2677408616997643214e-14 -> xyz=0.04353132847997370769 -0.0032046566522409836164 -0.024999999999999994449 rpy=1.570796326794896558 -1.0520766825141583123 -1.2677408616997643214e-14
- joint transmission_ankle3_left: origin xyz=6.2450045135165055399e-17 -0.046751999999999988011 -0.055000000000000014155 rpy=-3.1415926535897895633 -4.799310970213847672e-16 -1.2495340742674121426 -> xyz=7.6327832942979512154e-17 -0.0467519999999999325 -0.05499999999999967415 rpy=-3.1415926535897908956 -1.2924964444112278435e-16 -1.249534074267399042
- joint transmission_ankle4_left: origin xyz=4.5102810375396984455e-17 -0.046752000000000043523 -0.087999999999999981015 rpy=-8.8738167568813836499e-15 3.5840702149163616535e-15 -1.2172645625817111181 -> xyz=4.5102810375396984455e-17 -0.046752000000000043523 -0.087999999999999994893 rpy=-1.544415098831094204e-14 6.0086890509720742404e-15 -1.2172645625816977955
- joint transmission_hip1: origin xyz=-6.2450045135165055399e-17 0.046752000000000015767 -0.087999999999999967137 rpy=9.4681397285287776746e-15 -4.9405061162797479416e-15 0.77974518790642721733 -> xyz=-5.1694759584108851413e-16 0.046752000000001264768 -0.088000000000000022649 rpy=5.7225514480077479615e-15 -7.6451103975374452784e-15 1.22289950972905892
- joint transmission_hip2: origin xyz=-6.2450045135165055399e-17 0.046752000000000015767 -0.054999999999999993339 rpy=-3.1415926535897837901 -5.6800076792079728017e-15 0.82801632278258496811 -> xyz=-5.1000870193718128576e-16 0.046752000000001264768 -0.05500000000000004885 rpy=-3.1415926535897877869 -8.2007279796863668596e-15 1.2711706446052168928
- joint triangle_knee1: origin xyz=-0.21747050071615148248 -0.33571800862966283407 0.010000000000000008882 rpy=3.1415926535897922278 2.5397996671417581801e-15 3.0532620163569994531 -> xyz=-0.21747050071615151023 -0.33571800862966283407 0.010000000000000008882 rpy=3.1415926535897922278 2.5397996671417581801e-15 3.0532620163569994531
- joint triangle_knee2: origin xyz=-0.21747050071615164901 -0.33571800862966283407 -0.010000000000000008882 rpy=3.1415926535897926719 2.3960728016627840815e-15 3.0785068790704639419 -> xyz=-0.2174705007161515935 -0.33571800862966272305 -0.010000000000000008882 rpy=3.1415926535897926719 2.3960728016627840815e-15 3.0785068790704639419
- joint uneveral_foot1: origin xyz=0.21747050071614926203 -0.33571800862966427736 0 rpy=-1.5707963267948958919 -1.4835298641951766285 1.5707963267949329733 -> xyz=0.21747050071614928979 -0.33571800862966416634 0 rpy=-1.5707963267948958919 -1.4835298641951766285 1.5707963267949329733
- joint upper_knee: origin xyz=-6.2450045135165055399e-17 0.046752000000000015767 -0.071500000000000007994 rpy=-3.1415926535897842342 -1.2696304357689524271e-15 0.22729525162017977236 -> xyz=-5.2041704279304212832e-16 0.046752000000001264768 -0.071500000000000007994 rpy=-3.1415926535897860106 -5.537490036297666694e-15 0.67044957344281030931
- joint upper_knee_left: origin xyz=2.0469737016526323714e-16 -0.046752000000000043523 -0.071499999999999980238 rpy=-5.7342617493489877044e-15 7.864783300419491944e-15 -0.63853922414920383233 -> xyz=3.2265856653168611956e-16 -0.046752000000000043523 -0.071499999999999980238 rpy=-9.9086391638234093953e-15 1.3486642849930377956e-14 -0.63853922414919062067
