Commit message: fix frame

File: example_parallel_robots/robots/kangaroo_like_2legs/robot.urdf (robot description, URDF)
Before this commit: robot onshape, 131 links, 130 joints
Links:
- removed link closedloop14_A_6D
- removed link closedloop14_B_6D
- removed link closedloop15_A_6D
- removed link closedloop15_B_6D
- removed link closedloop1_A_6D
- removed link closedloop1_B_6D
- removed link closedloop2_A_6D
- removed link closedloop2_B_6D
- added link closedloop14_A_3D, mass 1e-9
- added link closedloop14_B_3D, mass 1e-9
- added link closedloop15_A_3D, mass 1e-9
- added link closedloop15_B_3D, mass 1e-9
- added link closedloop1_A_3D, mass 1e-9
- added link closedloop1_B_3D, mass 1e-9
- added link closedloop2_A_3D, mass 1e-9
- added link closedloop2_B_3D, mass 1e-9
- link part_1: mass 0.24432174426363428843 -> 0.24432174426363423292
- link part_1_gauche: mass 0.24432174482850421704 -> 0.24432174482850427255
- link part_4: mass 0.011311035579799526632 -> 0.011311035579799528367
- link part_4_2: mass 0.011311035579799526632 -> 0.011311035579799528367
- link part_8: mass 0.0062040903886272707676 -> 0.0062040903886272725024
- link part_8_2: mass 0.0062040903886272707676 -> 0.0062040903886272725024
- link part_9: mass 0.0062040903886272699003 -> 0.0062040903886272707676
- link part_9_2: mass 0.0062040903886272699003 -> 0.0062040903886272707676
- link renvois_cheville: mass 0.074310321213953561825 -> 0.074310321213953547947
- link renvois_cheville_2: mass 0.074310321213953561825 -> 0.074310321213953547947
Joints:
- removed joint closedloop14_A_6D_frame
- removed joint closedloop14_B_6D_frame
- removed joint closedloop15_A_6D_frame
- removed joint closedloop15_B_6D_frame
- removed joint closedloop1_A_6D_frame
- removed joint closedloop1_B_6D_frame
- removed joint closedloop2_A_6D_frame
- removed joint closedloop2_B_6D_frame
- added joint closedloop14_A_3D_frame: type fixed, parent piston_4, child closedloop14_A_3D, origin xyz=-6.9388939039072283776e-18 -2.7755575615628913511e-17 -0.021999999999999991784 rpy=-3.141592653589793116 4.6224429555000727957e-17 -1.570796326794896558, axis 0 0 0
- added joint closedloop14_B_3D_frame: type fixed, parent piston_8, child closedloop14_B_3D, origin xyz=0 -1.0408340855860842566e-17 -0.02200000000000001954 rpy=-2.7761328130793523422e-19 -6.9441320598627267313e-17 -3.141592653589793116, axis 0 0 0
- added joint closedloop15_A_3D_frame: type fixed, parent piston_7, child closedloop15_A_3D, origin xyz=4.1633363423443370266e-17 -5.5511151231257827021e-17 -0.022000000000000075051 rpy=-3.1415926535897922278 8.277323861869742215e-19 5.6322170327204818248e-20, axis 0 0 0
- added joint closedloop15_B_3D_frame: type fixed, parent piston_5, child closedloop15_B_3D, origin xyz=0 2.7755575615628913511e-17 -0.021999999999999977907 rpy=2.9668696099179873576e-15 -4.3043349733024282915e-15 1.570796326794896558, axis 0 0 0
- added joint closedloop1_A_3D_frame: type fixed, parent piston_18, child closedloop1_A_3D, origin xyz=0 -2.7755575615628913511e-17 -0.021999999999999964029 rpy=-3.5858412855701039305e-15 1.2795475548061141038e-14 1.9564349175002147908e-16, axis 0 0 0
- added joint closedloop1_B_3D_frame: type fixed, parent piston_15, child closedloop1_B_3D, origin xyz=1.1102230246251565404e-16 -5.5511151231257827021e-17 -0.021999999999999908518 rpy=-3.1415926535897900074 2.0244592807192931317e-15 -1.570796326794896336, axis 0 0 0
- added joint closedloop2_A_3D_frame: type fixed, parent piston_19, child closedloop2_A_3D, origin xyz=0 -2.7755575615628913511e-17 -0.021999999999999880762 rpy=-1.0697317727682620177e-15 -1.8801810800543854443e-17 -3.3869376106552871114e-17, axis 0 0 0
- added joint closedloop2_B_3D_frame: type fixed, parent piston_16, child closedloop2_B_3D, origin xyz=0 -8.3266726846886740532e-17 -0.021999999999999936273 rpy=3.1415926535897926719 3.2183378182619466957e-15 -1.570796326794896558, axis 0 0 0
- joint 4rof_knee_left: origin xyz=0.04604763173374580576 -0.01948372684352350781 7.6327832942979512154e-17 rpy=3.141592653589793116 4.4057711130820799237e-17 -1.2499268310990352404 -> xyz=0.046047631733747068639 -0.019483726843524284966 6.5919492087118669588e-17 rpy=3.141592653589793116 4.405771113082074377e-17 -1.2499268310990390152
- joint closedloop13_B_3D_frame: origin xyz=0.083867056794542510501 0.007711903501502720415 -0.071500000000000021871 rpy=1.570796326794896558 -3.7484973866353497179e-19 3.141592653589793116 -> xyz=0.083867056794542510501 0.007711903501502720415 -0.071500000000000063505 rpy=1.570796326794896558 -2.7708369985933544671e-19 3.141592653589793116
- joint closedloop16_A_6D_frame: origin xyz=0 -3.4694469519536141888e-18 -0.022000000000000088929 rpy=-1.8504633983418571518e-19 -6.260850223067403694e-19 -4.7624303933662426292e-20 -> xyz=0 2.0816681711721685133e-17 -0.022000000000000040357 rpy=3.8407815244357912106e-19 -7.2372460481629324552e-19 -1.0504212169390065499e-19
- joint closedloop16_B_6D_frame: origin xyz=-2.7755575615628913511e-17 -2.7755575615628913511e-17 -0.022000000000000033418 rpy=3.141592653589793116 1.5080939153133216998e-16 -1.57079632679489678 -> xyz=2.0816681711721685133e-17 -2.7755575615628913511e-17 -0.021999999999999977907 rpy=3.141592653589793116 1.2701984792014930899e-16 -1.57079632679489678
- joint closedloop17_A_6D_frame: origin xyz=-2.7755575615628913511e-17 -1.3877787807814456755e-17 -0.022000000000000186073 rpy=3.141592653589793116 -7.3264322513918817262e-18 -3.141592653589793116 -> xyz=0 2.168404344971008868e-17 -0.021999999999999964029 rpy=3.141592653589793116 -4.8517792999468327746e-19 -3.141592653589793116
- joint closedloop17_B_6D_frame: origin xyz=-8.3266726846886740532e-17 1.1449174941446926823e-16 -0.021999999999999755862 rpy=-1.0432559969542629084e-18 7.3670874017545408448e-18 3.141592653589793116 -> xyz=-1.3877787807814456755e-17 2.4286128663675299322e-17 -0.022000000000000116684 rpy=-3.9459199271606617764e-19 -2.2201859142713151923e-17 3.141592653589793116
- joint closedloop18_A_6D_frame: origin xyz=-1.3877787807814456755e-17 1.3877787807814456755e-17 -0.022000000000000047296 rpy=-3.141592653589793116 -9.9855164538881929072e-18 -1.8871733321435959936e-16 -> xyz=2.7755575615628913511e-17 1.3877787807814456755e-17 -0.022000000000000075051 rpy=3.141592653589793116 -5.3135589439629951664e-18 -2.4122454690407664662e-16
- joint closedloop18_B_6D_frame: origin xyz=6.9388939039072283776e-17 0 -0.021999999999999908518 rpy=2.6914833269231957991e-18 3.6319536955476601562e-17 1.9081360785855584273e-18 -> xyz=-2.7755575615628913511e-17 -1.3877787807814456755e-17 -0.021999999999999908518 rpy=1.7699474212156413685e-18 2.1115912505350949368e-17 3.4380251162177467281e-18
- joint closedloop23_A_3D_frame: origin xyz=5.5511151231257827021e-17 5.5511151231257827021e-17 -0.39999999999999996669 rpy=1.9591181760418772481e-16 6.806829491380363508e-16 -5.9600644535927175492e-16 -> xyz=2.7755575615628913511e-17 2.7755575615628913511e-17 -0.39999999999999996669 rpy=2.1692123864575216095e-16 7.3047674865800371478e-16 -4.6114240044222220693e-16
- joint frame_motor_ankle1_left: origin xyz=0.054086706326755322471 -0.014047405294960790823 -0.118249999999999994 rpy=1.570796326794896558 0.014238452528749003315 -0.28589337779933121642 -> xyz=0.054086706326755343288 -0.014047405294960818578 -0.11825000000000003564 rpy=1.570796326794896558 0.014238452528732936306 -0.2858933777993311609
- joint frame_motor_ankle2: origin xyz=0.054086706326755190632 0.014047405294960846334 -0.024750000000000133005 rpy=1.57079632679489678 -0.17956569756705714758 -2.855699275790474001 -> xyz=0.054086706326755190632 0.014047405294960846334 -0.024750000000000133005 rpy=1.5707963267948925612 -0.17956569756705717533 -2.855699275790474001
- joint frame_motor_ankle2_left: origin xyz=0.054086706326755301655 -0.014047405294960763067 -0.024750000000000056677 rpy=-1.570796326794896558 -0.014238452528749060561 2.8556992757904868796 -> xyz=0.054086706326755315533 -0.014047405294960790823 -0.024750000000000008105 rpy=-1.570796326794896558 -0.014238452528733023042 2.8556992757904868796
- joint free_motor_holder_1: origin xyz=0.012500000000000047531 -0.037124999999999713785 -0.077000000000000262679 rpy=1.57079632679489678 -0.021206259450686756884 -1.5707963267948974462 -> xyz=0.01249999999999999202 -0.037124999999999713785 -0.077000000000000151656 rpy=1.57079632679489678 -0.021206259450691003487 -1.5707963267948974462
- joint free_motor_holder_1_left: origin xyz=0.012499999999999990286 -0.037124999999999915012 -0.076999999999999957367 rpy=1.57079632679489678 -0.026529746372805688981 -1.5707963267948961139 -> xyz=0.012500000000000000694 -0.037125000000000150935 -0.076999999999999957367 rpy=1.570796326794896558 -0.026529746372805688981 -1.5707963267948918951
- joint free_motor_holder_2_left: origin xyz=0.012499999999999990286 0.037124999999999880318 -0.076999999999999860223 rpy=-1.570796326794896558 -0.026024394633311673242 1.5707963267948956698 -> xyz=0.012500000000000004163 0.037124999999999880318 -0.077000000000000082268 rpy=-1.570796326794896558 -0.026024394633311673242 1.5707963267948983344
- joint free_motor_holder_hip_xy1_left: origin xyz=2.7755575615628913511e-17 3.6082248300317587564e-16 -0.054999999999999979461 rpy=-1.5707963267948974462 1.4812643203298270222 1.5707963267949103248 -> xyz=-2.7755575615628913511e-17 4.1633363423443370266e-17 -0.0549999999999999864 rpy=-1.570796326794896558 1.4812643203298270222 1.5707963267949109909
- joint free_motor_holder_hip_xy2_left: origin xyz=-2.7755575615628913511e-17 5.5511151231257827021e-17 -0.055000000000000021094 rpy=-1.5707963267948961139 -1.4802679079841647436 1.5707963267948805708 -> xyz=0 -5.5511151231257827021e-17 -0.0549999999999999864 rpy=-1.570796326794896558 -1.4802679079841647436 1.5707963267948810149
- joint free_motor_holder_hipxy2: origin xyz=2.7755575615628913511e-17 5.5511151231257827021e-17 -0.054999999999999944766 rpy=-1.570796326794876796 -1.4788959325009420898 1.570796326794836606 -> xyz=2.7755575615628913511e-17 -5.5511151231257827021e-17 -0.055000000000000000278 rpy=-1.570796326794876796 -1.4788959325009420898 1.5707963267948323871
- joint free_motor_knee_left: origin xyz=-0.061655078133537488672 -0.018724201373191667885 4.2973298530757375602e-12 rpy=-1.570796326794896558 1.3873492000155343007 -0.60601731071219677727 -> xyz=-0.061655078133537329077 -0.018724201373191612374 4.2973576086513531891e-12 rpy=-1.5707963267948972241 1.3873492000155343007 -0.60601731071219733238
- joint free_spherical_hip_xy_1_left: origin xyz=-0.060499999999999991285 -2.7755575615628913511e-17 -0.038499999999999985623 rpy=1.570796326794896558 1.6842724911847358392e-14 -9.8608513340270172252e-16 -> xyz=-0.06049999999999995659 1.3877787807814456755e-16 -0.038500000000000034195 rpy=1.570796326794896558 4.477119026960201655e-15 -9.9292638772409921535e-16
- joint free_spherical_hipxy_2_left: origin xyz=-0.060499999999999991285 0 0.038499999999999964806 rpy=-1.570796326794896558 0.17430796725364161581 3.1415926535897917837 -> xyz=-0.06049999999999995659 8.3266726846886740532e-17 0.038499999999999964806 rpy=-1.57079632679489678 0.17430796725365393929 3.1415926535897908956
- joint free_spherical_motor_holder_1: origin xyz=-1.3877787807814456755e-17 5.5511151231257827021e-17 -0.051749999999999886369 rpy=1.570796326794896558 -0.094549574280562209694 1.5707963267948903408 -> xyz=-1.3877787807814456755e-17 0 -0.051749999999999886369 rpy=1.570796326794896558 -0.094549574280562209694 1.5707963267948930053
- joint free_universal_y_hip_left: origin xyz=-6.5999999999961922459e-05 -2.7755575615628913511e-17 -6.5999999999998351652e-05 rpy=-1.570796326795369291 -1.5358146150088136661 1.5707963267953790609 -> xyz=-6.6000000001009695438e-05 0 -6.5999999999575079124e-05 rpy=-1.5707963267950024733 -1.5358146150088136661 1.5707963267950271202
- joint lower_knee_left: origin xyz=-0.2174705007161515935 -0.33571800862966272305 -3.4694469519536141888e-18 rpy=-3.6654208353707214918e-17 7.4236255477340962066e-17 0.89630439304597309125 -> xyz=-0.21747050071615153799 -0.33571800862966250101 -1.3877787807814456755e-17 rpy=-3.6654208353707282711e-17 7.4236255477340986718e-17 0.89630439304596909444
- joint motor_ankle1: origin xyz=0 1.6653345369377348106e-16 0.043564478507036985544 rpy=3.1415926535897891192 2.698026123213506634e-15 3.1415926535897926719 -> xyz=0 0 0.043564478507036985544 rpy=3.1415926535897891192 2.6153764022898610303e-15 3.1415926535897926719
- joint motor_ankle1_left: origin xyz=-1.3877787807814456755e-17 1.0408340855860842566e-17 0.041658869056532793484 rpy=3.1415926535897820138 -6.6815401904784765465e-15 -3.1415926535897873428 -> xyz=0 4.8572257327350598644e-17 0.041658869056533182063 rpy=3.1415926535897820138 -6.7374372523019637495e-15 -3.1415926535897873428
- joint motor_ankle2_left: origin xyz=6.9388939039072283776e-17 2.7755575615628913511e-17 0.036860927393517151085 rpy=-3.141592653589793116 1.5408374369357243975e-14 -3.1415926535897824579 -> xyz=1.4988010832439613296e-15 0 0.036860927393518538864 rpy=-3.141592653589793116 1.5464271431180720134e-14 -3.1415926535897829019
- joint motor_hip_xy_1_left: origin xyz=1.3877787807814456755e-17 -0.044933728103784820185 -3.6602665343110629692e-16 rpy=-1.5707963267949507369 -8.3077011567330338006e-15 7.4116426331934598049e-15 -> xyz=-1.3877787807814456755e-17 -0.044933728103784570385 2.7755575615628913511e-17 rpy=-1.570796326794896558 -1.2579840982866257012e-14 7.4392748255148293694e-15
- joint motor_hip_xy_2_left: origin xyz=1.3877787807814456755e-17 -0.046444953521771831229 1.249000902703301108e-16 rpy=-1.5707963267948994446 2.6395580239470105185e-15 2.7853195712080230793e-15 -> xyz=4.1633363423443370266e-17 -0.046444953521772067151 0 rpy=-1.570796326794896558 7.4805795211536263427e-17 2.5368452273096694247e-15
- joint motor_hipz: origin xyz=-4.9960036108132044319e-16 -1.5959455978986625269e-16 -0.071499999999999813705 rpy=-6.0620461731129641165e-15 1.521560350042941006e-15 -1.5707963267949132113 -> xyz=-2.498001805406602216e-16 -1.8388068845354155201e-16 -0.071499999999999813705 rpy=-3.459434076669788135e-15 1.2825791172804655208e-15 -1.5707963267949132113
- joint motor_knee_left: origin xyz=4.8572257327350598644e-17 -2.498001805406602216e-16 0.0086304170048060457887 rpy=3.141592653589793116 -2.5197765118340936491e-15 -2.1135107621004381678e-15 -> xyz=2.8449465006019636348e-16 -1.1102230246251565404e-16 0.0086304170048063511 rpy=-3.141592653589793116 -1.9712230431965199595e-15 -2.1147901089949034214e-15
- joint spherical_actuation_knee_left: origin xyz=-0.01374999999999977629 -0.0024999999999999467093 -0.070875000000000007438 rpy=1.570796326794896558 3.5095903105758312051e-17 1.570796326794896558 -> xyz=-0.013749999999999821393 -0.0024999999999999744649 -0.070875000000000021316 rpy=1.570796326794896558 1.503667491693747211e-14 1.570796326794896558
- joint spherical_motor_transmission_hip1_left: origin xyz=0.043531328479973513401 0.0032046566522406227939 -0.02500000000000011241 rpy=1.5707963267948970021 -1.3881446540757382824 -3.1415926535897527039 -> xyz=0.043531328479973790957 0.0032046566522410530053 -0.024999999999999994449 rpy=1.5707963267948970021 -1.3881446540757560459 -3.1415926535897527039
- joint spherical_transmission_hip3_left: origin xyz=0.041074543378118194559 0.03657706776491259637 -0.00499999999999997842 rpy=-1.570796326794896558 0.67303436723393150753 3.1415926535897922278 -> xyz=0.041074543378118971715 0.036577067764912846171 -0.0050000000000000061756 rpy=-1.570796326794896558 0.67303436723391374397 3.1415926535897922278
- joint transmission_1_knee_left: origin xyz=-0.21747050071615153799 -0.33571800862966272305 0.0099999999999999741873 rpy=3.1415926535897922278 2.5607839141882122881e-15 3.0182803045709212242 -> xyz=-0.21747050071615148248 -0.33571800862966238999 0.009999999999999963779 rpy=3.1415926535897922278 2.5607839141882122881e-15 3.0182803045709176715
- joint transmission_2_knee_left: origin xyz=-0.2174705007161515935 -0.33571800862966272305 -0.01000000000000001929 rpy=3.1415926535897926719 2.4170968488441313662e-15 3.0435251672843857129 -> xyz=-0.21747050071615153799 -0.33571800862966250101 -0.010000000000000029698 rpy=3.1415926535897926719 2.4170968488441309718e-15 3.0435251672843821602
- joint transmission_ankle3_left: origin xyz=7.6327832942979512154e-17 -0.0467519999999999325 -0.05499999999999967415 rpy=-3.1415926535897908956 -1.2924964444112278435e-16 -1.249534074267399042 -> xyz=6.2450045135165055399e-17 -0.046752000000000043523 -0.055000000000000055789 rpy=-3.1415926535897895633 -4.7723251426136212841e-16 -1.2495340742673988199
- joint transmission_ankle4_left: origin xyz=4.5102810375396984455e-17 -0.046752000000000043523 -0.087999999999999994893 rpy=-1.544415098831094204e-14 6.0086890509720742404e-15 -1.2172645625816977955 -> xyz=7.1817551905439813709e-16 -0.04675200000000137579 -0.088000000000000341838 rpy=-9.0884089792933966647e-15 -1.2326465145342669532e-14 -1.2172645625816977955
- joint upper_knee_left: origin xyz=3.2265856653168611956e-16 -0.046752000000000043523 -0.071499999999999980238 rpy=-9.9086391638234093953e-15 1.3486642849930377956e-14 -0.63853922414919062067 -> xyz=7.2858385991025897965e-17 -0.046751999999999821478 -0.071500000000000313305 rpy=-1.4618783972762011617e-14 -5.3385657868507484047e-15 -0.63853922414918695694

Commit message: fix frame

File: example_parallel_robots/robots/kangaroo_like_2legs/robot.urdf (robot description, URDF)
Before this commit: robot onshape, 131 links, 130 joints
Links:
- removed link closedloop16_A_6D
- removed link closedloop16_B_6D
- removed link closedloop8_A_6D
- removed link closedloop8_B_6D
- added link closedloop16_A_3D, mass 1e-9
- added link closedloop16_B_3D, mass 1e-9
- added link closedloop8_A_3D, mass 1e-9
- added link closedloop8_B_3D, mass 1e-9
- link hanche_batis: mass 1.5865591647149872578 -> 1.5865591647149870358
- link hanche_batis_gauche: mass 1.5865591647149870358 -> 1.5865591647149868137
- link part_1: mass 0.24432174426363423292 -> 0.24432174426363428843
- link part_1_gauche: mass 0.24432174482850427255 -> 0.24432174482850421704
- link part_2: mass 0.39806472503371781446 -> 0.39806472503371786997
- link part_2_2: mass 0.39806472503371781446 -> 0.39806472503371786997
- link part_3: mass 0.2021348089396567127 -> 0.20213480893965668495
- link part_3_2: mass 0.2021348089396567127 -> 0.20213480893965668495
- link part_8: mass 0.0062040903886272725024 -> 0.006204090388627271635
- link part_8_2: mass 0.0062040903886272725024 -> 0.006204090388627271635
- link renvois_cheville: mass 0.074310321213953547947 -> 0.074310321213953561825
- link renvois_cheville_2: mass 0.074310321213953547947 -> 0.074310321213953561825
- link renvois_cheville_2_8: mass 0.074310320490072731547 -> 0.074310320490072745425
- link renvois_cheville_2_8_2: mass 0.074310320490072731547 -> 0.074310320490072745425
Joints:
- removed joint closedloop16_A_6D_frame
- removed joint closedloop16_B_6D_frame
- removed joint closedloop8_A_6D_frame
- removed joint closedloop8_B_6D_frame
- added joint closedloop16_A_3D_frame: type fixed, parent piston_6, child closedloop16_A_3D, origin xyz=0 2.0816681711721685133e-17 -0.022000000000000040357 rpy=3.8407815244357912106e-19 -7.2372460481629324552e-19 -1.0504212169390065499e-19, axis 0 0 0
- added joint closedloop16_B_3D_frame: type fixed, parent piston_3, child closedloop16_B_3D, origin xyz=2.0816681711721685133e-17 -2.7755575615628913511e-17 -0.021999999999999977907 rpy=3.141592653589793116 1.2701984792014930899e-16 -1.57079632679489678, axis 0 0 0
- added joint closedloop8_A_3D_frame: type fixed, parent piston_14, child closedloop8_A_3D, origin xyz=-8.3266726846886740532e-17 8.3266726846886740532e-17 -0.022000000000000075051 rpy=-3.141592653589793116 -7.5767938905805758326e-17 -1.570796326794896336, axis 0 0 0
- added joint closedloop8_B_3D_frame: type fixed, parent piston_17, child closedloop8_B_3D, origin xyz=-5.5511151231257827021e-17 -1.1275702593849246114e-17 -0.021999999999999950151 rpy=1.0351578883266661055e-15 -3.0410359695203482574e-16 1.5707963267948981123, axis 0 0 0
- joint 4rof_knee_left: origin xyz=0.046047631733747068639 -0.019483726843524284966 6.5919492087118669588e-17 rpy=3.141592653589793116 4.405771113082074377e-17 -1.2499268310990390152 -> xyz=0.046047631733746804961 -0.019483726843524645789 3.7470027081099033239e-16 rpy=-3.1415926535897922278 7.2938737706400957841e-16 -1.2499268310990416797
- joint free_motor_knee_left: origin xyz=-0.061655078133537329077 -0.018724201373191612374 4.2973576086513531891e-12 rpy=-1.5707963267948972241 1.3873492000155343007 -0.60601731071219733238 -> xyz=-0.061655078133537377649 -0.018724201373191806663 4.2973125058409777921e-12 rpy=-1.570796326794896558 1.3873492000155343007 -0.60601731071219677727
- joint lower_knee_left: origin xyz=-0.21747050071615153799 -0.33571800862966250101 -1.3877787807814456755e-17 rpy=-3.6654208353707282711e-17 7.4236255477340986718e-17 0.89630439304596909444 -> xyz=-0.21747050071615264821 -0.33571800862966216794 -1.8041124150158793782e-16 rpy=3.1711358110840073533e-17 -1.0781099766225485203e-15 0.89630439304596654093
- joint motor_knee_left: origin xyz=2.8449465006019636348e-16 -1.1102230246251565404e-16 0.0086304170048063511 rpy=-3.141592653589793116 -1.9712230431965199595e-15 -2.1147901089949034214e-15 -> xyz=-2.7755575615628913511e-17 2.7755575615628913511e-17 0.0086304170048063233445 rpy=-3.1415926535897908956 -2.5334648372852549721e-15 -2.1764592995127995022e-15
- joint transmission_1_knee_left: origin xyz=-0.21747050071615148248 -0.33571800862966238999 0.009999999999999963779 rpy=3.1415926535897922278 2.5607839141882122881e-15 3.0182803045709176715 -> xyz=-0.21747050071615253719 -0.33571800862966216794 0.0099999999999997972455 rpy=3.1415926535897913396 3.1061264621411137395e-15 3.0182803045709150069
- joint transmission_2_knee_left: origin xyz=-0.21747050071615153799 -0.33571800862966250101 -0.010000000000000029698 rpy=3.1415926535897926719 2.4170968488441309718e-15 3.0435251672843821602 -> xyz=-0.2174705007161525927 -0.33571800862966216794 -0.010000000000000192762 rpy=3.1415926535897917837 2.9873864412696137094e-15 3.0435251672843794957
- joint upper_knee_left: origin xyz=7.2858385991025897965e-17 -0.046751999999999821478 -0.071500000000000313305 rpy=-1.4618783972762011617e-14 -5.3385657868507484047e-15 -0.63853922414918695694 -> xyz=3.7816971776294394658e-16 -0.046751999999999793722 -0.071500000000000618616 rpy=-1.556236804210751295e-14 -4.6707669583509065136e-15 -0.63853922414918418138
