Commit message: update kangaroo 2 legs  to new standard

File: example_parallel_robots/robots/kangaroo_like_2legs/robot.urdf (robot description, URDF)
Before this commit: robot onshape, 131 links, 130 joints
Links:
- removed link attache_hanche
- removed link attache_hanche_2
- removed link cardan_foot
- removed link cardan_foot_2
- removed link cardan_foot_3
- removed link cardan_foot_4
- removed link cardan_hache
- removed link cardan_hache_2
- removed link cardan_hache_3
- removed link cardan_hache_4
- removed link hanche
- removed link hanche_batis
- removed link moteur_hanche1
- removed link moteur_hanche1_2
- removed link moteur_hanche1_3
- removed link moteur_hanche1_4
- removed link motteur_rotation
- removed link motteur_rotation_2
- removed link motteur_rotation_3
- removed link motteur_rotation_4
- removed link motteur_rotation_5
- removed link motteur_rotation_6
- removed link motteur_rotation_7
- removed link motteur_rotation_8
- removed link piston
- removed link piston_10
- removed link piston_11
- removed link piston_12
- removed link piston_13
- removed link piston_14
- removed link piston_15
- removed link piston_16
- removed link piston_17
- removed link piston_18
- removed link piston_19
- removed link piston_2
- removed link piston_20
- removed link piston_21
- removed link piston_22
- removed link piston_23
- removed link piston_24
- removed link piston_3
- removed link piston_4
- removed link piston_5
- removed link piston_6
- removed link piston_7
- removed link piston_8
- removed link piston_9
- removed link renvois_cheville
- removed link renvois_cheville_2
- removed link renvois_cheville_2_8
- removed link renvois_cheville_2_8_2
- added link cylinder, mass 0.0047041422996690132607; collision mesh filename=package:///cylinder.stl; visual mesh filename=package:///cylinder.stl
- added link cylinder_10, mass 0.0047041422996690132607; collision mesh filename=package:///cylinder.stl; visual mesh filename=package:///cylinder.stl
- added link cylinder_11, mass 0.0047041422996690132607; collision mesh filename=package:///cylinder.stl; visual mesh filename=package:///cylinder.stl
- added link cylinder_12, mass 0.0047041422996690132607; collision mesh filename=package:///cylinder.stl; visual mesh filename=package:///cylinder.stl
- added link cylinder_13, mass 0.0047041422996690132607; collision mesh filename=package:///cylinder.stl; visual mesh filename=package:///cylinder.stl
- added link cylinder_14, mass 0.0047041422996690132607; collision mesh filename=package:///cylinder.stl; visual mesh filename=package:///cylinder.stl
- added link cylinder_15, mass 0.0047041422996690132607; collision mesh filename=package:///cylinder.stl; visual mesh filename=package:///cylinder.stl
- added link cylinder_16, mass 0.0047041422996690132607; collision mesh filename=package:///cylinder.stl; visual mesh filename=package:///cylinder.stl
- added link cylinder_17, mass 0.0047041422996690132607; collision mesh filename=package:///cylinder.stl; visual mesh filename=package:///cylinder.stl
- added link cylinder_18, mass 0.0047041422996690132607; collision mesh filename=package:///cylinder.stl; visual mesh filename=package:///cylinder.stl
- added link cylinder_19, mass 0.0047041422996690132607; collision mesh filename=package:///cylinder.stl; visual mesh filename=package:///cylinder.stl
- added link cylinder_2, mass 0.0047041422996690132607; collision mesh filename=package:///cylinder.stl; visual mesh filename=package:///cylinder.stl
- added link cylinder_20, mass 0.0047041422996690132607; collision mesh filename=package:///cylinder.stl; visual mesh filename=package:///cylinder.stl
- added link cylinder_21, mass 0.0047041422996690132607; collision mesh filename=package:///cylinder.stl; visual mesh filename=package:///cylinder.stl
- added link cylinder_22, mass 0.0047041422996690132607; collision mesh filename=package:///cylinder.stl; visual mesh filename=package:///cylinder.stl
- added link cylinder_23, mass 0.0047041422996690132607; collision mesh filename=package:///cylinder.stl; visual mesh filename=package:///cylinder.stl
- added link cylinder_24, mass 0.0047041422996690132607; collision mesh filename=package:///cylinder.stl; visual mesh filename=package:///cylinder.stl
- added link cylinder_3, mass 0.0047041422996690132607; collision mesh filename=package:///cylinder.stl; visual mesh filename=package:///cylinder.stl
- added link cylinder_4, mass 0.0047041422996690132607; collision mesh filename=package:///cylinder.stl; visual mesh filename=package:///cylinder.stl
- added link cylinder_5, mass 0.0047041422996690132607; collision mesh filename=package:///cylinder.stl; visual mesh filename=package:///cylinder.stl
- added link cylinder_6, mass 0.0047041422996690132607; collision mesh filename=package:///cylinder.stl; visual mesh filename=package:///cylinder.stl
- added link cylinder_7, mass 0.0047041422996690132607; collision mesh filename=package:///cylinder.stl; visual mesh filename=package:///cylinder.stl
- added link cylinder_8, mass 0.0047041422996690132607; collision mesh filename=package:///cylinder.stl; visual mesh filename=package:///cylinder.stl
- added link cylinder_9, mass 0.0047041422996690132607; collision mesh filename=package:///cylinder.stl; visual mesh filename=package:///cylinder.stl
- added link hip, mass 0.14908820646980494584; collision mesh filename=package:///hip.stl; visual mesh filename=package:///hip.stl
- added link hip_ground, mass 1.5865591647149870358; collision mesh filename=package:///hip_ground.stl; visual mesh filename=package:///hip_ground.stl
- added link holder_hip, mass 0.01282947899909727546; collision mesh filename=package:///holder_hip.stl; visual mesh filename=package:///holder_hip.stl
- added link holder_hip_2, mass 0.01282947899909727546; collision mesh filename=package:///holder_hip.stl; visual mesh filename=package:///holder_hip.stl
- added link motor_hip1, mass 0.17794962537636813127; collision mesh filename=package:///motor_hip1.stl; visual mesh filename=package:///motor_hip1.stl
- added link motor_hip1_2, mass 0.17794962537636813127; collision mesh filename=package:///motor_hip1.stl; visual mesh filename=package:///motor_hip1.stl
- added link motor_hip1_3, mass 0.17794962537636813127; collision mesh filename=package:///motor_hip1.stl; visual mesh filename=package:///motor_hip1.stl
- added link motor_hip1_4, mass 0.17794962537636813127; collision mesh filename=package:///motor_hip1.stl; visual mesh filename=package:///motor_hip1.stl
- added link rotation_motor, mass 0.19339251676417062997; collision mesh filename=package:///rotation_motor.stl; visual mesh filename=package:///rotation_motor.stl
- added link rotation_motor_2, mass 0.19339251676417062997; collision mesh filename=package:///rotation_motor.stl; visual mesh filename=package:///rotation_motor.stl
- added link rotation_motor_3, mass 0.19339251676417062997; collision mesh filename=package:///rotation_motor.stl; visual mesh filename=package:///rotation_motor.stl
- added link rotation_motor_4, mass 0.19339251676417062997; collision mesh filename=package:///rotation_motor.stl; visual mesh filename=package:///rotation_motor.stl
- added link rotation_motor_5, mass 0.19339251676417062997; collision mesh filename=package:///rotation_motor.stl; visual mesh filename=package:///rotation_motor.stl
- added link rotation_motor_6, mass 0.19339251676417062997; collision mesh filename=package:///rotation_motor.stl; visual mesh filename=package:///rotation_motor.stl
- added link rotation_motor_7, mass 0.19339251676417062997; collision mesh filename=package:///rotation_motor.stl; visual mesh filename=package:///rotation_motor.stl
- added link rotation_motor_8, mass 0.19339251676417062997; collision mesh filename=package:///rotation_motor.stl; visual mesh filename=package:///rotation_motor.stl
- added link transmission_ankle, mass 0.074310321213953561825; collision mesh filename=package:///transmission_ankle.stl; visual mesh filename=package:///transmission_ankle.stl
- added link transmission_ankle2, mass 0.074310320490072745425; collision mesh filename=package:///transmission_ankle2.stl; visual mesh filename=package:///transmission_ankle2.stl
- added link transmission_ankle2_2, mass 0.074310320490072745425; collision mesh filename=package:///transmission_ankle2.stl; visual mesh filename=package:///transmission_ankle2.stl
- added link transmission_ankle_2, mass 0.074310321213953561825; collision mesh filename=package:///transmission_ankle.stl; visual mesh filename=package:///transmission_ankle.stl
- added link universal_foot, mass 0.0064135211594024202353; collision mesh filename=package:///universal_foot.stl; visual mesh filename=package:///universal_foot.stl
- added link universal_foot_2, mass 0.0064135211594024202353; collision mesh filename=package:///universal_foot.stl; visual mesh filename=package:///universal_foot.stl
- added link universal_foot_3, mass 0.0064135211594024202353; collision mesh filename=package:///universal_foot.stl; visual mesh filename=package:///universal_foot.stl
- added link universal_foot_4, mass 0.0064135211594024202353; collision mesh filename=package:///universal_foot.stl; visual mesh filename=package:///universal_foot.stl
- added link universal_hip, mass 0.015608633111865791165; collision mesh filename=package:///universal_hip.stl; visual mesh filename=package:///universal_hip.stl
- added link universal_hip_2, mass 0.015608633111865791165; collision mesh filename=package:///universal_hip.stl; visual mesh filename=package:///universal_hip.stl
- added link universal_hip_3, mass 0.015608633111865791165; collision mesh filename=package:///universal_hip.stl; visual mesh filename=package:///universal_hip.stl
- added link universal_hip_4, mass 0.015608633111865791165; collision mesh filename=package:///universal_hip.stl; visual mesh filename=package:///universal_hip.stl
- link foot: mass 0.3109129822293019707 -> 0.31091298222930191519
- link foot_2: mass 0.3109129822293019707 -> 0.31091298222930191519
- link hanche_batis_gauche: mass 1.5865591647149868137 -> 1.5865591647149870358
- link part_2: mass 0.39806472503371786997 -> 0.39806472503371781446
- link part_2_2: mass 0.39806472503371786997 -> 0.39806472503371781446
- link part_3: mass 0.20213480893965668495 -> 0.2021348089396567127
- link part_3_2: mass 0.20213480893965668495 -> 0.2021348089396567127
- link part_8: mass 0.006204090388627271635 -> 0.0062040903886272707676
- link part_8_2: mass 0.006204090388627271635 -> 0.0062040903886272707676
- link part_9: mass 0.0062040903886272707676 -> 0.0062040903886272699003
- link part_9_2: mass 0.0062040903886272707676 -> 0.0062040903886272699003
Joints:
- joint center_hip_frame: parent hanche_batis -> hip_ground
- joint closedloop10_B_3D_frame: parent renvois_cheville_2_8_2 -> transmission_ankle2_2
- joint closedloop14_A_3D_frame: parent piston_4 -> cylinder_4
- joint closedloop14_B_3D_frame: parent piston_8 -> cylinder_8
- joint closedloop15_A_3D_frame: parent piston_7 -> cylinder_7
- joint closedloop15_B_3D_frame: parent piston_5 -> cylinder_5
- joint closedloop16_A_3D_frame: parent piston_6 -> cylinder_6
- joint closedloop16_B_3D_frame: parent piston_3 -> cylinder_3
- joint closedloop17_A_6D_frame: parent piston -> cylinder
- joint closedloop17_B_6D_frame: parent piston_10 -> cylinder_10
- joint closedloop18_A_6D_frame: parent piston_2 -> cylinder_2
- joint closedloop18_B_6D_frame: parent piston_11 -> cylinder_11
- joint closedloop19_A_6D_frame: parent piston_24 -> cylinder_24
- joint closedloop19_B_6D_frame: parent piston_9 -> cylinder_9
- joint closedloop1_A_3D_frame: parent piston_18 -> cylinder_18
- joint closedloop1_B_3D_frame: parent piston_15 -> cylinder_15
- joint closedloop20_B_3D_frame: parent renvois_cheville -> transmission_ankle
- joint closedloop23_B_3D_frame: parent renvois_cheville_2_8 -> transmission_ankle2
- joint closedloop2_A_3D_frame: parent piston_19 -> cylinder_19
- joint closedloop2_B_3D_frame: parent piston_16 -> cylinder_16
- joint closedloop3_A_6D_frame: parent piston_12 -> cylinder_12
- joint closedloop3_B_6D_frame: parent piston_21 -> cylinder_21
- joint closedloop4_A_6D_frame: parent piston_13 -> cylinder_13
- joint closedloop4_B_6D_frame: parent piston_20 -> cylinder_20
- joint closedloop5_A_6D_frame: parent piston_23 -> cylinder_23
- joint closedloop5_B_6D_frame: parent piston_22 -> cylinder_22
- joint closedloop8_A_3D_frame: parent piston_14 -> cylinder_14
- joint closedloop8_B_3D_frame: parent piston_17 -> cylinder_17
- joint closedloop9_B_3D_frame: parent renvois_cheville_2 -> transmission_ankle_2
- joint frame_motor_ankle1: child motteur_rotation_5 -> rotation_motor_5
- joint frame_motor_ankle1_left: child motteur_rotation_2 -> rotation_motor_2
- joint frame_motor_ankle2: child motteur_rotation_6 -> rotation_motor_6
- joint frame_motor_ankle2_left: child motteur_rotation_3 -> rotation_motor_3
- joint frame_motor_knee: child motteur_rotation_4 -> rotation_motor_4
- joint free_ankle_universal_x_left: parent cardan_foot_2 -> universal_foot_2
- joint free_ankle_universalx: parent cardan_foot_4 -> universal_foot_4
- joint free_motor_holder_1: child cardan_hache_3 -> universal_hip_3; parent hanche -> hip
- joint free_motor_holder_1_left: child cardan_hache -> universal_hip
- joint free_motor_holder_2: child attache_hanche -> holder_hip; parent hanche_batis -> hip_ground
- joint free_motor_holder_2_left: child cardan_hache_2 -> universal_hip_2
- joint free_motor_holder_3: child cardan_hache_4 -> universal_hip_4; parent hanche -> hip
- joint free_motor_holder_hip_xy1_left: child moteur_hanche1_2 -> motor_hip1_2; parent cardan_hache_2 -> universal_hip_2
- joint free_motor_holder_hip_xy2_left: child moteur_hanche1 -> motor_hip1; parent cardan_hache -> universal_hip
- joint free_motor_holder_hipxy1: child moteur_hanche1_4 -> motor_hip1_4; parent cardan_hache_4 -> universal_hip_4
- joint free_motor_holder_hipxy2: child moteur_hanche1_3 -> motor_hip1_3; parent cardan_hache_3 -> universal_hip_3
- joint free_motor_knee_left: child motteur_rotation -> rotation_motor
- joint free_spherical_hip_xy_1_left: child piston -> cylinder
- joint free_spherical_hipxy_2_left: child piston_2 -> cylinder_2
- joint free_spherical_motor_holder_1: child motteur_rotation_7 -> rotation_motor_7; parent attache_hanche -> holder_hip
- joint free_spherical_motor_holder_hipz: child piston_22 -> cylinder_22; parent hanche -> hip
- joint free_universal_motor_holder_hipz_left: child attache_hanche_2 -> holder_hip_2
- joint free_universal_x_hip_left: child cardan_foot -> universal_foot
- joint free_universal_y_foot_left: child cardan_foot_2 -> universal_foot_2
- joint free_universal_y_hip_left: parent cardan_foot -> universal_foot
- joint free_universal_yhip: child cardan_foot_3 -> universal_foot_3; parent hanche -> hip
- joint free_zhip: child hanche -> hip; parent hanche_batis -> hip_ground
- joint lower_hip: parent cardan_foot_3 -> universal_foot_3
- joint motor_ankle1: child piston_19 -> cylinder_19; parent motteur_rotation_6 -> rotation_motor_6
- joint motor_ankle1_left: child piston_8 -> cylinder_8; parent motteur_rotation_3 -> rotation_motor_3
- joint motor_ankle2: child piston_18 -> cylinder_18; parent motteur_rotation_5 -> rotation_motor_5
- joint motor_ankle2_left: child piston_7 -> cylinder_7; parent motteur_rotation_2 -> rotation_motor_2
- joint motor_hip_xy_1: child piston_21 -> cylinder_21; parent moteur_hanche1_4 -> motor_hip1_4
- joint motor_hip_xy_1_left: child piston_10 -> cylinder_10; parent moteur_hanche1 -> motor_hip1
- joint motor_hip_xy_2: child piston_20 -> cylinder_20; parent moteur_hanche1_3 -> motor_hip1_3
- joint motor_hip_xy_2_left: child piston_11 -> cylinder_11; parent moteur_hanche1_2 -> motor_hip1_2
- joint motor_hip_z_left: child piston_24 -> cylinder_24; parent motteur_rotation_8 -> rotation_motor_8
- joint motor_hipz: child piston_23 -> cylinder_23; parent motteur_rotation_7 -> rotation_motor_7
- joint motor_knee: child piston_14 -> cylinder_14; parent motteur_rotation_4 -> rotation_motor_4
- joint motor_knee_left: child piston_3 -> cylinder_3; parent motteur_rotation -> rotation_motor
- joint spherical_actuation_knee_left: child piston_6 -> cylinder_6
- joint spherical_free_hip_left: child piston_9 -> cylinder_9
- joint spherical_lower_hip1: child piston_12 -> cylinder_12
- joint spherical_lower_hip2: child piston_13 -> cylinder_13
- joint spherical_motor_holder_hip_z_left: child motteur_rotation_8 -> rotation_motor_8; parent attache_hanche_2 -> holder_hip_2
- joint spherical_motor_knee_holder: child piston_17 -> cylinder_17
- joint spherical_motor_transmission_hip1_left: child piston_4 -> cylinder_4
- joint spherical_motor_transmission_hip2_left: child piston_5 -> cylinder_5
- joint spherical_transmission_foot1: parent renvois_cheville_2 -> transmission_ankle_2
- joint spherical_transmission_foot1_left: parent renvois_cheville -> transmission_ankle
- joint spherical_transmission_foot2: parent renvois_cheville_2_8_2 -> transmission_ankle2_2
- joint spherical_transmission_foot2_left: parent renvois_cheville_2_8 -> transmission_ankle2
- joint spherical_transmission_motor_hip1: child piston_15 -> cylinder_15
- joint spherical_transmission_motor_hip2: child piston_16 -> cylinder_16
- joint test: child hanche_batis -> hip_ground
- joint transmission_1_knee_left: child renvois_cheville_2_8 -> transmission_ankle2
- joint transmission_2_knee_left: child renvois_cheville -> transmission_ankle
- joint triangle_knee1: child renvois_cheville_2_8_2 -> transmission_ankle2_2
- joint triangle_knee2: child renvois_cheville_2 -> transmission_ankle_2
- joint uneveral_foot1: child cardan_foot_4 -> universal_foot_4
