Commit message: kangaroo 2 legs modified

File: example_parallel_robots/robots/kangaroo_like_2legs/robot.urdf (robot description, URDF)
Before this commit: robot onshape, 131 links, 130 joints
Links:
- added link hanche_gauche_int1_12, mass 0.0
- added link hanche_gauche_int2_12, mass 0.0
- added link hip_int1_24, mass 0.0
- added link hip_int2_24, mass 0.0
- added link holder_hip_2_int1_26, mass 0.0
- added link holder_hip_2_int2_26, mass 0.0
- added link holder_hip_int1_25, mass 0.0
- added link holder_hip_int2_25, mass 0.0
- added link part_1_gauche_int1_1, mass 0.0
- added link part_1_gauche_int1_11, mass 0.0
- added link part_1_gauche_int1_2, mass 0.0
- added link part_1_gauche_int2_1, mass 0.0
- added link part_1_gauche_int2_11, mass 0.0
- added link part_1_gauche_int2_2, mass 0.0
- added link part_1_int1_13, mass 0.0
- added link part_1_int1_14, mass 0.0
- added link part_1_int1_23, mass 0.0
- added link part_1_int2_13, mass 0.0
- added link part_1_int2_14, mass 0.0
- added link part_1_int2_23, mass 0.0
- added link part_3_2_int1_15, mass 0.0
- added link part_3_2_int2_15, mass 0.0
- added link part_3_int1_3, mass 0.0
- added link part_3_int2_3, mass 0.0
- added link part_4_2_int1_18, mass 0.0
- added link part_4_2_int2_18, mass 0.0
- added link part_4_int1_6, mass 0.0
- added link part_4_int2_6, mass 0.0
- added link part_8_2_int1_19, mass 0.0
- added link part_8_2_int1_20, mass 0.0
- added link part_8_2_int2_19, mass 0.0
- added link part_8_2_int2_20, mass 0.0
- added link part_8_int1_7, mass 0.0
- added link part_8_int1_8, mass 0.0
- added link part_8_int2_7, mass 0.0
- added link part_8_int2_8, mass 0.0
- added link part_9_2_int1_21, mass 0.0
- added link part_9_2_int1_22, mass 0.0
- added link part_9_2_int2_21, mass 0.0
- added link part_9_2_int2_22, mass 0.0
- added link part_9_int1_10, mass 0.0
- added link part_9_int1_9, mass 0.0
- added link part_9_int2_10, mass 0.0
- added link part_9_int2_9, mass 0.0
- added link transmission_ankle2_2_int1_16, mass 0.0
- added link transmission_ankle2_2_int2_16, mass 0.0
- added link transmission_ankle2_int1_4, mass 0.0
- added link transmission_ankle2_int2_4, mass 0.0
- added link transmission_ankle_2_int1_17, mass 0.0
- added link transmission_ankle_2_int2_17, mass 0.0
- added link transmission_ankle_int1_5, mass 0.0
- added link transmission_ankle_int2_5, mass 0.0
Joints:
- removed joint free_spherical_hip_xy_1_left
- removed joint free_spherical_hipxy_2_left
- removed joint free_spherical_motor_holder_1
- removed joint free_spherical_motor_holder_hipz
- removed joint spherical_4rod
- removed joint spherical_4rod_left
- removed joint spherical_actuation_knee_left
- removed joint spherical_free_hip_left
- removed joint spherical_lower_hip1
- removed joint spherical_lower_hip2
- removed joint spherical_motor_holder_hip_z_left
- removed joint spherical_motor_knee_holder
- removed joint spherical_motor_transmission_hip1_left
- removed joint spherical_motor_transmission_hip2_left
- removed joint spherical_shin_left
- removed joint spherical_shin_rod1
- removed joint spherical_transmission_foot1
- removed joint spherical_transmission_foot1_left
- removed joint spherical_transmission_foot2
- removed joint spherical_transmission_foot2_left
- removed joint spherical_transmission_hip3
- removed joint spherical_transmission_hip3_left
- removed joint spherical_transmission_hip4
- removed joint spherical_transmission_hip4_left
- removed joint spherical_transmission_motor_hip1
- removed joint spherical_transmission_motor_hip2
- added joint hanche_gauche_cylinder_9_rev0: type revolute, parent hanche_gauche, child hanche_gauche_int1_12, origin xyz=3.1537272793258352976e-15 -0.03850000000000006195 -0.046750000000000027645, axis 1 0 0, limit effort=1 velocity=20
- added joint hanche_gauche_cylinder_9_rev1: type revolute, parent hanche_gauche_int1_12, child hanche_gauche_int2_12, axis 0 1 0, limit effort=1 velocity=20
- added joint hanche_gauche_cylinder_9_rev2: type revolute, parent hanche_gauche_int2_12, child cylinder_9, axis 0 0 1, limit effort=1 velocity=20
- added joint hip_cylinder_22_rev0: type revolute, parent hip, child hip_int1_24, origin xyz=3.380976054678797027e-15 0.038499999999999978684 -0.046750000000000131728, axis 1 0 0, limit effort=1 velocity=20
- added joint hip_cylinder_22_rev1: type revolute, parent hip_int1_24, child hip_int2_24, axis 0 1 0, limit effort=1 velocity=20
- added joint hip_cylinder_22_rev2: type revolute, parent hip_int2_24, child cylinder_22, axis 0 0 1, limit effort=1 velocity=20
- added joint holder_hip_2_rotation_motor_8_rev0: type revolute, parent holder_hip_2, child holder_hip_2_int1_26, origin xyz=-1.3877787807814456755e-17 2.7755575615628913511e-17 -0.051749999999999934941, axis 1 0 0, limit effort=1 velocity=20
- added joint holder_hip_2_rotation_motor_8_rev1: type revolute, parent holder_hip_2_int1_26, child holder_hip_2_int2_26, axis 0 1 0, limit effort=1 velocity=20
- added joint holder_hip_2_rotation_motor_8_rev2: type revolute, parent holder_hip_2_int2_26, child rotation_motor_8, axis 0 0 1, limit effort=1 velocity=20
- added joint holder_hip_rotation_motor_7_rev0: type revolute, parent holder_hip, child holder_hip_int1_25, origin xyz=-1.3877787807814456755e-17 0 -0.051749999999999886369, axis 1 0 0, limit effort=1 velocity=20
- added joint holder_hip_rotation_motor_7_rev1: type revolute, parent holder_hip_int1_25, child holder_hip_int2_25, axis 0 1 0, limit effort=1 velocity=20
- added joint holder_hip_rotation_motor_7_rev2: type revolute, parent holder_hip_int2_25, child rotation_motor_7, axis 0 0 1, limit effort=1 velocity=20
- added joint part_1_cylinder_12_rev0: type revolute, parent part_1, child part_1_int1_13, origin xyz=-0.060500000000000109246 2.7755575615628913511e-17 -0.038499999999999978684, axis 1 0 0, limit effort=1 velocity=20
- added joint part_1_cylinder_12_rev1: type revolute, parent part_1_int1_13, child part_1_int2_13, axis 0 1 0, limit effort=1 velocity=20
- added joint part_1_cylinder_12_rev2: type revolute, parent part_1_int2_13, child cylinder_12, axis 0 0 1, limit effort=1 velocity=20
- added joint part_1_cylinder_13_rev0: type revolute, parent part_1, child part_1_int1_14, origin xyz=-0.06050000000000008149 -8.3266726846886740532e-17 0.038500000000000006439, axis 1 0 0, limit effort=1 velocity=20
- added joint part_1_cylinder_13_rev1: type revolute, parent part_1_int1_14, child part_1_int2_14, axis 0 1 0, limit effort=1 velocity=20
- added joint part_1_cylinder_13_rev2: type revolute, parent part_1_int2_14, child cylinder_13, axis 0 0 1, limit effort=1 velocity=20
- added joint part_1_cylinder_17_rev0: type revolute, parent part_1, child part_1_int1_23, origin xyz=-0.013750000000000071193 0.0024999999999999744649 -0.072000000000000008438, axis 1 0 0, limit effort=1 velocity=20
- added joint part_1_cylinder_17_rev1: type revolute, parent part_1_int1_23, child part_1_int2_23, axis 0 1 0, limit effort=1 velocity=20
- added joint part_1_cylinder_17_rev2: type revolute, parent part_1_int2_23, child cylinder_17, axis 0 0 1, limit effort=1 velocity=20
- added joint part_1_gauche_cylinder_2_rev0: type revolute, parent part_1_gauche, child part_1_gauche_int1_2, origin xyz=-0.06049999999999995659 8.3266726846886740532e-17 0.038499999999999964806, axis 1 0 0, limit effort=1 velocity=20
- added joint part_1_gauche_cylinder_2_rev1: type revolute, parent part_1_gauche_int1_2, child part_1_gauche_int2_2, axis 0 1 0, limit effort=1 velocity=20
- added joint part_1_gauche_cylinder_2_rev2: type revolute, parent part_1_gauche_int2_2, child cylinder_2, axis 0 0 1, limit effort=1 velocity=20
- added joint part_1_gauche_cylinder_6_rev0: type revolute, parent part_1_gauche, child part_1_gauche_int1_11, origin xyz=-0.013749999999999821393 -0.0024999999999999744649 -0.070875000000000021316, axis 1 0 0, limit effort=1 velocity=20
- added joint part_1_gauche_cylinder_6_rev1: type revolute, parent part_1_gauche_int1_11, child part_1_gauche_int2_11, axis 0 1 0, limit effort=1 velocity=20
- added joint part_1_gauche_cylinder_6_rev2: type revolute, parent part_1_gauche_int2_11, child cylinder_6, axis 0 0 1, limit effort=1 velocity=20
- added joint part_1_gauche_cylinder_rev0: type revolute, parent part_1_gauche, child part_1_gauche_int1_1, origin xyz=-0.06049999999999995659 1.3877787807814456755e-16 -0.038500000000000034195, axis 1 0 0, limit effort=1 velocity=20
- added joint part_1_gauche_cylinder_rev1: type revolute, parent part_1_gauche_int1_1, child part_1_gauche_int2_1, axis 0 1 0, limit effort=1 velocity=20
- added joint part_1_gauche_cylinder_rev2: type revolute, parent part_1_gauche_int2_1, child cylinder, axis 0 0 1, limit effort=1 velocity=20
- added joint part_3_2_part_6_2_rev0: type revolute, parent part_3_2, child part_3_2_int1_15, origin xyz=0.038967453687049735667 -0.092095263467496718546 1.1102230246251565404e-16, axis 1 0 0, limit effort=1 velocity=20
- added joint part_3_2_part_6_2_rev1: type revolute, parent part_3_2_int1_15, child part_3_2_int2_15, axis 0 1 0, limit effort=1 velocity=20
- added joint part_3_2_part_6_2_rev2: type revolute, parent part_3_2_int2_15, child part_6_2, axis 0 0 1, limit effort=1 velocity=20
- added joint part_3_part_6_rev0: type revolute, parent part_3, child part_3_int1_3, origin xyz=0.038967453687049735667 -0.092095263467496746301 -6.9388939039072283776e-18, axis 1 0 0, limit effort=1 velocity=20
- added joint part_3_part_6_rev1: type revolute, parent part_3_int1_3, child part_3_int2_3, axis 0 1 0, limit effort=1 velocity=20
- added joint part_3_part_6_rev2: type revolute, parent part_3_int2_3, child part_6, axis 0 0 1, limit effort=1 velocity=20
- added joint part_4_2_part_5_2_rev0: type revolute, parent part_4_2, child part_4_2_int1_18, origin xyz=0.0194837268435249511 -0.046047631733748387028 0, axis 1 0 0, limit effort=1 velocity=20
- added joint part_4_2_part_5_2_rev1: type revolute, parent part_4_2_int1_18, child part_4_2_int2_18, axis 0 1 0, limit effort=1 velocity=20
- added joint part_4_2_part_5_2_rev2: type revolute, parent part_4_2_int2_18, child part_5_2, axis 0 0 1, limit effort=1 velocity=20
- added joint part_4_part_5_rev0: type revolute, parent part_4, child part_4_int1_6, origin xyz=0.019483726843525006611 -0.046047631733748345395 1.0408340855860842566e-17, axis 1 0 0, limit effort=1 velocity=20
- added joint part_4_part_5_rev1: type revolute, parent part_4_int1_6, child part_4_int2_6, axis 0 1 0, limit effort=1 velocity=20
- added joint part_4_part_5_rev2: type revolute, parent part_4_int2_6, child part_5, axis 0 0 1, limit effort=1 velocity=20
- added joint part_8_2_cylinder_15_rev0: type revolute, parent part_8_2, child part_8_2_int1_19, origin xyz=0.043531328479973735446 0.0032046566522409003497 -0.025000000000000077716, axis 1 0 0, limit effort=1 velocity=20
- added joint part_8_2_cylinder_15_rev1: type revolute, parent part_8_2_int1_19, child part_8_2_int2_19, axis 0 1 0, limit effort=1 velocity=20
- added joint part_8_2_cylinder_15_rev2: type revolute, parent part_8_2_int2_19, child cylinder_15, axis 0 0 1, limit effort=1 velocity=20
- added joint part_8_2_part_7_7_rev0: type revolute, parent part_8_2, child part_8_2_int1_20, origin xyz=0.041074543378118805181 0.036577067764912860048 -0.0050000000000000044409, axis 1 0 0, limit effort=1 velocity=20
- added joint part_8_2_part_7_7_rev1: type revolute, parent part_8_2_int1_20, child part_8_2_int2_20, axis 0 1 0, limit effort=1 velocity=20
- added joint part_8_2_part_7_7_rev2: type revolute, parent part_8_2_int2_20, child part_7_7, axis 0 0 1, limit effort=1 velocity=20
- added joint part_8_cylinder_4_rev0: type revolute, parent part_8, child part_8_int1_7, origin xyz=0.043531328479973790957 0.0032046566522410530053 -0.024999999999999994449, axis 1 0 0, limit effort=1 velocity=20
- added joint part_8_cylinder_4_rev1: type revolute, parent part_8_int1_7, child part_8_int2_7, axis 0 1 0, limit effort=1 velocity=20
- added joint part_8_cylinder_4_rev2: type revolute, parent part_8_int2_7, child cylinder_4, axis 0 0 1, limit effort=1 velocity=20
- added joint part_8_part_7_3_rev0: type revolute, parent part_8, child part_8_int1_8, origin xyz=0.041074543378118971715 0.036577067764912846171 -0.0050000000000000061756, axis 1 0 0, limit effort=1 velocity=20
- added joint part_8_part_7_3_rev1: type revolute, parent part_8_int1_8, child part_8_int2_8, axis 0 1 0, limit effort=1 velocity=20
- added joint part_8_part_7_3_rev2: type revolute, parent part_8_int2_8, child part_7_3, axis 0 0 1, limit effort=1 velocity=20
- added joint part_9_2_cylinder_16_rev0: type revolute, parent part_9_2, child part_9_2_int1_21, origin xyz=0.04353132847997370769 -0.0032046566522409836164 -0.024999999999999994449, axis 1 0 0, limit effort=1 velocity=20
- added joint part_9_2_cylinder_16_rev1: type revolute, parent part_9_2_int1_21, child part_9_2_int2_21, axis 0 1 0, limit effort=1 velocity=20
- added joint part_9_2_cylinder_16_rev2: type revolute, parent part_9_2_int2_21, child cylinder_16, axis 0 0 1, limit effort=1 velocity=20
- added joint part_9_2_part_7_8_rev0: type revolute, parent part_9_2, child part_9_2_int1_22, origin xyz=0.041074543378118943959 -0.036577067764912887804 -0.005000000000000059952, axis 1 0 0, limit effort=1 velocity=20
- added joint part_9_2_part_7_8_rev1: type revolute, parent part_9_2_int1_22, child part_9_2_int2_22, axis 0 1 0, limit effort=1 velocity=20
- added joint part_9_2_part_7_8_rev2: type revolute, parent part_9_2_int2_22, child part_7_8, axis 0 0 1, limit effort=1 velocity=20
- added joint part_9_cylinder_5_rev0: type revolute, parent part_9, child part_9_int1_9, origin xyz=0.043531328479973624423 -0.0032046566522409697386 -0.025000000000000022204, axis 1 0 0, limit effort=1 velocity=20
- added joint part_9_cylinder_5_rev1: type revolute, parent part_9_int1_9, child part_9_int2_9, axis 0 1 0, limit effort=1 velocity=20
- added joint part_9_cylinder_5_rev2: type revolute, parent part_9_int2_9, child cylinder_5, axis 0 0 1, limit effort=1 velocity=20
- added joint part_9_part_7_4_rev0: type revolute, parent part_9, child part_9_int1_10, origin xyz=0.04107454337811874967 -0.036577067764912860048 -0.004999999999999997502, axis 1 0 0, limit effort=1 velocity=20
- added joint part_9_part_7_4_rev1: type revolute, parent part_9_int1_10, child part_9_int2_10, axis 0 1 0, limit effort=1 velocity=20
- added joint part_9_part_7_4_rev2: type revolute, parent part_9_int2_10, child part_7_4, axis 0 0 1, limit effort=1 velocity=20
- added joint transmission_ankle2_2_part_7_5_rev0: type revolute, parent transmission_ankle2_2, child transmission_ankle2_2_int1_16, origin xyz=-0.059494699261975467208 0.01098320352752724105 -0.021999999999999964029, axis 1 0 0, limit effort=1 velocity=20
- added joint transmission_ankle2_2_part_7_5_rev1: type revolute, parent transmission_ankle2_2_int1_16, child transmission_ankle2_2_int2_16, axis 0 1 0, limit effort=1 velocity=20
- added joint transmission_ankle2_2_part_7_5_rev2: type revolute, parent transmission_ankle2_2_int2_16, child part_7_5, axis 0 0 1, limit effort=1 velocity=20
- added joint transmission_ankle2_part_7_rev0: type revolute, parent transmission_ankle2, child transmission_ankle2_int1_4, origin xyz=-0.059494699261975370064 0.010983203527527130028 -0.02200000000000001607, axis 1 0 0, limit effort=1 velocity=20
- added joint transmission_ankle2_part_7_rev1: type revolute, parent transmission_ankle2_int1_4, child transmission_ankle2_int2_4, axis 0 1 0, limit effort=1 velocity=20
- added joint transmission_ankle2_part_7_rev2: type revolute, parent transmission_ankle2_int2_4, child part_7, axis 0 0 1, limit effort=1 velocity=20
- added joint transmission_ankle_2_part_7_6_rev0: type revolute, parent transmission_ankle_2, child transmission_ankle_2_int1_17, origin xyz=-0.059494699261975467208 0.010983203527527130028 0.02200000000000001954, axis 1 0 0, limit effort=1 velocity=20
- added joint transmission_ankle_2_part_7_6_rev1: type revolute, parent transmission_ankle_2_int1_17, child transmission_ankle_2_int2_17, axis 0 1 0, limit effort=1 velocity=20
- added joint transmission_ankle_2_part_7_6_rev2: type revolute, parent transmission_ankle_2_int2_17, child part_7_6, axis 0 0 1, limit effort=1 velocity=20
- added joint transmission_ankle_part_7_2_rev0: type revolute, parent transmission_ankle, child transmission_ankle_int1_5, origin xyz=-0.059494699261975619864 0.010983203527527019006 0.022000000000000040357, axis 1 0 0, limit effort=1 velocity=20
- added joint transmission_ankle_part_7_2_rev1: type revolute, parent transmission_ankle_int1_5, child transmission_ankle_int2_5, axis 0 1 0, limit effort=1 velocity=20
- added joint transmission_ankle_part_7_2_rev2: type revolute, parent transmission_ankle_int2_5, child part_7_2, axis 0 0 1, limit effort=1 velocity=20
