Commit message: talos like modified

File: example_parallel_robots/robots/talos_like/robot.urdf (robot description, URDF)
Before this commit: robot onshape, 14 links, 13 joints
Links:
- added link ankle_int1_1, mass 0.0
- added link ankle_int2_1, mass 0.0
- added link moteur_int1_2, mass 0.0
- added link moteur_int2_2, mass 0.0
Joints:
- removed joint free_spherical_foot
- removed joint free_spherical_shin
- added joint ankle_rod_2_rev0: type revolute, parent ankle, child ankle_int1_1, origin xyz=-0.071653553385825324851 -0.020555800061897278042 -0.0096809999999999951648, axis 1 0 0, limit effort=1 velocity=20
- added joint ankle_rod_2_rev1: type revolute, parent ankle_int1_1, child ankle_int2_1, axis 0 1 0, limit effort=1 velocity=20
- added joint ankle_rod_2_rev2: type revolute, parent ankle_int2_1, child rod_2, axis 0 0 1, limit effort=1 velocity=20
- added joint moteur_rod_1_rev0: type revolute, parent moteur, child moteur_int1_2, origin xyz=-0.071653553385825130562 0.020555800061898721331 -0.0096810000000000784315, axis 1 0 0, limit effort=1 velocity=20
- added joint moteur_rod_1_rev1: type revolute, parent moteur_int1_2, child moteur_int2_2, axis 0 1 0, limit effort=1 velocity=20
- added joint moteur_rod_1_rev2: type revolute, parent moteur_int2_2, child rod_1, axis 0 0 1, limit effort=1 velocity=20
