Commit message: true_talos modified

File: example_parallel_robots/robots/true_talos_2_legs/talos_full_v2.urdf (robot description, URDF)
Before this commit: robot talos, 68 links, 67 joints
Links:
- removed link closedloop1_A
- removed link closedloop1_B
- removed link closedloop2_A
- removed link closedloop2_B
- added link leg_left_5_link_int1_1, mass 0.0
- added link leg_left_5_link_int2_1, mass 0.0
- added link leg_right_5_link_int1_1, mass 0.0
- added link leg_right_5_link_int2_1, mass 0.0
- added link link_closedloop1_A, mass 1e-9
- added link link_closedloop1_B, mass 1e-9
- added link link_closedloop2_A, mass 1e-9
- added link link_closedloop2_B, mass 1e-9
Joints:
- removed joint leg_left_foot_free_joint
- removed joint leg_right_foot_free_joint
- added joint leg_left_5_link_leg_left_foot_free_link_rev0: type revolute, parent leg_left_5_link, child leg_left_5_link_int1_1, origin xyz=-0.08 0.105 0.02, axis 1 0 0, limit effort=1 velocity=20
- added joint leg_left_5_link_leg_left_foot_free_link_rev1: type revolute, parent leg_left_5_link_int1_1, child leg_left_5_link_int2_1, axis 0 1 0, limit effort=1 velocity=20
- added joint leg_left_5_link_leg_left_foot_free_link_rev2: type revolute, parent leg_left_5_link_int2_1, child leg_left_foot_free_link, axis 0 0 1, limit effort=1 velocity=20
- added joint leg_right_5_link_leg_right_foot_free_link_rev0: type revolute, parent leg_right_5_link, child leg_right_5_link_int1_1, origin xyz=-0.08 -0.105 0.02, axis 1 0 0, limit effort=1 velocity=20
- added joint leg_right_5_link_leg_right_foot_free_link_rev1: type revolute, parent leg_right_5_link_int1_1, child leg_right_5_link_int2_1, axis 0 1 0, limit effort=1 velocity=20
- added joint leg_right_5_link_leg_right_foot_free_link_rev2: type revolute, parent leg_right_5_link_int2_1, child leg_right_foot_free_link, axis 0 0 1, limit effort=1 velocity=20
- joint closedloop1_A: child closedloop1_A -> link_closedloop1_A
- joint closedloop1_B: child closedloop1_B -> link_closedloop1_B
- joint closedloop2_A: child closedloop2_A -> link_closedloop2_A
- joint closedloop2_B: child closedloop2_B -> link_closedloop2_B
