Commit message: update wl16  to new standard

File: example_parallel_robots/robots/wl16_like/robot.urdf (robot description, URDF)
Before this commit: robot onshape, 31 links, 30 joints
Links:
- removed link bout_pied
- removed link centre_hanche
- removed link fermeture1_A
- removed link fermeture1_B
- removed link fermeture2_A
- removed link fermeture2_B
- removed link fermeture3_A
- removed link fermeture3_B
- removed link fermeture4_A
- removed link fermeture4_B
- removed link fermeture5_A
- removed link fermeture5_B
- removed link hips
- added link closedloop1_A, mass 1e-9
- added link closedloop1_B, mass 1e-9
- added link closedloop2_A, mass 1e-9
- added link closedloop2_B, mass 1e-9
- added link closedloop3_A, mass 1e-9
- added link closedloop3_B, mass 1e-9
- added link closedloop4_A, mass 1e-9
- added link closedloop4_B, mass 1e-9
- added link closedloop5_A, mass 1e-9
- added link closedloop5_B, mass 1e-9
- added link foot_part, mass 1.2962021735874538209; collision mesh filename=package:///foot_part.stl; visual mesh filename=package:///foot_part.stl
- added link hip, mass 1e-9
- added link hip_part, mass 43.978349764609049544; collision mesh filename=package:///hip_part.stl; visual mesh filename=package:///hip_part.stl
- link foot: mass 1.2962021735874540429 -> 1e-9; geometry 
Joints:
- removed joint bout_pied_frame
- removed joint centre_hanche_frame
- removed joint fermeture1_A_frame
- removed joint fermeture1_B_frame
- removed joint fermeture2_A_frame
- removed joint fermeture2_B_frame
- removed joint fermeture3_A_frame
- removed joint fermeture3_B_frame
- removed joint fermeture4_A_frame
- removed joint fermeture4_B_frame
- removed joint fermeture5_A_frame
- removed joint fermeture5_B_frame
- removed joint mot_1
- removed joint mot_2
- removed joint mot_3
- removed joint mot_4
- removed joint mot_5
- removed joint mot_6
- removed joint to_rotule_1
- removed joint to_rotule_10
- removed joint to_rotule_11
- removed joint to_rotule_12
- removed joint to_rotule_2
- removed joint to_rotule_3
- removed joint to_rotule_4
- removed joint to_rotule_5
- removed joint to_rotule_6
- removed joint to_rotule_7
- removed joint to_rotule_8
- removed joint to_rotule_9
- added joint closedloop1_A_frame: type fixed, parent axis_1, child closedloop1_A, origin xyz=0 0 -0.09900000000000008793 rpy=0 -0 0, axis 0 0 0
- added joint closedloop1_B_frame: type fixed, parent axis_2_3, child closedloop1_B, origin xyz=0 -5.5511151231257827021e-17 -0.098999000000000059174 rpy=3.141592653589793116 -0 0, axis 0 0 0
- added joint closedloop2_A_frame: type fixed, parent axis_1_2, child closedloop2_A, origin xyz=0 0 -0.09900000000000008793 rpy=0 -0 0, axis 0 0 0
- added joint closedloop2_B_frame: type fixed, parent axis_1_4, child closedloop2_B, origin xyz=0 -5.5511151231257827021e-17 -0.099000000000000198952 rpy=-3.141592653589793116 -0 0, axis 0 0 0
- added joint closedloop3_A_frame: type fixed, parent axis_1_3, child closedloop3_A, origin xyz=0 0 -0.09900000000000008793 rpy=0 -0 0, axis 0 0 0
- added joint closedloop3_B_frame: type fixed, parent axis_1_5, child closedloop3_B, origin xyz=0 -5.5511151231257827021e-17 -0.099000000000000198952 rpy=-3.141592653589793116 -0 0, axis 0 0 0
- added joint closedloop4_A_frame: type fixed, parent axis_2, child closedloop4_A, origin xyz=0 0 -0.098998999999999948152 rpy=0 -0 0, axis 0 0 0
- added joint closedloop4_B_frame: type fixed, parent axis_2_4, child closedloop4_B, origin xyz=0 2.7755575615628913511e-17 -0.098999000000000059174 rpy=3.141592653589793116 -0 0, axis 0 0 0
- added joint closedloop5_A_frame: type fixed, parent axis_2_2, child closedloop5_A, origin xyz=0 0 -0.098998999999999948152 rpy=0 -0 0, axis 0 0 0
- added joint closedloop5_B_frame: type fixed, parent axis_1_6, child closedloop5_B, origin xyz=0 -5.5511151231257827021e-17 -0.099000000000000143441 rpy=-3.141592653589793116 -0 0, axis 0 0 0
- added joint foot_frame: type fixed, parent foot_part, child foot, origin xyz=-0.01474114045414495755 -0.10478907385791688678 -0.058000000000000051514 rpy=0 -0 0, axis 0 0 0
- added joint hip_frame: type fixed, parent hip_part, child hip, origin xyz=2.4027501270446963816e-19 -0.22000000000000002887 0.0024999999999999996184 rpy=0 -0 0, axis 0 0 0
- added joint motor_1: type prismatic, parent motor_2, child axis_1_2, origin xyz=0 0 -0.48779999999999995586 rpy=0 -0 0, axis 0 0 1, limit effort=1 velocity=20
- added joint motor_2: type prismatic, parent motor_3, child axis_1_3, origin xyz=0 0 -0.48779999999999995586 rpy=0 -0 0, axis 0 0 1, limit effort=1 velocity=20
- added joint motor_3: type prismatic, parent motor_4, child axis_2, origin xyz=0 0 -0.49860000000000009868 rpy=0 -0 0, axis 0 0 1, limit effort=1 velocity=20
- added joint motor_4: type prismatic, parent motor, child axis_1, origin xyz=0 0 -0.48779999999999995586 rpy=0 -0 0, axis 0 0 1, limit effort=1 velocity=20
- added joint motor_5: type prismatic, parent motor_5, child axis_2_2, origin xyz=0 0 -0.49860000000000009868 rpy=0 -0 0, axis 0 0 1, limit effort=1 velocity=20
- added joint motor_6: type prismatic, parent motor_6, child part_4, origin xyz=0 0 -0.35820000000000012941 rpy=0 -0 0, axis 0 0 1, limit effort=1 velocity=20
- added joint spherical_1: type revolute, parent hip_part, child motor, origin xyz=-0.27500000000000007772 -0.22647302994931878262 -0.066000000000000003109 rpy=0 -0 0, axis 0 0 1, limit effort=1 velocity=20
- added joint spherical_10: type revolute, parent foot_part, child axis_2_4, origin xyz=0.090750000000000025091 -0.15718361078687545507 0 rpy=2.6179938779914944114 -0 0, axis 0 0 1, limit effort=1 velocity=20
- added joint spherical_11: type revolute, parent foot_part, child axis_1_6, origin xyz=0 0 0 rpy=-2.6179938779914944114 -0 0, axis 0 0 1, limit effort=1 velocity=20
- added joint spherical_12: type revolute, parent part_4, child foot_part, origin xyz=0 0 -0.19800000000000006484 rpy=0 -0 0, axis 0 0 1, limit effort=1 velocity=20
- added joint spherical_2: type revolute, parent hip_part, child motor_2, origin xyz=-0.09899999999999996303 -0.53131397208144126587 -0.066000000000000003109 rpy=0 -0 0, axis 0 0 1, limit effort=1 velocity=20
- added joint spherical_3: type revolute, parent hip_part, child motor_3, origin xyz=0.099000000000000074052 -0.53131397208144148792 -0.066000000000000003109 rpy=0 -0 0, axis 0 0 1, limit effort=1 velocity=20
- added joint spherical_4: type revolute, parent hip_part, child motor_4, origin xyz=0.2750000000000000222 -0.22647302994931894915 -0.066000000000000003109 rpy=0 -0 0, axis 0 0 1, limit effort=1 velocity=20
- added joint spherical_5: type revolute, parent hip_part, child motor_5, origin xyz=-0.1760000000000000453 -0.054999999999999993339 -0.066000000000000003109 rpy=0 -0 0, axis 0 0 1, limit effort=1 velocity=20
- added joint spherical_6: type revolute, parent hip_part, child motor_6, origin xyz=0.17600000000000012856 -0.054999999999999993339 -0.066000000000000003109 rpy=0 -0 0, axis 0 0 1, limit effort=1 velocity=20
- added joint spherical_7: type revolute, parent foot_part, child axis_1_4, origin xyz=-0.090749999999999997335 -0.15718361078687548282 -1.1102230246251565404e-16 rpy=-2.6179938779914944114 -0 0, axis 0 0 1, limit effort=1 velocity=20
- added joint spherical_8: type revolute, parent foot_part, child axis_2_3, origin xyz=-0.090749999999999997335 -0.15718361078687553833 0 rpy=2.6179938779914944114 -0 0, axis 0 0 1, limit effort=1 velocity=20
- added joint spherical_9: type revolute, parent foot_part, child axis_1_5, origin xyz=0.090750000000000025091 -0.15718361078687545507 -1.1102230246251565404e-16 rpy=-2.6179938779914944114 -0 0, axis 0 0 1, limit effort=1 velocity=20

Commit message: wl16 modified

File: example_parallel_robots/robots/wl16_like/robot.urdf (robot description, URDF)
Before this commit: robot onshape, 31 links, 30 joints
Links:
- added link foot_part_int1_10, mass 0.0
- added link foot_part_int1_6, mass 0.0
- added link foot_part_int1_7, mass 0.0
- added link foot_part_int1_8, mass 0.0
- added link foot_part_int1_9, mass 0.0
- added link foot_part_int2_10, mass 0.0
- added link foot_part_int2_6, mass 0.0
- added link foot_part_int2_7, mass 0.0
- added link foot_part_int2_8, mass 0.0
- added link foot_part_int2_9, mass 0.0
- added link hip_part_int1_1, mass 0.0
- added link hip_part_int1_12, mass 0.0
- added link hip_part_int1_2, mass 0.0
- added link hip_part_int1_3, mass 0.0
- added link hip_part_int1_4, mass 0.0
- added link hip_part_int1_5, mass 0.0
- added link hip_part_int2_1, mass 0.0
- added link hip_part_int2_12, mass 0.0
- added link hip_part_int2_2, mass 0.0
- added link hip_part_int2_3, mass 0.0
- added link hip_part_int2_4, mass 0.0
- added link hip_part_int2_5, mass 0.0
- added link part_4_int1_11, mass 0.0
- added link part_4_int2_11, mass 0.0
Joints:
- removed joint spherical_1
- removed joint spherical_10
- removed joint spherical_11
- removed joint spherical_12
- removed joint spherical_2
- removed joint spherical_3
- removed joint spherical_4
- removed joint spherical_5
- removed joint spherical_6
- removed joint spherical_7
- removed joint spherical_8
- removed joint spherical_9
- added joint foot_part_axis_1_4_rev0: type revolute, parent foot_part, child foot_part_int1_6, origin xyz=-0.090749999999999997335 -0.15718361078687548282 -1.1102230246251565404e-16, axis 1 0 0, limit effort=1 velocity=20
- added joint foot_part_axis_1_4_rev1: type revolute, parent foot_part_int1_6, child foot_part_int2_6, axis 0 1 0, limit effort=1 velocity=20
- added joint foot_part_axis_1_4_rev2: type revolute, parent foot_part_int2_6, child axis_1_4, axis 0 0 1, limit effort=1 velocity=20
- added joint foot_part_axis_1_5_rev0: type revolute, parent foot_part, child foot_part_int1_8, origin xyz=0.090750000000000025091 -0.15718361078687545507 -1.1102230246251565404e-16, axis 1 0 0, limit effort=1 velocity=20
- added joint foot_part_axis_1_5_rev1: type revolute, parent foot_part_int1_8, child foot_part_int2_8, axis 0 1 0, limit effort=1 velocity=20
- added joint foot_part_axis_1_5_rev2: type revolute, parent foot_part_int2_8, child axis_1_5, axis 0 0 1, limit effort=1 velocity=20
- added joint foot_part_axis_1_6_rev0: type revolute, parent foot_part, child foot_part_int1_10, origin xyz=0 0 0, axis 1 0 0, limit effort=1 velocity=20
- added joint foot_part_axis_1_6_rev1: type revolute, parent foot_part_int1_10, child foot_part_int2_10, axis 0 1 0, limit effort=1 velocity=20
- added joint foot_part_axis_1_6_rev2: type revolute, parent foot_part_int2_10, child axis_1_6, axis 0 0 1, limit effort=1 velocity=20
- added joint foot_part_axis_2_3_rev0: type revolute, parent foot_part, child foot_part_int1_7, origin xyz=-0.090749999999999997335 -0.15718361078687553833 0, axis 1 0 0, limit effort=1 velocity=20
- added joint foot_part_axis_2_3_rev1: type revolute, parent foot_part_int1_7, child foot_part_int2_7, axis 0 1 0, limit effort=1 velocity=20
- added joint foot_part_axis_2_3_rev2: type revolute, parent foot_part_int2_7, child axis_2_3, axis 0 0 1, limit effort=1 velocity=20
- added joint foot_part_axis_2_4_rev0: type revolute, parent foot_part, child foot_part_int1_9, origin xyz=0.090750000000000025091 -0.15718361078687545507 0, axis 1 0 0, limit effort=1 velocity=20
- added joint foot_part_axis_2_4_rev1: type revolute, parent foot_part_int1_9, child foot_part_int2_9, axis 0 1 0, limit effort=1 velocity=20
- added joint foot_part_axis_2_4_rev2: type revolute, parent foot_part_int2_9, child axis_2_4, axis 0 0 1, limit effort=1 velocity=20
- added joint hip_part_motor_part_2_rev0: type revolute, parent hip_part, child hip_part_int1_2, origin xyz=-0.09899999999999996303 -0.53131397208144126587 -0.066000000000000003109, axis 1 0 0, limit effort=1 velocity=20
- added joint hip_part_motor_part_2_rev1: type revolute, parent hip_part_int1_2, child hip_part_int2_2, axis 0 1 0, limit effort=1 velocity=20
- added joint hip_part_motor_part_2_rev2: type revolute, parent hip_part_int2_2, child motor_part_2, axis 0 0 1, limit effort=1 velocity=20
- added joint hip_part_motor_part_3_rev0: type revolute, parent hip_part, child hip_part_int1_3, origin xyz=0.099000000000000074052 -0.53131397208144148792 -0.066000000000000003109, axis 1 0 0, limit effort=1 velocity=20
- added joint hip_part_motor_part_3_rev1: type revolute, parent hip_part_int1_3, child hip_part_int2_3, axis 0 1 0, limit effort=1 velocity=20
- added joint hip_part_motor_part_3_rev2: type revolute, parent hip_part_int2_3, child motor_part_3, axis 0 0 1, limit effort=1 velocity=20
- added joint hip_part_motor_part_4_rev0: type revolute, parent hip_part, child hip_part_int1_4, origin xyz=0.2750000000000000222 -0.22647302994931894915 -0.066000000000000003109, axis 1 0 0, limit effort=1 velocity=20
- added joint hip_part_motor_part_4_rev1: type revolute, parent hip_part_int1_4, child hip_part_int2_4, axis 0 1 0, limit effort=1 velocity=20
- added joint hip_part_motor_part_4_rev2: type revolute, parent hip_part_int2_4, child motor_part_4, axis 0 0 1, limit effort=1 velocity=20
- added joint hip_part_motor_part_5_rev0: type revolute, parent hip_part, child hip_part_int1_5, origin xyz=-0.1760000000000000453 -0.054999999999999993339 -0.066000000000000003109, axis 1 0 0, limit effort=1 velocity=20
- added joint hip_part_motor_part_5_rev1: type revolute, parent hip_part_int1_5, child hip_part_int2_5, axis 0 1 0, limit effort=1 velocity=20
- added joint hip_part_motor_part_5_rev2: type revolute, parent hip_part_int2_5, child motor_part_5, axis 0 0 1, limit effort=1 velocity=20
- added joint hip_part_motor_part_6_rev0: type revolute, parent hip_part, child hip_part_int1_12, origin xyz=0.17600000000000012856 -0.054999999999999993339 -0.066000000000000003109, axis 1 0 0, limit effort=1 velocity=20
- added joint hip_part_motor_part_6_rev1: type revolute, parent hip_part_int1_12, child hip_part_int2_12, axis 0 1 0, limit effort=1 velocity=20
- added joint hip_part_motor_part_6_rev2: type revolute, parent hip_part_int2_12, child motor_part_6, axis 0 0 1, limit effort=1 velocity=20
- added joint hip_part_motor_part_rev0: type revolute, parent hip_part, child hip_part_int1_1, origin xyz=-0.27500000000000007772 -0.22647302994931878262 -0.066000000000000003109, axis 1 0 0, limit effort=1 velocity=20
- added joint hip_part_motor_part_rev1: type revolute, parent hip_part_int1_1, child hip_part_int2_1, axis 0 1 0, limit effort=1 velocity=20
- added joint hip_part_motor_part_rev2: type revolute, parent hip_part_int2_1, child motor_part, axis 0 0 1, limit effort=1 velocity=20
- added joint part_4_foot_part_rev0: type revolute, parent part_4, child part_4_int1_11, origin xyz=0 0 -0.19800000000000006484, axis 1 0 0, limit effort=1 velocity=20
- added joint part_4_foot_part_rev1: type revolute, parent part_4_int1_11, child part_4_int2_11, axis 0 1 0, limit effort=1 velocity=20
- added joint part_4_foot_part_rev2: type revolute, parent part_4_int2_11, child foot_part, axis 0 0 1, limit effort=1 velocity=20
