Commit message: Update Digit

File: robots/digit_like_2legs/robot.urdf (robot description, URDF)
Before this commit: robot onshape, 24 links, 23 joints
Links:
- added link bout_pied_gauche, mass 1e-9
- added link fermeture4_A, mass 1e-9
- added link fermeture4_B, mass 1e-9
- added link fermeture5_A, mass 1e-9
- added link fermeture5_B, mass 1e-9
- added link fermeture6_A, mass 1e-9
- added link fermeture6_B, mass 1e-9
- added link foot_2, mass 0.33095167420253668311; collision mesh filename=package:///foot.stl; visual mesh filename=package:///foot.stl
- added link foot_roll_2, mass 0.0027067106871796996204; collision mesh filename=package:///foot_roll.stl; visual mesh filename=package:///foot_roll.stl
- added link hip_x_2, mass 1.4197410037164888141; collision mesh filename=package:///hip_x.stl; visual mesh filename=package:///hip_x.stl
- added link hip_y_2, mass 1.2895238899898622265; collision mesh filename=package:///hip_y.stl; visual mesh filename=package:///hip_y.stl
- added link hip_z_2, mass 3.8932756153047387571; collision mesh filename=package:///hip_z.stl; visual mesh filename=package:///hip_z.stl
- added link molet_3, mass 0.0045332434126214744829; collision mesh filename=package:///molet.stl; visual mesh filename=package:///molet.stl
- added link molet_4, mass 0.0045332434126214744829; collision mesh filename=package:///molet.stl; visual mesh filename=package:///molet.stl
- added link shin_2, mass 0.55578140933316366734; collision mesh filename=package:///shin.stl; visual mesh filename=package:///shin.stl
- added link tarsus_2, mass 0.7428461942208621771; collision mesh filename=package:///actuator_molet.stl; collision mesh filename=package:///tarsus.stl
- added link toe_a_1/2_2, mass 0.015704036277131967758; collision mesh filename=package:///toe_a_1_2.stl; visual mesh filename=package:///toe_a_1_2.stl
- added link toe_a_2/2_2, mass 0.015704036277131950411; collision mesh filename=package:///toe_a_2_2.stl; visual mesh filename=package:///toe_a_2_2.stl
- added link toe_b_1/2_3, mass 0.0060293446207695467268; collision mesh filename=package:///toe_b_1_2.stl; visual mesh filename=package:///toe_b_1_2.stl
- added link toe_b_1/2_4, mass 0.0060293446207695467268; collision mesh filename=package:///toe_b_1_2.stl; visual mesh filename=package:///toe_b_1_2.stl
- added link toe_b_2/2_3, mass 0.0060293446207695345837; collision mesh filename=package:///toe_b_2_2.stl; visual mesh filename=package:///toe_b_2_2.stl
- added link toe_b_2/2_4, mass 0.0060293446207695345837; collision mesh filename=package:///toe_b_2_2.stl; visual mesh filename=package:///toe_b_2_2.stl
- link foot: mass 0.3309516742025366276 -> 0.33095167420253668311
- link foot_roll: mass 0.0027067106871796991867 -> 0.0027067106871796996204
- link hip_x: mass 1.4197410037164885921 -> 1.4197410037164888141
- link shin: mass 0.5557814093331634453 -> 0.55578140933316366734
- link tarsus: mass 0.74284619422086206608 -> 0.7428461942208621771
Joints:
- added joint bout_pied_gauche_frame: type fixed, parent foot_2, child bout_pied_gauche, origin xyz=-0.055897619600577430621 0 0.0037840702321054742185 rpy=-2.0029632011476419211e-16 -1.0420837364882549192 -3.141592653589793116, axis 0 0 0
- added joint fermeture4_A_frame: type fixed, parent toe_b_1/2_3, child fermeture4_A, origin xyz=0 -1.1102230246251565404e-16 -0.11995000000000000107 rpy=-3.1415926535897926719 1.4557857793770605109e-15 1.570796326794896558, axis 0 0 0
- added joint fermeture4_B_frame: type fixed, parent toe_b_2/2_4, child fermeture4_B, origin xyz=0 -2.7755575615628913511e-17 -0.11994999999999983453 rpy=2.5132107670464821188e-16 -1.5516628120086465861e-16 -7.8371506725709791247e-17, axis 0 0 0
- added joint fermeture5_A_frame: type fixed, parent toe_b_2/2_3, child fermeture5_A, origin xyz=0 1.1102230246251565404e-16 -0.11994999999999977902 rpy=-3.1415926535897926719 1.4557857793770605109e-15 1.570796326794896558, axis 0 0 0
- added joint fermeture5_B_frame: type fixed, parent toe_b_1/2_4, child fermeture5_B, origin xyz=-3.3306690738754696213e-16 0 -0.1199499999999999178 rpy=1.3570894085680469023e-16 1.1131720658713263778e-15 -3.141592653589793116, axis 0 0 0
- added joint fermeture6_A_frame: type fixed, parent toe_a_1/2_2, child fermeture6_A, origin xyz=6.5919492087118669588e-17 0 -0.19995000000000007212 rpy=-3.141592653589793116 -7.0048445437832687964e-17 -2.6752620058038898353e-33, axis 0 0 0
- added joint fermeture6_B_frame: type fixed, parent toe_a_2/2_2, child fermeture6_B, origin xyz=6.9388939039072283776e-18 -2.0816681711721685133e-17 -0.19994999999999985008 rpy=-6.1223473960463149353e-17 2.4651903288156618919e-32 9.6553912330110834249e-33, axis 0 0 0
- added joint libre_genoux_left: type revolute, parent shin_2, child tarsus_2, origin xyz=0.39567486363081372236 -0.053875166733171747646 -0.024999999999999994449 rpy=0 -0 1.570796326794896558, axis 0 0 1, limit effort=1 velocity=20
- added joint libre_pied1_left: type revolute, parent tarsus_2, child foot_roll_2, origin xyz=-0.325998400000000077 -0.038657982377658717255 -5.5511151231257827021e-17 rpy=5.5511151231257814695e-17 2.7597873481449337343e-16 -3.1415926535897624738, axis 0 0 1, limit effort=1 velocity=20
- added joint libre_pied2_left: type revolute, parent foot_roll_2, child foot_2, origin xyz=1.1102230246251565404e-16 0.0090000000000000079936 -8.3266726846886740532e-17 rpy=-1.570796326794896558 7.3354943207976340417e-16 -3.141592653589793116, axis 0 0 1, limit effort=1 velocity=20
- added joint mot_genoux_left: type revolute, parent hip_z_2, child shin_2, origin xyz=0.1199999999999999678 0 1.6930901125533637241e-15 rpy=3.141592653589793116 -0 -0.55703373375772102793, axis 0 0 1, limit effort=1 velocity=20
- added joint mot_hanche_left_x: type revolute, parent torso, child hip_y_2, origin xyz=-0.02999999999999999889 0.072800000000000031353 0.059867854479678822566 rpy=-0 1.570796326794896558 0, axis 0 0 1, limit effort=1 velocity=20
- added joint mot_hanche_left_y: type revolute, parent hip_x_2, child hip_z_2, origin xyz=-0.029117226656781597383 0 -0.047379470518249228173 rpy=-1.570796326794896558 1.2655169802117200994 -1.570796326794896558, axis 0 0 1, limit effort=1 velocity=20
- added joint mot_hanche_left_z: type revolute, parent hip_y_2, child hip_x_2, origin xyz=0.050000000000000016653 0 -0.035199999999999981304 rpy=1.570796326794896558 -0 -1.570796326794896558, axis 0 0 1, limit effort=1 velocity=20
- added joint mot_servo1_left: type revolute, parent tarsus_2, child molet_3, origin xyz=-0.088800000000002418665 -0.026113982377657718459 0.02999999999999999889 rpy=3.141592653589793116 -0 -1.1936089721976891145e-17, axis 0 0 1, limit effort=1 velocity=20
- added joint mot_servo2_left: type revolute, parent tarsus_2, child molet_4, origin xyz=-0.08880000000000000393 -0.026113982377658606637 -0.029999999999999978073 rpy=-2.4214412524677942898e-16 -8.9555256306153669199e-17 3.141592653589793116, axis 0 0 1, limit effort=1 velocity=20
- added joint to_rotule_libre_hanche2_left: type revolute, parent hip_x_2, child toe_a_2/2_2, origin xyz=0.030568773343218405558 0 -0.054400000000000003908 rpy=-1.57079632679489678 1.570796326794896558 0, axis 0 0 1, limit effort=1 velocity=20
- added joint to_rotule_libre_hanche_left: type revolute, parent tarsus_2, child toe_a_1/2_2, origin xyz=0.1141899349863718105 0.03620674973129278662 7.3552275381416620803e-16 rpy=-1.570796326794896558 -6.032224767520871884e-18 3.141592653589793116, axis 0 0 1, limit effort=1 velocity=20
- added joint to_rotule_pied_gauche_1: type revolute, parent foot_2, child toe_b_1/2_3, origin xyz=-0.0091288304490432237159 -0.014276000000000010903 -0.034653600000000173154 rpy=1.5707963267948970021 -1.0103389770218152502e-16 -1.5707963267948961139, axis 0 0 1, limit effort=1 velocity=20
- added joint to_rotule_pied_gauche_2: type revolute, parent foot_2, child toe_b_2/2_3, origin xyz=-0.0091288304490432237159 0.014275999999999927637 -0.034653600000000284176 rpy=1.5707963267948970021 -1.0103389770218157432e-16 -1.5707963267948961139, axis 0 0 1, limit effort=1 velocity=20
- added joint to_rotule_servo_gauche_1: type revolute, parent molet_3, child toe_b_2/2_4, origin xyz=-5.5511151231257827021e-17 0.057000000000000050626 0.0025000000000000022204 rpy=-1.57079632679489678 -6.1989581036318994383e-14 -1.570796326794896558, axis 0 0 1, limit effort=1 velocity=20
- added joint to_rotule_servo_gauche_2: type revolute, parent molet_4, child toe_b_1/2_4, origin xyz=2.2204460492503130808e-16 0.057000000000000494715 0.0025000000000004185541 rpy=-1.570796326794896558 -1.866329740155221443e-16 1.5707963267948970021, axis 0 0 1, limit effort=1 velocity=20
- joint bout_pied_frame: origin xyz=-0.05589761960057737511 0 0.014375929767894424227 rpy=3.141592653589793116 1.0420837364882535869 3.141592653589793116 -> xyz=-0.055897619600577819199 2.7755575615628913511e-16 0.014375929767894812805 rpy=3.141592653589793116 1.0420837364882524767 3.141592653589793116
- joint centre_hanche_frame: origin xyz=-2.4027501270446886779e-19 1.626303258728255688e-19 0.0024999999999999996184 rpy=2.8421709430404007435e-14 3.0814879110196404233e-31 3.141592653589793116 -> xyz=2.4027501270446886779e-19 -1.626303258728255688e-19 0.0024999999999999996184 rpy=2.8421709430404007435e-14 3.0814879110196404233e-31 0
- joint fermeture1_A_frame: origin xyz=9.0205620750793968909e-17 0 -0.19994999999999990559 rpy=-3.7112781480334425034e-16 8.2442115866850430893e-18 1.0097912624895015577e-27 -> xyz=8.3266726846886740532e-17 -6.9388939039072283776e-18 -0.19994999999999990559 rpy=-3.7112781480334543363e-16 -7.6145285777054681417e-31 -1.2325951642497940378e-32
- joint fermeture1_B_frame: origin xyz=0 1.3877787807814456755e-17 -0.1999500000000002109 rpy=3.141592653589793116 -9.7378114602005348959e-18 3.141592653589793116 -> xyz=-4.1633363423443370266e-17 -8.3266726846886740532e-17 -0.19995000000000001661 rpy=3.141592653589793116 -4.3598202726084071025e-18 3.141592653589793116
- joint fermeture2_A_frame: origin xyz=0 0 -0.11994999999999994555 rpy=6.1280808278935614477e-17 3.5225097907092313716e-17 -1.5770158750347860435e-21 -> xyz=0 0 -0.11994999999999994555 rpy=1.7235773343990823765e-16 -3.2166375860020982159e-18 -9.2330428060222376469e-17
- joint fermeture2_B_frame: origin xyz=-4.1633363423443370266e-17 0 -0.11995000000000000107 rpy=3.141592653589793116 1.9682319780529215571e-17 1.570796326794896558 -> xyz=-1.0408340855860842566e-16 1.6653345369377348106e-16 -0.11995000000000022311 rpy=3.141592653589793116 -3.4014104205904975495e-17 1.570796326794896558
- joint fermeture3_A_frame: origin xyz=0 0 -0.11994999999999983453 rpy=1.7991914157564876276e-16 3.9760952339837050232e-18 -2.1710651278743624535e-18 -> xyz=-2.7755575615628913511e-17 0 -0.11994999999999972351 rpy=2.4425794194715678642e-16 -1.2567090974513322893e-17 9.4104185549181988163e-18
- joint fermeture3_B_frame: origin xyz=0 -1.1102230246251565404e-16 -0.11995000000000022311 rpy=3.141592653589793116 5.765418484336821195e-17 1.570796326794896558 -> xyz=-4.1633363423443370266e-17 5.5511151231257827021e-17 -0.11995000000000011209 rpy=-3.141592653589793116 6.050439432614581419e-18 1.570796326794896558
- joint libre_genoux: origin xyz=0.39567486363081372236 0.053875166733171692135 -0.025000000000000015266 rpy=3.141592653589793116 1.8170376977777737139e-18 -1.6910768536229012771 -> xyz=0.39567486363081366685 0.053875166733171879485 -0.025000000000000008327 rpy=3.141592653589793116 1.7052319612022700791e-18 -1.6910768536229012771
- joint libre_pied1: origin xyz=-0.32599840000000018803 -0.038657982377658606232 -0.014000000000000074885 rpy=3.141592653589793116 -2.7008077392723998759e-16 -2.8764747500822966941 -> xyz=-0.32599840000000002149 -0.038657982377658606232 -0.01400000000000004019 rpy=-3.1415926535897926719 3.4117039112211768089e-17 -2.8764747500822966941
- joint libre_pied_2: origin xyz=0 0.0090000000000000079936 -0.013999999999999998557 rpy=-1.570796326794896558 3.0369740063504090599e-05 -3.1415926535897926719 -> xyz=1.1102230246251565404e-16 0.0089999999999998969713 -0.013999999999999956923 rpy=-1.5707963267948961139 0.00018013600906293872469 -3.141592653589793116
- joint mot_genoux: origin xyz=-0.11999999999999998168 -1.3877787807814456755e-17 0 rpy=3.141592653589793116 1.6140181441454188796e-16 -2.6828651102102365478 -> xyz=-0.11999999999999998168 0 0 rpy=3.141592653589793116 1.6137487424794804186e-16 -2.6828651102102365478
- joint mot_hanche_x: origin xyz=0.02999999999999999889 0.072799999999999975842 0.059867854479678822566 rpy=-3.141592653589793116 1.570796326794896558 0 -> xyz=-0.02999999999999999889 -0.072799999999999975842 0.059867854479678822566 rpy=1.0689153541114032999e-25 1.570796326794896558 0
- joint mot_hanche_y: origin xyz=-0.026000000000000002276 0 -0.054400000000000010847 rpy=-1.570796326794896558 -1.1931918349460191031 -1.5707963267948970021 -> xyz=-0.025999999999999995337 -2.7755575615628913511e-17 -0.054400000000000010847 rpy=-1.570796326794896336 -1.1931918349460142181 -1.570796326794896558
- joint mot_hanche_z: origin xyz=0.052665792973456596049 0 -0.035200000000000009059 rpy=1.570796326794896558 9.2157185462955552578e-18 -1.570796326794896558 -> xyz=0.05266579297345658911 1.3877787807814456755e-17 -0.035199999999999995182 rpy=-1.57079632679489678 1.1102230246014436281e-16 1.570796326794896558
- joint mot_servo1: origin xyz=-0.088800000000000045564 -0.026113982377658551126 0.029999999999999985012 rpy=-3.141592653589793116 5.2844134501331837538e-18 0.085487820950950324517 -> xyz=-0.088800000000000073319 -0.026113982377658606637 0.02999999999999999889 rpy=-3.141592653589793116 3.3674348063693462321e-18 0.085487820950950324517
- joint mot_servo2: origin xyz=-0.088800000000000045564 -0.026113982377658551126 -0.030000000000000019706 rpy=-7.2028754011234369278e-17 -2.0682911281837146378e-18 -3.0334710307071497404 -> xyz=-0.088800000000000017808 -0.02611398237765871766 -0.02999999999999999889 rpy=-7.5875284351392275809e-17 -8.5523186607038729703e-18 -3.0649221372054666901
- joint to_rotule_libre_genoux: origin xyz=0.11418993498637036721 0.036206749731294507466 0 rpy=-1.57079632679489678 -1.2731099122301607895 -3.1415926535897926719 -> xyz=0.1141899349863703117 0.036206749731294562977 0 rpy=-1.57079632679489678 -1.2731099122301605675 -3.1415926535897926719
- joint to_rotule_libre_hanche: origin xyz=0.033685999999999993726 0 -0.054399999999999996969 rpy=1.57079632679489678 -1.570796326794896336 0 -> xyz=0.033686000000000014543 -4.1633363423443370266e-17 -0.054400000000000017786 rpy=1.5707963267948970021 -1.5707963267948892305 0
- joint to_rotule_libre_molet1: origin xyz=0 0.056999999999999995115 0.0025000000000000022204 rpy=1.5707963267948970021 -1.438335209354334232 -1.5707963267948930053 -> xyz=5.5511151231257827021e-17 0.056999999999999939604 0.0024999999999999883427 rpy=1.5707963267948970021 -1.438335209354334232 -1.5707963267948930053
- joint to_rotule_libre_molet2: origin xyz=0 0.057000000000000050626 0.0025000000000000022204 rpy=1.570796326794896558 -0.00025864959668214364567 1.57079632679489678 -> xyz=5.5511151231257827021e-17 0.057000000000000050626 0.002499999999999967526 rpy=-1.5707963267948958919 -1.0579268199450198029 -1.5707963267948983344
- joint to_rotule_libre_pied1: origin xyz=-0.0091288304490430016713 -0.014275999999999990087 0.052813599999999960577 rpy=1.57079632679489678 -8.3440173426621114272e-05 -1.570796326794896558 -> xyz=-0.0091288304490431126936 -0.014275999999999927637 0.052813599999999960577 rpy=1.570796326794896558 -8.3440173396949238421e-05 -1.5707963267948978903
- joint to_rotule_libre_pied2: origin xyz=-0.0091288304490430016713 0.014276000000000010903 0.052813599999999960577 rpy=1.5707963267948970021 -8.3440173426648856295e-05 -1.570796326794896558 -> xyz=-0.009128830449042890649 0.014276000000000017842 0.052813599999999794044 rpy=1.570796326794896558 -8.3440173395629059646e-05 -1.570796326794896558
