Commit message: Update Digit Model

File: robots/digit_like_2legs/robot.urdf (robot description, URDF)
Before this commit: robot onshape, 70 links, 69 joints
Links:
- removed link crank_2_int1_4
- removed link crank_2_int2_4
- removed link crank_3_int1_9
- removed link crank_3_int2_9
- removed link crank_4_int1_10
- removed link crank_4_int2_10
- removed link crank_int1_3
- removed link crank_int2_3
- removed link foot_part_2_int1_7
- removed link foot_part_2_int1_8
- removed link foot_part_2_int2_7
- removed link foot_part_2_int2_8
- removed link foot_part_int1_1
- removed link foot_part_int1_2
- removed link foot_part_int2_1
- removed link foot_part_int2_2
- removed link hip_x_2_int1_12
- removed link hip_x_2_int2_12
- removed link hip_x_int1_6
- removed link hip_x_int2_6
- removed link tarsus_2_int1_11
- removed link tarsus_2_int2_11
- removed link tarsus_int1_5
- removed link tarsus_int2_5
- link hip_x: mass 1.4197410037164888141 -> 1.4197410037164885921
- link hip_x_2: mass 1.4197410037164888141 -> 1.4197410037164885921
- link hip_z: mass 3.893275615304738313 -> 3.8932756153047387571
- link hip_z_2: mass 3.893275615304738313 -> 3.8932756153047387571
- link shin: mass 0.55578140933316355632 -> 0.5557814093331634453
- link shin_2: mass 0.55578140933316355632 -> 0.5557814093331634453
- link tarsus: mass 0.74284619422086228813 -> 0.7428461942208621771
- link tarsus_2: mass 0.74284619422086228813 -> 0.7428461942208621771
Joints:
- removed joint crank_2_toe_b_2/2_2_rev0
- removed joint crank_2_toe_b_2/2_2_rev1
- removed joint crank_2_toe_b_2/2_2_rev2
- removed joint crank_3_toe_b_2/2_4_rev0
- removed joint crank_3_toe_b_2/2_4_rev1
- removed joint crank_3_toe_b_2/2_4_rev2
- removed joint crank_4_toe_b_1/2_4_rev0
- removed joint crank_4_toe_b_1/2_4_rev1
- removed joint crank_4_toe_b_1/2_4_rev2
- removed joint crank_toe_b_2/2_rev0
- removed joint crank_toe_b_2/2_rev1
- removed joint crank_toe_b_2/2_rev2
- removed joint foot_part_2_toe_b_1/2_3_rev0
- removed joint foot_part_2_toe_b_1/2_3_rev1
- removed joint foot_part_2_toe_b_1/2_3_rev2
- removed joint foot_part_2_toe_b_2/2_3_rev0
- removed joint foot_part_2_toe_b_2/2_3_rev1
- removed joint foot_part_2_toe_b_2/2_3_rev2
- removed joint foot_part_toe_b_1/2_2_rev0
- removed joint foot_part_toe_b_1/2_2_rev1
- removed joint foot_part_toe_b_1/2_2_rev2
- removed joint foot_part_toe_b_1/2_rev0
- removed joint foot_part_toe_b_1/2_rev1
- removed joint foot_part_toe_b_1/2_rev2
- removed joint hip_x_2_toe_a_2/2_2_rev0
- removed joint hip_x_2_toe_a_2/2_2_rev1
- removed joint hip_x_2_toe_a_2/2_2_rev2
- removed joint hip_x_toe_a_2/2_rev0
- removed joint hip_x_toe_a_2/2_rev1
- removed joint hip_x_toe_a_2/2_rev2
- removed joint tarsus_2_toe_a_1/2_2_rev0
- removed joint tarsus_2_toe_a_1/2_2_rev1
- removed joint tarsus_2_toe_a_1/2_2_rev2
- removed joint tarsus_toe_a_1/2_rev0
- removed joint tarsus_toe_a_1/2_rev1
- removed joint tarsus_toe_a_1/2_rev2
- added joint spherical_free_foot1: type revolute, parent foot_part, child toe_b_1/2, origin xyz=-0.0091288304490427796267 -0.014275999999999955392 0.052813600000000016088 rpy=1.570796326794896558 0.00015724417883685367909 -1.5707963267948981123, axis 0 0 1, limit effort=1 velocity=20
- added joint spherical_free_foot1_left: type revolute, parent foot_part_2, child toe_b_1/2_3, origin xyz=-0.0091288304490432237159 -0.014276000000000010903 -0.034653600000000173154 rpy=1.5707963267948970021 -1.0103389770218152502e-16 -1.5707963267948961139, axis 0 0 1, limit effort=1 velocity=20
- added joint spherical_free_foot2: type revolute, parent foot_part, child toe_b_1/2_2, origin xyz=-0.0091288304490430016713 0.014276000000000024781 0.052813600000000016088 rpy=1.57079632679489678 0.00015724417883817773389 -1.570796326794896558, axis 0 0 1, limit effort=1 velocity=20
- added joint spherical_free_foot2_left: type revolute, parent foot_part_2, child toe_b_2/2_3, origin xyz=-0.0091288304490432237159 0.014275999999999927637 -0.034653600000000284176 rpy=1.5707963267948970021 -1.0103389770218157432e-16 -1.5707963267948961139, axis 0 0 1, limit effort=1 velocity=20
- added joint spherical_free_hip: type revolute, parent hip_x, child toe_a_2/2, origin xyz=0.033685999999999945154 5.5511151231257827021e-17 -0.054400000000000010847 rpy=1.570796326794896558 -1.5706708750796685159 6.9310404253907578621e-11, axis 0 0 1, limit effort=1 velocity=20
- added joint spherical_free_hip_left: type revolute, parent tarsus_2, child toe_a_1/2_2, origin xyz=0.1141899349863718105 0.03620674973129278662 7.3552275381416620803e-16 rpy=-1.570796326794896558 -6.032224767520871884e-18 3.141592653589793116, axis 0 0 1, limit effort=1 velocity=20
- added joint spherical_free_knee: type revolute, parent tarsus, child toe_a_1/2, origin xyz=0.11418993498637028394 0.036206749731294674 0 rpy=-1.57079632679489678 -1.273128742691381099 -3.141592653589793116, axis 0 0 1, limit effort=1 velocity=20
- added joint spherical_free_knee_left: type revolute, parent hip_x_2, child toe_a_2/2_2, origin xyz=0.030568773343218405558 0 -0.054400000000000003908 rpy=-1.57079632679489678 1.570796326794896558 0, axis 0 0 1, limit effort=1 velocity=20
- added joint spherical_free_shin1: type revolute, parent crank_2, child toe_b_2/2_2, origin xyz=5.5511151231257827021e-17 0.057000000000000161648 0.0025000000000000160982 rpy=1.5707963267949196506 -1.477603911516246038 -1.5707963267949121011, axis 0 0 1, limit effort=1 velocity=20
- added joint spherical_free_shin1_left: type revolute, parent crank_4, child toe_b_1/2_4, origin xyz=2.2204460492503130808e-16 0.057000000000000494715 0.0025000000000004185541 rpy=-1.570796326794896558 -1.866329740155221443e-16 1.5707963267948970021, axis 0 0 1, limit effort=1 velocity=20
- added joint spherical_free_shin2: type revolute, parent crank, child toe_b_2/2, origin xyz=-1.6653345369377348106e-16 0.056999999999999828582 0.0025000000000000091593 rpy=-1.570796326794896558 -1.0576818073076525994 -1.5707963267948981123, axis 0 0 1, limit effort=1 velocity=20
- added joint spherical_free_shin2_left: type revolute, parent crank_3, child toe_b_2/2_4, origin xyz=-5.5511151231257827021e-17 0.057000000000000050626 0.0025000000000000022204 rpy=-1.57079632679489678 -6.1989581036318994383e-14 -1.570796326794896558, axis 0 0 1, limit effort=1 velocity=20
- joint closedloop1_A_frame: origin xyz=8.3266726846886740532e-17 -6.9388939039072283776e-18 -0.19994999999999990559 rpy=-3.7112781480334543363e-16 -7.6145285777054681417e-31 -1.2325951642497940378e-32 -> xyz=8.3266726846886740532e-17 -2.0816681711721685133e-17 -0.19994999999999985008 rpy=-3.6730477635741736581e-16 2.9460981308595112864e-21 7.5096808214324432057e-23
- joint closedloop1_B_frame: origin xyz=-4.1633363423443370266e-17 -8.3266726846886740532e-17 -0.19995000000000001661 rpy=3.141592653589793116 -4.3598202726084071025e-18 3.141592653589793116 -> xyz=-1.3877787807814456755e-17 -4.1633363423443370266e-17 -0.19995000000000007212 rpy=-3.141592653589793116 -1.7835368752394309275e-19 -3.141592653589793116
- joint closedloop2_A_frame: origin xyz=0 0 -0.11994999999999994555 rpy=1.7235773343990823765e-16 -3.2166375860020982159e-18 -9.2330428060222376469e-17 -> xyz=5.5511151231257827021e-17 1.1102230246251565404e-16 -0.11994999999999994555 rpy=2.1842893656284317977e-16 3.267742848578937711e-17 2.8391108377426899969e-17
- joint closedloop2_B_frame: origin xyz=-1.0408340855860842566e-16 1.6653345369377348106e-16 -0.11995000000000022311 rpy=3.141592653589793116 -3.4014104205904975495e-17 1.570796326794896558 -> xyz=-4.1633363423443370266e-17 5.5511151231257827021e-17 -0.11995000000000022311 rpy=3.141592653589793116 -9.2337153002951306109e-17 1.570796326794896558
- joint closedloop3_A_frame: origin xyz=-2.7755575615628913511e-17 0 -0.11994999999999972351 rpy=2.4425794194715678642e-16 -1.2567090974513322893e-17 9.4104185549181988163e-18 -> xyz=0 -1.1102230246251565404e-16 -0.11994999999999994555 rpy=4.3153759858238539441e-16 5.5326454623166440589e-19 2.690743573481835155e-17
- joint closedloop3_B_frame: origin xyz=-4.1633363423443370266e-17 5.5511151231257827021e-17 -0.11995000000000011209 rpy=-3.141592653589793116 6.050439432614581419e-18 1.570796326794896558 -> xyz=0 -5.5511151231257827021e-17 -0.11995000000000000107 rpy=-3.141592653589793116 1.4082337349770990484e-17 1.570796326794896558
- joint foot_frame: origin xyz=-0.055897619600577819199 2.7755575615628913511e-16 0.014375929767894812805 rpy=3.141592653589793116 1.0420837364882524767 3.141592653589793116 -> xyz=-0.055897619600577264087 1.3877787807814456755e-17 0.014375929767894479738 rpy=3.141592653589793116 1.0420837364882529208 3.141592653589793116
- joint free_foot1: origin xyz=-0.32599840000000002149 -0.038657982377658606232 -0.01400000000000004019 rpy=-3.1415926535897926719 3.4117039112211768089e-17 -2.8764747500822966941 -> xyz=-0.325998400000000077 -0.038657982377658606232 -0.014000000000000067946 rpy=3.141592653589793116 -5.0097838604174264603e-17 -2.8759599356941945025
- joint free_foot2: origin xyz=1.1102230246251565404e-16 0.0089999999999998969713 -0.013999999999999956923 rpy=-1.5707963267948961139 0.00018013600906293872469 -3.141592653589793116 -> xyz=1.1102230246251565404e-16 0.0089999999999999524825 -0.013999999999999998557 rpy=-1.570796326794896558 0.00022603698986956599648 -3.1415926535897913396
- joint free_knee: origin xyz=0.39567486363081366685 0.053875166733171879485 -0.025000000000000008327 rpy=3.141592653589793116 1.7052319612022700791e-18 -1.6910768536229012771 -> xyz=0.39567486363081449952 0.053875166733173364408 -0.024999999999999911182 rpy=-3.141592653589793116 1.7396919582285806086e-15 -1.6905869617439772679
- joint motor_hip_x: origin xyz=-0.02999999999999999889 -0.072799999999999975842 0.059867854479678822566 rpy=1.0689153541114032999e-25 1.570796326794896558 0 -> xyz=-0.02999999999999999889 -0.072799999999999975842 0.059867854479678822566 rpy=1.570796326794408504 1.5706708750796680718 1.570796326794408504
- joint motor_hip_y: origin xyz=-0.025999999999999995337 -2.7755575615628913511e-17 -0.054400000000000010847 rpy=-1.570796326794896336 -1.1931918349460142181 -1.570796326794896558 -> xyz=-0.026000000000000023093 5.5511151231257827021e-17 -0.05440000000000011493 rpy=-1.5707963267948976682 -1.1932852897669119496 -1.5707963267948954478
- joint motor_hip_z: origin xyz=0.05266579297345658911 1.3877787807814456755e-17 -0.035199999999999995182 rpy=-1.57079632679489678 1.1102230246014436281e-16 1.570796326794896558 -> xyz=0.052665792973456582171 0 -0.035199999999999995182 rpy=-1.570796326794896558 -0.000210470252546097027 1.570796326794896336
- joint motor_knee: origin xyz=-0.11999999999999998168 0 0 rpy=3.141592653589793116 1.6137487424794804186e-16 -2.6828651102102365478 -> xyz=-0.12000000000000010658 -5.5511151231257827021e-17 -2.7755575615628913511e-17 rpy=3.1415926535897926719 6.6787990227716521976e-17 -2.6827965911004429955
- joint motor_shin1: origin xyz=-0.088800000000000073319 -0.026113982377658606637 0.02999999999999999889 rpy=-3.141592653589793116 3.3674348063693462321e-18 0.085487820950950324517 -> xyz=-0.088800000000000045564 -0.026113982377658828682 0.029999999999999943379 rpy=-3.141592653589793116 -2.1102062293755973316e-16 0.086002635339051156094
- joint motor_shin2: origin xyz=-0.088800000000000017808 -0.02611398237765871766 -0.02999999999999999889 rpy=-7.5875284351392275809e-17 -8.5523186607038729703e-18 -3.0649221372054666901 -> xyz=-0.088799999999999990052 -0.026113982377658495615 -0.030000000000000026645 rpy=6.3640585351423805025e-17 -1.0365439080542638912e-15 -3.0644073228173649426
