Commit message: Update Digit

File: robots/digit_like_2legs_old/robot.urdf (robot description, URDF)
Before this commit: robot onshape, 46 links, 45 joints
Links:
- link foot_roll: mass 0.0027067106871796991867 -> 0.0027067106871796996204
- link foot_roll_2: mass 0.0027067106871796991867 -> 0.0027067106871796996204
- link shin: mass 0.55578140933316355632 -> 0.5557814093331634453
- link shin_2: mass 0.55578140933316355632 -> 0.5557814093331634453
Joints:
- joint closedloop2_A_frame: origin xyz=-5.5511151231257827021e-17 -3.4694469519536141888e-18 -0.11994999999999983453 rpy=3.4326414718463428853e-16 -3.9801083377604632754e-20 -1.7060090772934402995e-18 -> xyz=5.5511151231257827021e-17 -3.4694469519536141888e-18 -0.11994999999999994555 rpy=3.4063828878721196103e-16 -2.2014753343827181929e-20 6.3501031464105377993e-19
- joint closedloop2_B_frame: origin xyz=-1.3877787807814456755e-17 0 -0.1199500000000001676 rpy=-3.141592653589793116 -1.7785462404289089151e-17 1.570796326794896558 -> xyz=-2.7755575615628913511e-17 -1.1102230246251565404e-16 -0.11995000000000013984 rpy=3.141592653589793116 8.8295612703919830242e-17 1.570796326794896558
- joint closedloop3_A_frame: origin xyz=-5.5511151231257827021e-17 -1.3877787807814456755e-17 -0.11994999999999989004 rpy=5.4796299760769498158e-16 -1.6492169195407397826e-20 -3.2718841564329059315e-18 -> xyz=-5.5511151231257827021e-17 0 -0.11994999999999994555 rpy=5.4938147692151912312e-16 3.88885177613581823e-20 -1.9295956924994820687e-18
- joint closedloop3_B_frame: origin xyz=1.9949319973733281586e-17 -1.1102230246251565404e-16 -0.11995000000000011209 rpy=3.141592653589793116 6.1562166213320717002e-17 1.570796326794896558 -> xyz=1.3877787807814456755e-17 -1.1102230246251565404e-16 -0.11995000000000012597 rpy=-3.141592653589793116 -1.4358405587370260483e-17 1.570796326794896558
- joint closedloop4_A_frame: origin xyz=0 -5.5511151231257827021e-17 -0.11995000000000000107 rpy=-3.1415926535897926719 1.5256704509479419219e-15 1.57079632679489678 -> xyz=-2.7755575615628913511e-17 2.2204460492503130808e-16 -0.11995000000000013984 rpy=-3.1415926535897926719 1.4315792633067183667e-15 1.57079632679489678
- joint closedloop4_B_frame: origin xyz=-5.5511151231257827021e-17 -1.3877787807814456755e-17 -0.11994999999999994555 rpy=1.7099006292900051404e-16 -3.8344261464318977883e-16 -8.2337209764616805999e-17 -> xyz=5.5511151231257827021e-17 1.3877787807814456755e-17 -0.11994999999999989004 rpy=1.6709049170258792098e-16 -3.8336666344612196835e-16 -7.6597093190821181337e-17
- joint closedloop5_A_frame: origin xyz=2.7755575615628913511e-17 0 -0.11994999999999977902 rpy=-3.1415926535897922278 4.1186175175171797252e-15 1.570796326794896558 -> xyz=0 1.1102230246251565404e-16 -0.11995000000000000107 rpy=-3.1415926535897922278 4.1571142832877555497e-15 1.570796326794896558
- joint closedloop5_B_frame: origin xyz=0 0 -0.1199500000000001676 rpy=1.2623163092897104231e-16 1.1091301729747949746e-15 -3.141592653589793116 -> xyz=-5.5511151231257827021e-17 -6.9388939039072283776e-18 -0.11995000000000011209 rpy=1.258009249659380946e-16 1.1091975987985855455e-15 -3.141592653589793116
- joint foot_frame: origin xyz=-0.05589761960057737511 1.3877787807814456755e-17 0.014375929767894479738 rpy=3.1415926535897926719 1.0420837364882549192 3.141592653589793116 -> xyz=-0.05589761960057725021 0 0.014375929767894368716 rpy=3.1415926535897926719 1.0420837364882549192 -3.141592653589793116
- joint foot_left_frame: origin xyz=-0.055897619600577208576 -2.7755575615628913511e-17 0.0037840702321054742185 rpy=1.3316860532596122812e-16 -1.0420837364882493681 -3.141592653589793116 -> xyz=-0.05589761960057737511 0 0.0037840702321053631962 rpy=-3.2399764691790045377e-15 -1.0420837364882542531 3.141592653589793116
- joint free_foot1: origin xyz=-0.32599840000000002149 -0.038657982377658606232 -0.014000000000000067946 rpy=-3.1415926535897917837 -6.8122768436356686698e-17 1.8602703927245938242 -> xyz=-0.325998400000000077 -0.038657982377658606232 -0.014000000000000054068 rpy=-3.1415926535897917837 -1.2907497451769181967e-15 2.7453650200287231797
- joint free_foot1_left: origin xyz=-0.32599839999999913331 -0.038657982377660826678 -1.8041124150158793782e-16 rpy=1.3712330642673959594e-15 1.4865211215266053391e-15 1.8602703927245916038 -> xyz=-0.32599839999999896678 -0.038657982377660826678 -2.7755575615628913511e-16 rpy=9.1857826099949105318e-16 2.9669073048643708657e-16 2.7453650200287267324
- joint free_foot2: origin xyz=0 0.0089999999999999524825 -0.014000000000000012434 rpy=-1.570796326794896558 0.0068053161721140344523 -3.1415926535897904515 -> xyz=-2.7755575615628913511e-17 0.008999999999999785949 -0.014000000000000012434 rpy=-1.570796326794896558 0.0018265628936102844011 -3.1415926535897913396
- joint free_foot2_left: origin xyz=5.5511151231257827021e-17 0.0089999999999998969713 -2.7755575615628913511e-17 rpy=-1.570796326794896558 -0.0068053161721121089092 3.1415926535897917837 -> xyz=2.7755575615628913511e-17 0.0090000000000000079936 -1.3877787807814456755e-17 rpy=-1.5707963267948976682 -0.0018265628936090377854 3.1415926535897864547
- joint free_knee: origin xyz=0.39567486363081366685 0.053875166733171858668 -0.024999999999999994449 rpy=-3.1415926535897913396 -5.6727426674657804652e-16 -1.1259608736106343496 -> xyz=0.39567486363081377787 0.053875166733171803157 -0.025000000000000008327 rpy=-3.1415926535897913396 -5.6991269667964937762e-16 -1.1259608736106334614
- joint motor_hip_y: origin xyz=-0.025999999999999870437 4.1633363423443370266e-17 -0.054399999999993300936 rpy=1.5707963267948970021 -1.3059816663625789523 1.570796326794901665 -> xyz=-0.025999999999999967581 -1.3877787807814456755e-17 -0.054399999999999976152 rpy=1.5707963267948970021 -1.3059816663625809507 1.570796326794901665
- joint motor_hip_y_left: origin xyz=-0.029117226656781597383 0 -0.047379470518249235111 rpy=1.5707963267948958919 1.305981666362586946 1.5707963267949012209 -> xyz=-0.029117226656781597383 1.3877787807814456755e-17 -0.047379470518249228173 rpy=1.5707963267948958919 1.3059816663625891664 1.5707963267949012209
- joint motor_knee: origin xyz=-0.11999999999999930167 -1.1102230246251565404e-16 2.7755575615628913511e-17 rpy=-3.1415926535897900074 -2.8892848188444140326e-15 -1.5679404125952058902 -> xyz=-0.11999999999999313993 1.8457457784393227485e-15 9.7144514654701197287e-17 rpy=-3.1415926535897900074 -2.8790473541599528652e-15 -1.5679404125952072224
- joint motor_knee_left: origin xyz=0.12000000000000005107 2.6506574712925612403e-15 1.3877787807814456755e-17 rpy=-3.1415926535897917837 3.0237971669895305397e-15 -1.5552457051742101246 -> xyz=0.12000000000000005107 2.8727020762175925483e-15 1.3877787807814456755e-17 rpy=-3.1415926535897917837 3.0163080839021476512e-15 -1.5552457051742081262
- joint motor_shin1: origin xyz=-0.088800000000000017808 -0.02611398237765871766 0.029999999999999971134 rpy=3.141592653589793116 1.1559547673004707569e-15 0.7069149543481728637 -> xyz=-0.088799999999999962297 -0.026113982377658606637 0.029999999999999978073 rpy=3.141592653589793116 1.1588285902909991479e-15 0.70691495434820683652
- joint motor_shin1_left: origin xyz=-0.088799999999999004729 -0.026113982377660716061 0.02999999999999987399 rpy=3.141592653589793116 1.1145641153506547459e-15 0.70691495434817341881 -> xyz=-0.088799999999998935341 -0.02611398237766116015 0.029999999999999887867 rpy=3.141592653589793116 1.1035601505333686801e-15 0.70691495434820739163
- joint motor_shin2: origin xyz=-0.088800000000000017808 -0.02611398237765871766 -0.030000000000000012768 rpy=9.0029948949621089308e-16 -1.3909315756828847546e-15 -2.4346776992416199192 -> xyz=-0.08880000000000000393 -0.026113982377658606637 -0.030000000000000012768 rpy=8.9897733374673702766e-16 -1.372988716961691066e-15 -2.4346776992415857244
- joint motor_shin2_left: origin xyz=-0.088799999999999046363 -0.026113982377660827083 -0.030000000000000102973 rpy=1.4361021807975174281e-16 -1.2580190192396560789e-15 -2.4346776992416208074 -> xyz=-0.088799999999998990852 -0.026113982377661049128 -0.030000000000000130729 rpy=1.4227913028969940573e-16 -1.2435456074704160044e-15 -2.4346776992415866125
- joint spherical_free_foot1: origin xyz=-0.0091288304490430571825 -0.01427599999999996927 0.052813599999999905066 rpy=1.57079632679489678 0.17116739882267056894 -1.5707963267948981123 -> xyz=-0.0091288304490430710603 -0.01427599999999996927 0.05281360000000012711 rpy=1.570796326794896558 0.16707679024231919529 -1.5707963267948981123
- joint spherical_free_foot1_left: origin xyz=-0.0091288304490428351379 -0.014276000000000024781 -0.034653600000000062131 rpy=1.570796326794896558 0.17135811403969766764 -1.570796326794896336 -> xyz=-0.0091288304490430571825 -0.014276000000000010903 -0.034653600000000173154 rpy=1.570796326794896558 0.16726750545934601644 -1.57079632679489678
- joint spherical_free_foot2: origin xyz=-0.0091288304490430016713 0.014276000000000024781 0.052813600000000016088 rpy=1.570796326794896558 0.17116739882267226203 -1.570796326794896558 -> xyz=-0.0091288304490430155491 0.014275999999999997025 0.052813600000000238133 rpy=1.57079632679489678 0.16707679024232066634 -1.570796326794896558
- joint spherical_free_foot2_left: origin xyz=-0.009128830449042890649 0.014276000000000003964 -0.034653600000000117642 rpy=1.5707963267948950037 0.17135811403969555822 -1.5707963267948961139 -> xyz=-0.0091288304490430710603 0.014276000000000010903 -0.034653600000000173154 rpy=1.570796326794896558 0.16726750545934351844 -1.5707963267948958919
- joint spherical_free_shin1: origin xyz=5.5511151231257827021e-17 0.056999999999999884093 0.0025000000000000022204 rpy=-1.57079632679489678 0.040608021976129123065 1.5707963267948990005 -> xyz=5.5511151231257827021e-17 0.057000000000000050626 0.0025000000000000022204 rpy=-1.57079632679489678 0.040608021976129206332 1.5707963267948990005
- joint spherical_free_shin1_left: origin xyz=0 0.057000000000000050626 0.0024999999999999952816 rpy=-1.57079632679489678 -0.027781755534719884682 1.5707963267949012209 -> xyz=0 0.056999999999999939604 0.0025000000000000160982 rpy=-1.57079632679489678 -0.027781755534719749373 1.5707963267949012209
- joint spherical_free_shin2: origin xyz=0 0.057000000000000050626 0.0025000000000000022204 rpy=1.570796326794896558 -0.043999020249819484341 1.5707963267948952257 -> xyz=0 0.056999999999999884093 0.0025000000000000160982 rpy=1.570796326794896558 -0.043999020249819477402 1.5707963267948952257
- joint spherical_free_shin2_left: origin xyz=-1.1102230246251565404e-16 0.057000000000000106137 0.0024999999999999744649 rpy=-1.57079632679489678 -0.027781755534782608813 -1.5707963267949005548 -> xyz=5.5511151231257827021e-17 0.056999999999999995115 0.002500000000000029976 rpy=-1.57079632679489678 -0.027781755534782716366 -1.5707963267949005548
